Commit message: read parameter from yaml and urdf

File: cob3_defs/ros/defs/torso.urdf (robot description, URDF)
Before this commit: robot torso, 19 links, 18 joints
Joints:
- joint joint_headZ_head: limit lower=-1 upper=1 effort=100 velocity=5 -> lower=-1 upper=1 effort=100 velocity=0.5
- joint joint_neckZ_neck: limit lower=-0.5 upper=0.5 effort=100 velocity=1.0 -> lower=-0.1 upper=0.5 effort=100 velocity=0.5
- joint joint_neck_headZ: limit lower=-1 upper=1 effort=100 velocity=5 -> lower=-1 upper=1 effort=100 velocity=0.5
- joint joint_platform_neckZ: limit lower=-0.5 upper=0.5 effort=100 velocity=1.0 -> lower=-0.1 upper=0.5 effort=100 velocity=0.5

Commit message: added error handling and exact urdf parameters

File: cob3_defs/ros/defs/torso.urdf (robot description, URDF)
Before this commit: robot torso, 19 links, 18 joints
Joints:
- joint joint_headZ_head: limit lower=-1 upper=1 effort=100 velocity=0.5 -> lower=-1.5 upper=1.5 effort=100 velocity=0.5
- joint joint_neckZ_neck: limit lower=-0.1 upper=0.5 effort=100 velocity=0.5 -> lower=-1.5 upper=1.5 effort=100 velocity=0.5
- joint joint_neck_headZ: limit lower=-1 upper=1 effort=100 velocity=0.5 -> lower=-6.2831 upper=6.2831 effort=100 velocity=0.5
- joint joint_platform_neckZ: limit lower=-0.1 upper=0.5 effort=100 velocity=0.5 -> lower=-6.2831 upper=6.2831 effort=100 velocity=0.5

Commit message: neck is working

File: cob3_defs/ros/defs/torso.urdf (robot description, URDF)
Before this commit: robot torso, 19 links, 18 joints
Joints:
- joint joint_headZ_head: axis 0 1 0 -> 0 0 1; limit lower=-1.5 upper=1.5 effort=100 velocity=0.5 -> lower=-1.5 upper=1.5 effort=24 velocity=0.5; origin xyz=0 0 0.001 rpy=0 0 0 -> xyz=0 0 0 rpy=1.5708 0 0
- joint joint_head_eyes: axis 0 1 0 -> 0 0 1; limit lower=-1 upper=1 effort=100 velocity=5 -> lower=-0.1745 upper=3.316 effort=100 velocity=0.5; origin xyz=-0.1 0 0.2 rpy=0 0 0 -> xyz=0 -0.1575 0 rpy=0 0 0
- joint joint_neckZ_neck: axis 0 1 0 -> 0 0 1; limit lower=-1.5 upper=1.5 effort=100 velocity=0.5 -> lower=-1.5 upper=1.5 effort=46 velocity=0.5; origin xyz=0 0 0.001 rpy=0 0 0 -> xyz=0 0 -0.115 rpy=1.5708 0 0
- joint joint_neck_headZ: limit lower=-6.2831 upper=6.2831 effort=100 velocity=0.5 -> lower=-6.2831 upper=6.2831 effort=4 velocity=0.5; origin xyz=-0.09039 0 0.30489 rpy=0 0 0 -> xyz=0 -0.237 0.0 rpy=-1.5708 0 0
- joint joint_platform_neckZ: limit lower=-6.2831 upper=6.2831 effort=100 velocity=0.5 -> lower=-6.2831 upper=6.2831 effort=24 velocity=0.5; origin xyz=0.24627 0 0.7798 rpy=0 0 0 -> xyz=0.155 0 0.7798 rpy=3.1415926 0 0

Commit message: version of powercubes with trajectory controller

File: cob3_defs/ros/defs/torso.urdf (robot description, URDF)
Before this commit: robot torso, 19 links, 18 joints
Joints:
- joint joint_head_eyes: origin xyz=0 -0.1575 0 rpy=0 0 0 -> xyz=0 -0.154 0 rpy=0 0 0
