Commit message: working version of arm, correct arm defs

File: cob3_defs/ros/defs/arm.urdf (robot description, URDF)
Before this commit: robot arm, 8 links, 7 joints
Joints:
- joint joint_arm1: origin xyz=0 0 0.0569 rpy=0 0 0 -> xyz=0 0 -0.25 rpy=0 0 0
- joint joint_arm2: axis 0 1 0 -> 0 0 1; origin xyz=0 0 0.1931 rpy=0 0 0 -> xyz=0 0 0 rpy=1.5708 0 0
- joint joint_arm3: origin xyz=0 0 0.110 rpy=0 0 0 -> xyz=0 -0.408 0 rpy=-1.5708 0 0
- joint joint_arm4: axis 0 1 0 -> 0 0 1; origin xyz=0 0 0.298 rpy=0 0 0 -> xyz=0 0 0 rpy=1.5708 0 0
- joint joint_arm5: origin xyz=0 0 0.100 rpy=0 0 0 -> xyz=0 -0.3165 0 rpy=-1.5708 0 0
- joint joint_arm6: axis 0 1 0 -> 0 0 1; origin xyz=0 0 0.2165 rpy=0 0 0 -> xyz=0 0 0 rpy=1.5708 0 0
- joint joint_arm7: origin xyz=0 0 0.080 rpy=0 0 0 -> xyz=0 -0.1927 0 rpy=-1.5708 0 0
