Commit message: care-o-bot picture at ipa kitchen

File: cob_gazebo_worlds/common/worlds/ipa-kitchen.urdf (robot description, URDF)
Before this commit: robot ipa_kitchen, 14 links, 13 joints
Links:
- removed link box1
- removed link box2
- removed link box3
- removed link dummy_link
- removed link sofa
- removed link wall_1
- removed link wall_2
- removed link wall_3
- removed link wall_4
- removed link wall_5
- removed link wall_6
- removed link wall_7
- removed link wall_8
- removed link wall_9
Joints:
- removed joint joint_box1
- removed joint joint_box2
- removed joint joint_box3
- removed joint joint_sofa
- removed joint joint_wall_1
- removed joint joint_wall_2
- removed joint joint_wall_3
- removed joint joint_wall_4
- removed joint joint_wall_5
- removed joint joint_wall_6
- removed joint joint_wall_7
- removed joint joint_wall_8
- removed joint joint_wall_9
