Commit message: modified ipa-kitchen.urdf.xacro

File: cob_gazebo_worlds/common/worlds/ipa-kitchen.urdf.xacro (robot description, xacro)
@@ -297,84 +297,81 @@
     <child link="sofa"/>
  </joint>
-  <link name="box1">
-    <inertial>
-      <origin xyz="0 0 0" />
-      <mass value="1.0" />
-      <inertia  ixx="1.0" ixy="0.0"  ixz="0.0"  iyy="100.0"  iyz="0.0"  izz="1.0" />
-    </inertial>
-    <visual>
-      <origin xyz="0 0 0"/>
-      <geometry>
-        <box size="0.6 0.6 1.4" />
-      </geometry>
-    </visual>
-    <collision>
-      <origin xyz="0 0 0"/>
-      <geometry>
-        <box size="1.75 0.89 0.45" />
-      </geometry>
-    </collision>
-  </link>
-  <gazebo reference="box1">
-    <material>Gazebo/Red</material>
-  </gazebo>
-   <joint name="joint_box1" type="fixed">
-    <origin xyz="-3.2 1.36 0.7" rpy="0 0 0"/>
-    <parent link="dummy_link"/>
-    <child link="box1"/>
- </joint>
-   <link name="box2">
-    <inertial>
-      <origin xyz="0 0 0" />
-      <mass value="1.0" />
-      <inertia  ixx="1.0" ixy="0.0"  ixz="0.0"  iyy="100.0"  iyz="0.0"  izz="1.0" />
-    </inertial>
-    <visual>
-      <origin xyz="0 0 0"/>
-      <geometry>
-        <box size="0.6 1.8 0.85" />
-      </geometry>
-    </visual>
-    <collision>
-      <origin xyz="0 0 0"/>
-      <geometry>
-        <box size="0.6 1.8 0.85" />
-      </geometry>
-    </collision>
-  </link>
-  <gazebo reference="box2">
-    <material>Gazebo/Blue</material>
-  </gazebo>
-   <joint name="joint_box2" type="fixed">
-    <origin xyz="-3.2 0.16 0.425" rpy="0 0 0"/>
-    <parent link="dummy_link"/>
-    <child link="box2"/>
- </joint>
-   <link name="box3">
-    <inertial>
-      <origin xyz="0 0 0" />
-      <mass value="1.0" />
-      <inertia  ixx="1.0" ixy="0.0"  ixz="0.0"  iyy="100.0"  iyz="0.0"  izz="1.0" />
-    </inertial>
-    <visual>
-      <origin xyz="0 0 0"/>
-      <geometry>
-        <box size="0.6 0.6 1.4" />
-      </geometry>
-    </visual>
-    <collision>
-      <origin xyz="0 0 0"/>
-      <geometry>
-        <box size="0.6 0.6 1.4" />
-      </geometry>
-    </collision>
-  </link>
-  <gazebo reference="box3">
-    <material>Gazebo/Red</material>
-  </gazebo>
-   <joint name="joint_box3" type="fixed">
-    <origin xyz="-3.2 -1.04 0.7" rpy="0 0 0"/>
-    <parent link="dummy_link"/>
-    <child link="box3"/>
+   <link name="kitchen_right">
+    <inertial>
+      <origin xyz="0 0 0" />
+      <mass value="1.0" />
+      <inertia  ixx="1.0" ixy="0.0"  ixz="0.0"  iyy="100.0"  iyz="0.0"  izz="1.0" />
+    </inertial>
+    <visual>
+      <origin xyz="0 0 0"/>
+      <geometry>
+		<mesh filename="package://cob_gazebo_worlds/Media/materials/textures/kitchen_right.dae"/>
+      </geometry>
+    </visual>
+    <collision>
+      <origin xyz="0 0 0"/>
+      <geometry>
+        <box size="0.66 0.62 1.44" />
+      </geometry>
+    </collision>
+  </link>
+  <gazebo reference="kitchen_right">
+  </gazebo>
+   <joint name="joint_kitchen_right" type="fixed">
+    <origin xyz="-3.141 1.321 0.72" rpy="0 0 0"/>
+    <parent link="dummy_link"/>
+    <child link="kitchen_right"/>
+ </joint>
+   <link name="kitchen_middle">
+    <inertial>
+      <origin xyz="0 0 0" />
+      <mass value="1.0" />
+      <inertia  ixx="1.0" ixy="0.0"  ixz="0.0"  iyy="100.0"  iyz="0.0"  izz="1.0" />
+    </inertial>
+    <visual>
+      <origin xyz="0 0 0"/>
+      <geometry>
+		<mesh filename="package://cob_gazebo_worlds/Media/materials/textures/kitchen_middle.dae"/>
+      </geometry>
+    </visual>
+    <collision>
+      <origin xyz="0 0 0"/>
+      <geometry>
+        <box size="0.66 1.8 0.9" />
+      </geometry>
+    </collision>
+  </link>
+  <gazebo reference="kitchen_middle">
+  </gazebo>
+   <joint name="joint_kitchen_middle" type="fixed">
+    <origin xyz="-3.141 0.111 0.45" rpy="0 0 0"/>
+    <parent link="dummy_link"/>
+    <child link="kitchen_middle"/>
+ </joint>
+  <link name="kitchen_left">
+    <inertial>
+      <origin xyz="0 0 0" />
+      <mass value="1.0" />
+      <inertia  ixx="1.0" ixy="0.0"  ixz="0.0"  iyy="100.0"  iyz="0.0"  izz="1.0" />
+    </inertial>
+    <visual>
+      <origin xyz="0 0 0"/>
+      <geometry>
+		<mesh filename="package://cob_gazebo_worlds/Media/materials/textures/kitchen_left.dae"/>
+      </geometry>
+    </visual>
+    <collision>
+      <origin xyz="0 0 0"/>
+      <geometry>
+        <box size="0.66 0.62 1.44" />
+      </geometry>
+    </collision>
+  </link>
+  <gazebo reference="kitchen_left">
+  </gazebo>
+   <joint name="joint_kitchen_left" type="fixed">
+    <origin xyz="-3.141 -1.099 0.72" rpy="0 0 0"/>
+    <parent link="dummy_link"/>
+    <child link="kitchen_left"/>
  </joint>
   <link name="picture_cob">

Commit message: changes to ipa-kitchen for freezer door

File: cob_gazebo_worlds/common/worlds/ipa-kitchen.urdf.xacro (robot description, xacro)
@@ -5,10 +5,11 @@
        xmlns:xacro="http://playerstage.sourceforge.net/gazebo/xmlschema/#interface"
        name="ipa-kitchen" >
+  <property name="M_PI" value="3.1415926535897931" />
 <xacro:macro name="ipa-kitchen" params="name">
   <link name="dummy_link">
     <inertial>
-      <origin xyz="0 0 0" />
-      <mass value="1.0" />
-      <inertia  ixx="1.0" ixy="0.0"  ixz="0.0"  iyy="100.0"  iyz="0.0"  izz="1.0" />
+      <origin xyz="0 0 -10" />
+      <mass value="100000.0" />
+      <inertia  ixx="100.0" ixy="0.0"  ixz="0.0"  iyy="100.0"  iyz="0.0"  izz="100.0" />
     </inertial>
     <visual>
@@ -297,5 +298,5 @@
     <child link="sofa"/>
  </joint>
-  <link name="box1">
+  <link name="kaffe_maschine">
     <inertial>
       <origin xyz="0 0 0" />
@@ -312,17 +313,17 @@
       <origin xyz="0 0 0"/>
       <geometry>
-        <box size="1.75 0.89 0.45" />
-      </geometry>
-    </collision>
-  </link>
-  <gazebo reference="box1">
+        <box size="0.6 0.6 1.4" />
+      </geometry>
+    </collision>
+  </link>
+  <gazebo reference="kaffe_maschine">
     <material>Gazebo/Red</material>
   </gazebo>
-   <joint name="joint_box1" type="fixed">
-    <origin xyz="-3.2 1.36 0.7" rpy="0 0 0"/>
-    <parent link="dummy_link"/>
-    <child link="box1"/>
- </joint>
-   <link name="box2">
+   <joint name="joint_kaffe_maschine" type="fixed">
+    <origin xyz="-3.2 -1.04 0.7" rpy="0 0 0"/>
+    <parent link="dummy_link"/>
+    <child link="kaffe_maschine"/>
+ </joint>
+   <link name="spuele">
     <inertial>
       <origin xyz="0 0 0" />
@@ -343,38 +344,94 @@
     </collision>
   </link>
-  <gazebo reference="box2">
+  <gazebo reference="spuele">
     <material>Gazebo/Blue</material>
   </gazebo>
-   <joint name="joint_box2" type="fixed">
+   <joint name="joint_spuele" type="fixed">
     <origin xyz="-3.2 0.16 0.425" rpy="0 0 0"/>
     <parent link="dummy_link"/>
-    <child link="box2"/>
- </joint>
-   <link name="box3">
-    <inertial>
-      <origin xyz="0 0 0" />
-      <mass value="1.0" />
-      <inertia  ixx="1.0" ixy="0.0"  ixz="0.0"  iyy="100.0"  iyz="0.0"  izz="1.0" />
-    </inertial>
-    <visual>
-      <origin xyz="0 0 0"/>
-      <geometry>
-        <box size="0.6 0.6 1.4" />
-      </geometry>
-    </visual>
-    <collision>
-      <origin xyz="0 0 0"/>
-      <geometry>
-        <box size="0.6 0.6 1.4" />
-      </geometry>
-    </collision>
-  </link>
-  <gazebo reference="box3">
+    <child link="spuele"/>
+ </joint>
+<!--
+   <link name="freezer_right">
+    <inertial>
+      <origin xyz="0 0 0" />
+      <mass value="1.0" />
+      <inertia  ixx="1.0" ixy="0.0"  ixz="0.0"  iyy="100.0"  iyz="0.0"  izz="1.0" />
+    </inertial>
+    <visual>
+      <origin xyz="0 0 0"/>
+      <geometry>
+        <box size="0.6 0.01 1.4" />
+      </geometry>
+    </visual>
+    <collision>
+      <origin xyz="0 0 0"/>
+      <geometry>
+        <box size="0.6 0.01 1.4" />
+      </geometry>
+    </collision>
+  </link>
+  <gazebo reference="freezer_right">
     <material>Gazebo/Red</material>
   </gazebo>
-   <joint name="joint_box3" type="fixed">
-    <origin xyz="-3.2 -1.04 0.7" rpy="0 0 0"/>
-    <parent link="dummy_link"/>
-    <child link="box3"/>
+   <joint name="joint_freezer_right" type="fixed">
+    <origin xyz="-3.2 1.66 0.7" rpy="0 0 0"/>
+    <parent link="dummy_link"/>
+    <child link="freezer_right"/>
+ </joint>
+ -->
+  <link name="freezer_left">
+    <inertial>
+      <origin xyz="0 0 0" />
+      <mass value="1.0" />
+      <inertia  ixx="1.0" ixy="0.0"  ixz="0.0"  iyy="100.0"  iyz="0.0"  izz="1.0" />
+    </inertial>
+    <visual>
+      <origin xyz="0 0 0"/>
+      <geometry>
+        <box size="0.6 0.01 1.4" />
+      </geometry>
+    </visual>
+    <collision>
+      <origin xyz="0 0 0"/>
+      <geometry>
+        <box size="0.6 0.01 1.4" />
+      </geometry>
+    </collision>
+  </link>
+  <gazebo reference="freezer_left">
+    <material>Gazebo/Red</material>
+  </gazebo>
+   <joint name="joint_freezer_left" type="fixed">
+    <origin xyz="-3.2 1.06 0.7" rpy="0 0 0"/>
+    <parent link="dummy_link"/>
+    <child link="freezer_left"/>
+ </joint>
+  <link name="freezer_top">
+    <inertial>
+      <origin xyz="0 0 0" />
+      <mass value="1.0" />
+      <inertia  ixx="1.0" ixy="0.0"  ixz="0.0"  iyy="100.0"  iyz="0.0"  izz="1.0" />
+    </inertial>
+    <visual>
+      <origin xyz="0 0 0"/>
+      <geometry>
+        <box size="0.6 0.6 0.01" />
+      </geometry>
+    </visual>
+    <collision>
+      <origin xyz="0 0 0"/>
+      <geometry>
+        <box size="0.6 0.6 0.01" />
+      </geometry>
+    </collision>
+  </link>
+  <gazebo reference="freezer_top">
+    <material>Gazebo/Red</material>
+  </gazebo>
+   <joint name="joint_freezer_top" type="fixed">
+    <origin xyz="-3.2 1.36 1.4" rpy="0 0 0"/>
+    <parent link="dummy_link"/>
+    <child link="freezer_top"/>
  </joint>
   <link name="picture_cob">
@@ -513,4 +570,129 @@
     <child link="comic"/>
  </joint>
+ <!-- Start simulated freezer door -->
+    <link name="freezer_right">
+    <inertial>
+      <origin xyz="0 0 0" />
+      <mass value="100.0" />
+      <inertia  ixx="1.0" ixy="0.0"  ixz="0.0"  iyy="100.0"  iyz="0.0"  izz="1.0" />
+    </inertial>
+    <visual>
+      <origin xyz="0 0 0"/>
+      <geometry>
+        <box size="0.6 0.01 1.4" />
+      </geometry>
+    </visual>
+    <collision>
+      <origin xyz="0 0 0"/>
+      <geometry>
+        <box size="0.6 0.01 1.4" />
+      </geometry>
+    </collision>
+  </link>
+  <gazebo reference="freezer_right">
+    <material>Gazebo/Red</material>
+  </gazebo>
+   <joint name="joint_freezer_right" type="fixed">
+    <origin xyz="-3.2 1.66 0.7" rpy="0 0 0"/>
+    <parent link="dummy_link"/>
+    <child link="freezer_right"/>
+ </joint>
+  <gazebo reference="door_link">
+    <latchJoint>handle_joint</latchJoint>
+    <latchAngle>-1.57</latchAngle>
+    <doorClosedAngle>0.0</doorClosedAngle>
+    <latchKp>200.0</latchKp>
+    <latchKd>0.0</latchKd>
+    <latchFMax>1000.0</latchFMax>
+  </gazebo>
+  <joint name="door_joint" type="revolute" >
+    <origin xyz="0.305 0 0.02" rpy="0 0 0" />
+    <axis xyz="0 0 1" />
+    <limit lower="${-M_PI}" upper="${M_PI}" effort="1000" velocity="10" />
+    <safety_controller soft_lower_limit="${-M_PI+0.1}" soft_upper_limit="${M_PI-0.1}"
+           k_position="100.0" k_velocity="10.0" />
+    <dynamics damping="100" friction="0.0" />
+    <parent link="freezer_right" />
+    <child link="door_link" />
+  </joint>
+  <link name="door_link">
+    <inertial >
+      <mass value="30" />
+      <origin xyz="0 0 0" />
+      <inertia  ixx="1.0" ixy="0.0"  ixz="0.0"
+                iyy="1.0" iyz="0.0"
+                izz="3.0" />
+    </inertial>
+    <visual >
+      <origin xyz="0 -0.305 0" rpy="0 0 ${M_PI}" />
+      <geometry name="sholder_roll_mesh_file">
+        <box size="0.01 0.59 1.36" />
+      </geometry>
+    </visual>
+    <collision >
+      <origin xyz="0 -0.305 0" rpy="0 0 ${M_PI}" />
+      <geometry name="door_collision_geom">
+        <box size="0.01 0.59 1.36" />
+      </geometry>
+    </collision>
+  </link>
+  <gazebo reference="door_link">
+    <material>Gazebo/Yellow</material>
+    <laserRetro>2000</laserRetro>
+    <turnGravityOff>true</turnGravityOff>
+    <selfCollide>false</selfCollide>
+    <dampingFactor>0.01</dampingFactor>
+  </gazebo>
+   <link name="handle">
+    <inertial>
+      <origin xyz="0 0 0" />
+      <mass value="1.0" />
+      <inertia  ixx="1.0" ixy="0.0"  ixz="0.0"  iyy="100.0"  iyz="0.0"  izz="1.0" />
+    </inertial>
+    <visual>
+      <origin xyz="0 0 0"/>
+      <geometry>
+        <box size="0.08 0.01 0.3" />
+      </geometry>
+    </visual>
+    <collision>
+      <origin xyz="0 0 0"/>
+      <geometry>
+        <box size="0.08 0.01 0.3" />
+      </geometry>
+    </collision>
+  </link>
+  <gazebo reference="handle">
+    <material>Gazebo/Blue</material>
+  </gazebo>
+   <joint name="joint_handle" type="fixed">
+    <origin xyz="0.051 -0.55  0.0" rpy="0 0 0"/>
+    <parent link="door_link"/>
+    <child link="handle"/>
+ </joint>
+  <gazebo>
+    <!-- gazebo_ros_p3d for position groundtruth -->
+    <controller:gazebo_ros_p3d name="p3d_door_controller" plugin="libgazebo_ros_p3d.so">
+        <alwaysOn>true</alwaysOn>
+        <updateRate>100.0</updateRate>
+        <bodyName>door_link</bodyName>
+        <topicName>door_pose</topicName>
+        <frameName>/map</frameName>
+        <interface:position name="p3d_door_position"/>
+    </controller:gazebo_ros_p3d>
+    <controller:gazebo_ros_controller_manager name="door_controller_manager" plugin="libgazebo_ros_controller_manager.so">
+      <alwaysOn>true</alwaysOn>
+      <updateRate>1000.0</updateRate>
+      <robotParam>/world_description</robotParam>
+      <robotNamespace>/world</robotNamespace>
+      <interface:audio name="gazebo_ros_controller_manager_dummy_iface" />
+    </controller:gazebo_ros_controller_manager>
+  </gazebo>
+  <!-- transmission mechanism controls -->
+  <transmission type="pr2_mechanism_model/SimpleTransmission" name="door_trans">
+    <actuator name="door_motor" />
+    <joint name="door_joint" />
+    <mechanicalReduction>100</mechanicalReduction>
+  </transmission>
 </xacro:macro>
   <xacro:ipa-kitchen name="ipa-kitchen"/>

Commit message: added new controllers for platform verrsion 1

File: cob_gazebo_worlds/common/worlds/ipa-kitchen.urdf.xacro (robot description, xacro)
@@ -402,5 +402,5 @@
   </gazebo>
    <joint name="joint_freezer_top" type="fixed">
-    <origin xyz="-3.2 1.36 1.4" rpy="0 0 0"/>
+    <origin xyz="-3.15 1.36 1.4" rpy="0 0 0"/>
     <parent link="dummy_link"/>
     <child link="freezer_top"/>
@@ -542,4 +542,31 @@
  </joint>
  <!-- Start simulated freezer door -->
+	<link name="freezer_left">
+    <inertial>
+      <origin xyz="0 0 0" />
+      <mass value="100.0" />
+      <inertia  ixx="1.0" ixy="0.0"  ixz="0.0"  iyy="100.0"  iyz="0.0"  izz="1.0" />
+    </inertial>
+    <visual>
+      <origin xyz="0 0 0"/>
+      <geometry>
+        <box size="0.6 0.01 1.4" />
+      </geometry>
+    </visual>
+    <collision>
+      <origin xyz="0 0 0"/>
+      <geometry>
+        <box size="0.55 0.005 1.38" />
+      </geometry>
+    </collision>
+  </link>
+  <gazebo reference="freezer_left">
+    <material>Gazebo/Red</material>
+  </gazebo>
+   <joint name="joint_freezer_lefft" type="fixed">
+    <origin xyz="-3.15 1.06 0.7" rpy="0 0 0"/>
+    <parent link="dummy_link"/>
+    <child link="freezer_left"/>
+ </joint>
     <link name="freezer_right">
     <inertial>
@@ -557,5 +584,5 @@
       <origin xyz="0 0 0"/>
       <geometry>
-        <box size="0.6 0.01 1.4" />
+        <box size="0.55 0.005 1.38" />
       </geometry>
     </collision>
@@ -565,5 +592,5 @@
   </gazebo>
    <joint name="joint_freezer_right" type="fixed">
-    <origin xyz="-3.2 1.66 0.7" rpy="0 0 0"/>
+    <origin xyz="-3.15 1.66 0.7" rpy="0 0 0"/>
     <parent link="dummy_link"/>
     <child link="freezer_right"/>
@@ -604,5 +631,5 @@
       <origin xyz="0 -0.305 0" rpy="0 0 ${M_PI}" />
       <geometry name="door_collision_geom">
-        <box size="0.01 0.59 1.36" />
+        <box size="0.0 0 0" />
       </geometry>
     </collision>
@@ -630,5 +657,5 @@
       <origin xyz="0 0 0"/>
       <geometry>
-        <box size="0.08 0.01 0.3" />
+        <box size="0.07 0.005 0.25" />
       </geometry>
     </collision>
