Commit message: modified models and added four new objects

File: cob_gazebo_worlds/common/worlds/ipa-kitchen.urdf.xacro (robot description, xacro)
@@ -1,43 +1,858 @@
 <?xml version="1.0"?>
-<robot xmlns:sensor="http://playerstage.sourceforge.net/gazebo/xmlschema/#sensor"
-       xmlns:controller="http://playerstage.sourceforge.net/gazebo/xmlschema/#controller"
-       xmlns:interface="http://playerstage.sourceforge.net/gazebo/xmlschema/#interface"
-       xmlns:xacro="http://playerstage.sourceforge.net/gazebo/xmlschema/#interface"
-       name="ipa-kitchen" >
+<robot
+	xmlns:sensor="http://playerstage.sourceforge.net/gazebo/xmlschema/#sensor"
+	xmlns:controller="http://playerstage.sourceforge.net/gazebo/xmlschema/#controller"
+	xmlns:interface="http://playerstage.sourceforge.net/gazebo/xmlschema/#interface"
+	xmlns:xacro="http://playerstage.sourceforge.net/gazebo/xmlschema/#interface"
+	name="ipa-kitchen"
+>
 <xacro:macro name="ipa-kitchen" params="name">
-  <link name="dummy_link">
+<!-- dummy_link -->
+	<link name="dummy_link">
+		<inertial>
+			<origin xyz="0 0 0" />
+			<mass value="5.0" />
+			<inertia  ixx="0.0" ixy="0.0"  ixz="0.0"  iyy="0.0"  iyz="0.0"  izz="0.0" />
+		</inertial>
+		<visual>
+			<origin xyz="0 0 0" />
+			<geometry>
+				<box size="0.01 0.01 0.01" />
+			</geometry>
+		</visual>
+		<collision>
+			<origin xyz="0 0 0" />
+			<geometry>
+				<box size="0.01 0.01 0.01" />
+			</geometry>
+		</collision>
+	</link>
+<!-- walls -->
+<!-- wall_00 -->
+	<link name="wall_00">
+		<inertial>
+			<origin xyz="0 0 0" />
+			<mass value="5.0" />
+			<inertia  ixx="0.0" ixy="0.0"  ixz="0.0"  iyy="0.0"  iyz="0.0"  izz="0.0" />
+		</inertial>
+		<visual>
+			<origin xyz="0 0 0" />
+			<geometry>
+				<box size="2.75 0.06 0.50" />
+			</geometry>
+		</visual>
+		<collision>
+			<origin xyz="0 0 0" />
+			<geometry>
+				<box size="2.73 0.04 0.48" />
+			</geometry>
+		</collision>
+	</link>
+	<gazebo reference="wall_00">
+		<material>IPA/Wall2</material>
+	</gazebo>
+	<joint name="joint_wall_00" type="fixed">
+		<origin xyz="-2.156 4.791 0.250" rpy="0 0 0" />
+		<parent link="dummy_link" />
+		<child link="wall_00" />
+	</joint>
+<!-- wall_01 -->
+	<link name="wall_01">
+		<inertial>
+			<origin xyz="0 0 0" />
+			<mass value="5.0" />
+			<inertia  ixx="0.0" ixy="0.0"  ixz="0.0"  iyy="0.0"  iyz="0.0"  izz="0.0" />
+		</inertial>
+		<visual>
+			<origin xyz="0 0 0" />
+			<geometry>
+				<box size="0.10 0.80 2.40" />
+			</geometry>
+		</visual>
+		<collision>
+			<origin xyz="0 0 0" />
+			<geometry>
+				<box size="0.08 0.78 2.38" />
+			</geometry>
+		</collision>
+	</link>
+	<gazebo reference="wall_01">
+		<material>IPA/Wall</material>
+	</gazebo>
+	<joint name="joint_wall_01" type="fixed">
+		<origin xyz="-0.731 4.421 1.200" rpy="0 0 0" />
+		<parent link="dummy_link" />
+		<child link="wall_01" />
+	</joint>
+<!-- wall_02 -->
+	<link name="wall_02">
+		<inertial>
+			<origin xyz="0 0 0" />
+			<mass value="5.0" />
+			<inertia  ixx="0.0" ixy="0.0"  ixz="0.0"  iyy="0.0"  iyz="0.0"  izz="0.0" />
+		</inertial>
+		<visual>
+			<origin xyz="0 0 0" />
+			<geometry>
+				<box size="3.29 0.06 0.50" />
+			</geometry>
+		</visual>
+		<collision>
+			<origin xyz="0 0 0" />
+			<geometry>
+				<box size="3.27 0.04 0.48" />
+			</geometry>
+		</collision>
+	</link>
+	<gazebo reference="wall_02">
+		<material>IPA/Wall2</material>
+	</gazebo>
+	<joint name="joint_wall_02" type="fixed">
+		<origin xyz="0.964 4.791 0.250" rpy="0 0 0" />
+		<parent link="dummy_link" />
+		<child link="wall_02" />
+	</joint>
+<!-- wall_03 -->
+	<link name="wall_03">
+		<inertial>
+			<origin xyz="0 0 0" />
+			<mass value="5.0" />
+			<inertia  ixx="0.0" ixy="0.0"  ixz="0.0"  iyy="0.0"  iyz="0.0"  izz="0.0" />
+		</inertial>
+		<visual>
+			<origin xyz="0 0 0" />
+			<geometry>
+				<box size="0.80 0.10 3.20" />
+			</geometry>
+		</visual>
+		<collision>
+			<origin xyz="0 0 0" />
+			<geometry>
+				<box size="0.78 0.08 3.18" />
+			</geometry>
+		</collision>
+	</link>
+	<gazebo reference="wall_03">
+		<material>IPA/Wall</material>
+	</gazebo>
+	<joint name="joint_wall_03" type="fixed">
+		<origin xyz="3.009 4.771 1.600" rpy="0 0 0" />
+		<parent link="dummy_link" />
+		<child link="wall_03" />
+	</joint>
+<!-- wall_04 -->
+	<link name="wall_04">
+		<inertial>
+			<origin xyz="0 0 0" />
+			<mass value="5.0" />
+			<inertia  ixx="0.0" ixy="0.0"  ixz="0.0"  iyy="0.0"  iyz="0.0"  izz="0.0" />
+		</inertial>
+		<visual>
+			<origin xyz="0 0 0" />
+			<geometry>
+				<box size="0.06 6.80 0.50" />
+			</geometry>
+		</visual>
+		<collision>
+			<origin xyz="0 0 0" />
+			<geometry>
+				<box size="0.04 6.78 0.48" />
+			</geometry>
+		</collision>
+	</link>
+	<gazebo reference="wall_04">
+		<material>IPA/Wall2</material>
+	</gazebo>
+	<joint name="joint_wall_04" type="fixed">
+		<origin xyz="3.379 1.321 0.250" rpy="0 0 0" />
+		<parent link="dummy_link" />
+		<child link="wall_04" />
+	</joint>
+<!-- wall_05 -->
+	<link name="wall_05">
+		<inertial>
+			<origin xyz="0 0 0" />
+			<mass value="5.0" />
+			<inertia  ixx="0.0" ixy="0.0"  ixz="0.0"  iyy="0.0"  iyz="0.0"  izz="0.0" />
+		</inertial>
+		<visual>
+			<origin xyz="0 0 0" />
+			<geometry>
+				<box size="0.80 0.10 3.20" />
+			</geometry>
+		</visual>
+		<collision>
+			<origin xyz="0 0 0" />
+			<geometry>
+				<box size="0.78 0.08 3.18" />
+			</geometry>
+		</collision>
+	</link>
+	<gazebo reference="wall_05">
+		<material>IPA/Wall</material>
+	</gazebo>
+	<joint name="joint_wall_05" type="fixed">
+		<origin xyz="3.009 -2.129 1.600" rpy="0 0 0" />
+		<parent link="dummy_link" />
+		<child link="wall_05" />
+	</joint>
+<!-- wall_06 -->
+	<link name="wall_06">
+		<inertial>
+			<origin xyz="0 0 0" />
+			<mass value="5.0" />
+			<inertia  ixx="0.0" ixy="0.0"  ixz="0.0"  iyy="0.0"  iyz="0.0"  izz="0.0" />
+		</inertial>
+		<visual>
+			<origin xyz="0 0 0" />
+			<geometry>
+				<box size="6.14 0.06 0.50" />
+			</geometry>
+		</visual>
+		<collision>
+			<origin xyz="0 0 0" />
+			<geometry>
+				<box size="6.12 0.04 0.48" />
+			</geometry>
+		</collision>
+	</link>
+	<gazebo reference="wall_06">
+		<material>IPA/Wall2</material>
+	</gazebo>
+	<joint name="joint_wall_06" type="fixed">
+		<origin xyz="-0.461 -2.149 0.250" rpy="0 0 0" />
+		<parent link="dummy_link" />
+		<child link="wall_06" />
+	</joint>
+<!-- wall_07 -->
+	<link name="wall_07">
+		<inertial>
+			<origin xyz="0 0 0" />
+			<mass value="5.0" />
+			<inertia  ixx="0.0" ixy="0.0"  ixz="0.0"  iyy="0.0"  iyz="0.0"  izz="0.0" />
+		</inertial>
+		<visual>
+			<origin xyz="0 0 0" />
+			<geometry>
+				<box size="0.06 7.00 2.60" />
+			</geometry>
+		</visual>
+		<collision>
+			<origin xyz="0 0 0" />
+			<geometry>
+				<box size="0.04 6.98 2.58" />
+			</geometry>
+		</collision>
+	</link>
+	<gazebo reference="wall_07">
+		<material>IPA/Wall</material>
+	</gazebo>
+	<joint name="joint_wall_07" type="fixed">
+		<origin xyz="-3.561 1.321 1.300" rpy="0 0 0" />
+		<parent link="dummy_link" />
+		<child link="wall_07" />
+	</joint>
+<!-- wall_08 -->
+	<link name="wall_08">
+		<inertial>
+			<origin xyz="0 0 0" />
+			<mass value="5.0" />
+			<inertia  ixx="0.0" ixy="0.0"  ixz="0.0"  iyy="0.0"  iyz="0.0"  izz="0.0" />
+		</inertial>
+		<visual>
+			<origin xyz="0 0 0" />
+			<geometry>
+				<box size="1.69 0.06 2.06" />
+			</geometry>
+		</visual>
+		<collision>
+			<origin xyz="0 0 0" />
+			<geometry>
+				<box size="1.67 0.04 2.04" />
+			</geometry>
+		</collision>
+	</link>
+	<gazebo reference="wall_08">
+		<material>IPA/Wall</material>
+	</gazebo>
+	<joint name="joint_wall_08" type="fixed">
+		<origin xyz="-2.686 3.641 1.030" rpy="0 0 0" />
+		<parent link="dummy_link" />
+		<child link="wall_08" />
+	</joint>
+<!-- wall_09 -->
+	<link name="wall_09">
+		<inertial>
+			<origin xyz="0 0 0" />
+			<mass value="5.0" />
+			<inertia  ixx="0.0" ixy="0.0"  ixz="0.0"  iyy="0.0"  iyz="0.0"  izz="0.0" />
+		</inertial>
+		<visual>
+			<origin xyz="0 0 0" />
+			<geometry>
+				<box size="0.06 1.30 2.06" />
+			</geometry>
+		</visual>
+		<collision>
+			<origin xyz="0 0 0" />
+			<geometry>
+				<box size="0.04 1.28 2.04" />
+			</geometry>
+		</collision>
+	</link>
+	<gazebo reference="wall_09">
+		<material>IPA/Wall</material>
+	</gazebo>
+	<joint name="joint_wall_09" type="fixed">
+		<origin xyz="-1.811 3.021 1.030" rpy="0 0 0" />
+		<parent link="dummy_link" />
+		<child link="wall_09" />
+	</joint>
+<!-- wall_10 -->
+	<link name="wall_10">
+		<inertial>
+			<origin xyz="0 0 0" />
+			<mass value="5.0" />
+			<inertia  ixx="0.0" ixy="0.0"  ixz="0.0"  iyy="0.0"  iyz="0.0"  izz="0.0" />
+		</inertial>
+		<visual>
+			<origin xyz="0 0 0" />
+			<geometry>
+				<box size="1.75 0.10 3.20" />
+			</geometry>
+		</visual>
+		<collision>
+			<origin xyz="0 0 0" />
+			<geometry>
+				<box size="1.73 0.08 3.18" />
+			</geometry>
+		</collision>
+	</link>
+	<gazebo reference="wall_10">
+		<material>IPA/Wall</material>
+	</gazebo>
+	<joint name="joint_wall_10" type="fixed">
+		<origin xyz="-2.656 2.321 1.600" rpy="0 0 0" />
+		<parent link="dummy_link" />
+		<child link="wall_10" />
+	</joint>
+<!-- wall_11 -->
+	<link name="wall_11">
+		<inertial>
+			<origin xyz="0 0 0" />
+			<mass value="5.0" />
+			<inertia  ixx="0.0" ixy="0.0"  ixz="0.0"  iyy="0.0"  iyz="0.0"  izz="0.0" />
+		</inertial>
+		<visual>
+			<origin xyz="0 0 0" />
+			<geometry>
+				<box size="0.75 0.06 2.60" />
+			</geometry>
+		</visual>
+		<collision>
+			<origin xyz="0 0 0" />
+			<geometry>
+				<box size="0.73 0.04 2.58" />
+			</geometry>
+		</collision>
+	</link>
+	<gazebo reference="wall_11">
+		<material>IPA/Wall</material>
+	</gazebo>
+	<joint name="joint_wall_11" type="fixed">
+		<origin xyz="-1.406 2.301 1.300" rpy="0 0 0" />
+		<parent link="dummy_link" />
+		<child link="wall_11" />
+	</joint>
+<!-- wall_12 -->
+	<link name="wall_12">
+		<inertial>
+			<origin xyz="0 0 0" />
+			<mass value="5.0" />
+			<inertia  ixx="0.0" ixy="0.0"  ixz="0.0"  iyy="0.0"  iyz="0.0"  izz="0.0" />
+		</inertial>
+		<visual>
+			<origin xyz="0 0 0" />
+			<geometry>
+				<box size="0.85 0.06 0.55" />
+			</geometry>
+		</visual>
+		<collision>
+			<origin xyz="0 0 0" />
+			<geometry>
+				<box size="0.83 0.04 0.53" />
+			</geometry>
+		</collision>
+	</link>
+	<gazebo reference="wall_12">
+		<material>IPA/Wall</material>
+	</gazebo>
+	<joint name="joint_wall_12" type="fixed">
+		<origin xyz="-0.606 2.301 2.325" rpy="0 0 0" />
+		<parent link="dummy_link" />
+		<child link="wall_12" />
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
Commit message: modified ipa-kitchen.urdf.xacro

File: cob_gazebo_worlds/common/worlds/ipa-kitchen.urdf.xacro (robot description, xacro)
@@ -840,249 +840,5 @@
 	</joint>
 <!-- couch -->
-<!--
-  <link name="wall_1">
-    <inertial>
-      <origin xyz="0 0 0" />
-      <mass value="5.0" />
-      <inertia  ixx="1.0" ixy="0.0"  ixz="0.0"  iyy="5.0"  iyz="0.0"  izz="1.0" />
-    </inertial>
-    <visual>
-      <origin xyz="0 0 0" />
-      <geometry>
-        <box size="7 .02 0.5" />
-      </geometry>
-    </visual>
-    <collision>
-      <origin xyz="0 0 0" />
-      <geometry>
-        <box size="7 .02 0.5" />
-      </geometry>
-    </collision>
-  </link>
-  <gazebo reference="wall_1">
-    <material>Gazebo/Green</material>
-  </gazebo>
-  <joint name="joint_wall_1" type="fixed">
-    <origin xyz="0 -2.36 0.25" rpy="0 0 0" />
-    <parent link="dummy_link" />
-    <child link="wall_1" />
- </joint>
-  <link name="wall_2">
-    <inertial>
-      <origin xyz="0 0 0" />
-      <mass value="1.0" />
-      <inertia  ixx="1.0" ixy="0.0"  ixz="0.0"  iyy="5.0"  iyz="0.0"  izz="1.0" />
-    </inertial>
-    <visual>
-      <origin xyz="0 0 0" />
-      <geometry>
-        <box size="2.5 0.058 3" />
-      </geometry>
-    </visual>
-    <collision>
-      <origin xyz="0 0 0" />
-      <geometry>
-        <box size="2.5 0.058 3" />
-      </geometry>
-    </collision>
-  </link>
-  <gazebo reference="wall_2">
-    <material>Gazebo/Green</material>
-  </gazebo>
-   <joint name="joint_wall_2" type="fixed">
-    <origin xyz="-2.25 2.36 1.5" rpy="0 0 0" />
-    <parent link="dummy_link" />
-    <child link="wall_2" />
- </joint>
- <link name="wall_3">
-    <inertial>
-      <origin xyz="0 0 0" />
-      <mass value="1.0" />
-      <inertia  ixx="1.0" ixy="0.0"  ixz="0.0"  iyy="5.0"  iyz="0.0"  izz="1.0" />
-    </inertial>
-    <visual>
-      <origin xyz="0 0 0" />
-      <geometry>
-        <box size="0.16 0.058 2.5" />
-      </geometry>
-    </visual>
-    <collision>
-      <origin xyz="0 0 0" />
-      <geometry>
-        <box size="0.16 0.058 2.5" />
-      </geometry>
-    </collision>
-  </link>
-  <gazebo reference="wall_3">
-    <material>Gazebo/Green</material>
-  </gazebo>
-   <joint name="joint_wall_3" type="fixed">
-    <origin xyz="-0.08 2.36 1.25" rpy="0 0 0" />
-    <parent link="dummy_link" />
-    <child link="wall_3" />
- </joint>
-  <link name="wall_4">
-    <inertial>
-      <origin xyz="0 0 0" />
-      <mass value="1.0" />
-      <inertia  ixx="1.0" ixy="0.0"  ixz="0.0"  iyy="5.0"  iyz="0.0"  izz="1.0" />
-    </inertial>
-    <visual>
-      <origin xyz="0 0 0" />
-      <geometry>
-        <box size="0.058 0.66 2.5" />
-      </geometry>
-    </visual>
-    <collision>
-      <origin xyz="0 0 0" />
-      <geometry>
-        <box size="0.058 0.66 2.5" />
-      </geometry>
-    </collision>
-  </link>
-  <gazebo reference="wall_4">
-    <material>Gazebo/Green</material>
-  </gazebo>
-   <joint name="joint_wall_4" type="fixed">
-    <origin xyz="0 2.03 1.25" rpy="0 0 0" />
-    <parent link="dummy_link" />
-    <child link="wall_4" />
- </joint>
- <link name="wall_5">
-    <inertial>
-      <origin xyz="0 0 0" />
-      <mass value="1.0" />
-      <inertia  ixx="1.0" ixy="0.0"  ixz="0.0"  iyy="5.0"  iyz="0.0"  izz="1.0" />
-    </inertial>
-    <visual>
-      <origin xyz="0 0 0" />
-      <geometry>
-        <box size="1.75 0.058 2.5" />
-      </geometry>
-    </visual>
-    <collision>
-      <origin xyz="0 0 0" />
-      <geometry>
-        <box size="1.75 0.058 2.5" />
-      </geometry>
-    </collision>
-  </link>
-  <gazebo reference="wall_5">
-    <material>Gazebo/Green</material>
-  </gazebo>
-   <joint name="joint_wall_5" type="fixed">
-    <origin xyz="0.875 1.7 1.25" rpy="0 0 0" />
-    <parent link="dummy_link" />
-    <child link="wall_5" />
- </joint>
- <link name="wall_6">
-    <inertial>
-      <origin xyz="0 0 0" />
-      <mass value="1.0" />
-      <inertia  ixx="1.0" ixy="0.0"  ixz="0.0"  iyy="5.0"  iyz="0.0"  izz="1.0" />
-    </inertial>
-    <visual>
-      <origin xyz="0 0 0" />
-      <geometry>
-        <box size="0.058 0.66 2.5" />
-      </geometry>
-    </visual>
-    <collision>
-      <origin xyz="0 0 0" />
-      <geometry>
-        <box size="0.058 0.66 2.5" />
-      </geometry>
-    </collision>
-  </link>
-  <gazebo reference="wall_6">
-    <material>Gazebo/Green</material>
-  </gazebo>
-   <joint name="joint_wall_6" type="fixed">
-    <origin xyz="1.75 1.37 1.25" rpy="0 0 0" />
-    <parent link="dummy_link" />
-    <child link="wall_6" />
- </joint>
-  <link name="wall_7">
-    <inertial>
-      <origin xyz="0 0 0" />
-      <mass value="1.0" />
-      <inertia  ixx="1.0" ixy="0.0"  ixz="0.0"  iyy="5.0"  iyz="0.0"  izz="1.0" />
-    </inertial>
-    <visual>
-      <origin xyz="0 0 0" />
-      <geometry>
-        <box size="1.75 0.058 2.5" />
-      </geometry>
-    </visual>
-    <collision>
-      <origin xyz="0 0 0" />
-      <geometry>
-        <box size="1.75 0.058 2.5" />
-      </geometry>
-    </collision>
-  </link>
-  <gazebo reference="wall_7">
-    <material>Gazebo/Green</material>
-  </gazebo>
-   <joint name="joint_wall_7" type="fixed">
-    <origin xyz="2.625 1.04 1.25" rpy="0 0 0" />
-    <parent link="dummy_link" />
-    <child link="wall_7" />
- </joint>
-  <link name="wall_8">
-    <inertial>
-      <origin xyz="0 0 0" />
-      <mass value="1.0" />
-      <inertia  ixx="1.0" ixy="0.0"  ixz="0.0"  iyy="5.0"  iyz="0.0"  izz="1.0" />
-    </inertial>
-    <visual>
-      <origin xyz="0 0 0" />
-      <geometry>
-        <box size="0.02 3.4 0.5" />
-      </geometry>
-    </visual>
-    <collision>
-      <origin xyz="0 0 0" />
-      <geometry>
-        <box size="0.02 3.4 0.5" />
-      </geometry>
-    </collision>
-  </link>
-  <gazebo reference="wall_8">
-    <material>Gazebo/Green</material>
-  </gazebo>
-   <joint name="joint_wall_8" type="fixed">
-    <origin xyz="3.5 -0.66 0.25" rpy="0 0 0" />
-    <parent link="dummy_link" />
-    <child link="wall_8" />
- </joint>
- <link name="wall_9">
-    <inertial>
-      <origin xyz="0 0 0" />
-      <mass value="1.0" />
-      <inertia  ixx="1.0" ixy="0.0"  ixz="0.0"  iyy="5.0"  iyz="0.0"  izz="1.0" />
-    </inertial>
-    <visual>
-      <origin xyz="0 0 0" />
-      <geometry>
-        <box size="0.058 4.72 2.5" />
-      </geometry>
-    </visual>
-    <collision>
-      <origin xyz="0 0 0" />
-      <geometry>
-        <box size="0.058 4.72 2.5" />
-      </geometry>
-    </collision>
-  </link>
-  <gazebo reference="wall_9">
-    <material>Gazebo/Green</material>
-  </gazebo>
-   <joint name="joint_wall_9" type="fixed">
-    <origin xyz="-3.5 0 1.25" rpy="0 0 0" />
-    <parent link="dummy_link" />
-    <child link="wall_9" />
- </joint>
--->
+<!-- will be add soon -->
 </xacro:macro>
 <xacro:ipa-kitchen name="ipa-kitchen" />
