Commit message: added cabinet and couch

File: cob_gazebo_worlds/common/worlds/ipa-kitchen.urdf.xacro (robot description, xacro)
@@ -13,5 +13,5 @@
 			<origin xyz="0 0 0" />
 			<mass value="5.0" />
-			<inertia  ixx="0.0" ixy="0.0"  ixz="0.0"  iyy="0.0"  iyz="0.0"  izz="0.0" />
+			<inertia ixx="0.0" ixy="0.0" ixz="0.0" iyy="0.0" iyz="0.0" izz="0.0" />
 		</inertial>
 		<visual>
@@ -29,10 +29,10 @@
 	</link>
 <!-- walls -->
-<!-- wall_00 -->
+	<!-- wall_00 -->
 	<link name="wall_00">
 		<inertial>
 			<origin xyz="0 0 0" />
 			<mass value="5.0" />
-			<inertia  ixx="0.0" ixy="0.0"  ixz="0.0"  iyy="0.0"  iyz="0.0"  izz="0.0" />
+			<inertia ixx="0.0" ixy="0.0" ixz="0.0" iyy="0.0" iyz="0.0" izz="0.0" />
 		</inertial>
 		<visual>
@@ -45,5 +45,5 @@
 			<origin xyz="0 0 0" />
 			<geometry>
-				<box size="2.73 0.04 0.48" />
+				<box size="2.77 0.08 0.52" />
 			</geometry>
 		</collision>
@@ -57,10 +57,10 @@
 		<child link="wall_00" />
 	</joint>
-<!-- wall_01 -->
+	<!-- wall_01 -->
 	<link name="wall_01">
 		<inertial>
 			<origin xyz="0 0 0" />
 			<mass value="5.0" />
-			<inertia  ixx="0.0" ixy="0.0"  ixz="0.0"  iyy="0.0"  iyz="0.0"  izz="0.0" />
+			<inertia ixx="0.0" ixy="0.0" ixz="0.0" iyy="0.0" iyz="0.0" izz="0.0" />
 		</inertial>
 		<visual>
@@ -73,5 +73,5 @@
 			<origin xyz="0 0 0" />
 			<geometry>
-				<box size="0.08 0.78 2.38" />
+				<box size="0.12 0.82 2.42" />
 			</geometry>
 		</collision>
@@ -85,10 +85,10 @@
 		<child link="wall_01" />
 	</joint>
-<!-- wall_02 -->
+	<!-- wall_02 -->
 	<link name="wall_02">
 		<inertial>
 			<origin xyz="0 0 0" />
 			<mass value="5.0" />
-			<inertia  ixx="0.0" ixy="0.0"  ixz="0.0"  iyy="0.0"  iyz="0.0"  izz="0.0" />
+			<inertia ixx="0.0" ixy="0.0" ixz="0.0" iyy="0.0" iyz="0.0" izz="0.0" />
 		</inertial>
 		<visual>
@@ -101,5 +101,5 @@
 			<origin xyz="0 0 0" />
 			<geometry>
-				<box size="3.27 0.04 0.48" />
+				<box size="3.31 0.08 0.52" />
 			</geometry>
 		</collision>
@@ -113,10 +113,10 @@
 		<child link="wall_02" />
 	</joint>
-<!-- wall_03 -->
+	<!-- wall_03 -->
 	<link name="wall_03">
 		<inertial>
 			<origin xyz="0 0 0" />
 			<mass value="5.0" />
-			<inertia  ixx="0.0" ixy="0.0"  ixz="0.0"  iyy="0.0"  iyz="0.0"  izz="0.0" />
+			<inertia ixx="0.0" ixy="0.0" ixz="0.0" iyy="0.0" iyz="0.0" izz="0.0" />
 		</inertial>
 		<visual>
@@ -129,5 +129,5 @@
 			<origin xyz="0 0 0" />
 			<geometry>
-				<box size="0.78 0.08 3.18" />
+				<box size="0.82 0.12 3.22" />
 			</geometry>
 		</collision>
@@ -141,10 +141,10 @@
 		<child link="wall_03" />
 	</joint>
-<!-- wall_04 -->
+	<!-- wall_04 -->
 	<link name="wall_04">
 		<inertial>
 			<origin xyz="0 0 0" />
 			<mass value="5.0" />
-			<inertia  ixx="0.0" ixy="0.0"  ixz="0.0"  iyy="0.0"  iyz="0.0"  izz="0.0" />
+			<inertia ixx="0.0" ixy="0.0" ixz="0.0" iyy="0.0" iyz="0.0" izz="0.0" />
 		</inertial>
 		<visual>
@@ -157,5 +157,5 @@
 			<origin xyz="0 0 0" />
 			<geometry>
-				<box size="0.04 6.78 0.48" />
+				<box size="0.08 6.82 0.52" />
 			</geometry>
 		</collision>
@@ -169,10 +169,10 @@
 		<child link="wall_04" />
 	</joint>
-<!-- wall_05 -->
+	<!-- wall_05 -->
 	<link name="wall_05">
 		<inertial>
 			<origin xyz="0 0 0" />
 			<mass value="5.0" />
-			<inertia  ixx="0.0" ixy="0.0"  ixz="0.0"  iyy="0.0"  iyz="0.0"  izz="0.0" />
+			<inertia ixx="0.0" ixy="0.0" ixz="0.0" iyy="0.0" iyz="0.0" izz="0.0" />
 		</inertial>
 		<visual>
@@ -185,5 +185,5 @@
 			<origin xyz="0 0 0" />
 			<geometry>
-				<box size="0.78 0.08 3.18" />
+				<box size="0.82 0.12 3.22" />
 			</geometry>
 		</collision>
@@ -197,10 +197,10 @@
 		<child link="wall_05" />
 	</joint>
-<!-- wall_06 -->
+	<!-- wall_06 -->
 	<link name="wall_06">
 		<inertial>
 			<origin xyz="0 0 0" />
 			<mass value="5.0" />
-			<inertia  ixx="0.0" ixy="0.0"  ixz="0.0"  iyy="0.0"  iyz="0.0"  izz="0.0" />
+			<inertia ixx="0.0" ixy="0.0" ixz="0.0" iyy="0.0" iyz="0.0" izz="0.0" />
 		</inertial>
 		<visual>
@@ -213,5 +213,5 @@
 			<origin xyz="0 0 0" />
 			<geometry>
-				<box size="6.12 0.04 0.48" />
+				<box size="6.16 0.08 0.52" />
 			</geometry>
 		</collision>
@@ -225,10 +225,10 @@
 		<child link="wall_06" />
 	</joint>
-<!-- wall_07 -->
+	<!-- wall_07 -->
 	<link name="wall_07">
 		<inertial>
 			<origin xyz="0 0 0" />
 			<mass value="5.0" />
-			<inertia  ixx="0.0" ixy="0.0"  ixz="0.0"  iyy="0.0"  iyz="0.0"  izz="0.0" />
+			<inertia ixx="0.0" ixy="0.0" ixz="0.0" iyy="0.0" iyz="0.0" izz="0.0" />
 		</inertial>
 		<visual>
@@ -241,5 +241,5 @@
 			<origin xyz="0 0 0" />
 			<geometry>
-				<box size="0.04 6.98 2.58" />
+				<box size="0.08 7.02 2.62" />
 			</geometry>
 		</collision>
@@ -253,10 +253,10 @@
 		<child link="wall_07" />
 	</joint>
-<!-- wall_08 -->
+	<!-- wall_08 -->
 	<link name="wall_08">
 		<inertial>
 			<origin xyz="0 0 0" />
 			<mass value="5.0" />
-			<inertia  ixx="0.0" ixy="0.0"  ixz="0.0"  iyy="0.0"  iyz="0.0"  izz="0.0" />
+			<inertia ixx="0.0" ixy="0.0" ixz="0.0" iyy="0.0" iyz="0.0" izz="0.0" />
 		</inertial>
 		<visual>
@@ -269,5 +269,5 @@
 			<origin xyz="0 0 0" />
 			<geometry>
-				<box size="1.67 0.04 2.04" />
+				<box size="1.71 0.08 2.08" />
 			</geometry>
 		</collision>
@@ -281,10 +281,10 @@
 		<child link="wall_08" />
 	</joint>
-<!-- wall_09 -->
+	<!-- wall_09 -->
 	<link name="wall_09">
 		<inertial>
 			<origin xyz="0 0 0" />
 			<mass value="5.0" />
-			<inertia  ixx="0.0" ixy="0.0"  ixz="0.0"  iyy="0.0"  iyz="0.0"  izz="0.0" />
+			<inertia ixx="0.0" ixy="0.0" ixz="0.0" iyy="0.0" iyz="0.0" izz="0.0" />
 		</inertial>
 		<visual>
@@ -297,5 +297,5 @@
 			<origin xyz="0 0 0" />
 			<geometry>
-				<box size="0.04 1.28 2.04" />
+				<box size="0.08 1.32 2.08" />
 			</geometry>
 		</collision>
@@ -309,10 +309,10 @@
 		<child link="wall_09" />
 	</joint>
-<!-- wall_10 -->
+	<!-- wall_10 -->
 	<link name="wall_10">
 		<inertial>
 			<origin xyz="0 0 0" />
 			<mass value="5.0" />
-			<inertia  ixx="0.0" ixy="0.0"  ixz="0.0"  iyy="0.0"  iyz="0.0"  izz="0.0" />
+			<inertia ixx="0.0" ixy="0.0" ixz="0.0" iyy="0.0" iyz="0.0" izz="0.0" />
 		</inertial>
 		<visual>
@@ -325,5 +325,5 @@
 			<origin xyz="0 0 0" />
 			<geometry>
-				<box size="1.73 0.08 3.18" />
+				<box size="1.77 0.08 3.22" />
 			</geometry>
 		</collision>
@@ -337,10 +337,10 @@
 		<child link="wall_10" />
 	</joint>
-<!-- wall_11 -->
+	<!-- wall_11 -->
 	<link name="wall_11">
 		<inertial>
 			<origin xyz="0 0 0" />
 			<mass value="5.0" />
-			<inertia  ixx="0.0" ixy="0.0"  ixz="0.0"  iyy="0.0"  iyz="0.0"  izz="0.0" />
+			<inertia ixx="0.0" ixy="0.0" ixz="0.0" iyy="0.0" iyz="0.0" izz="0.0" />
 		</inertial>
 		<visual>
@@ -353,5 +353,5 @@
 			<origin xyz="0 0 0" />
 			<geometry>
-				<box size="0.73 0.04 2.58" />
+				<box size="0.77 0.08 2.62" />
 			</geometry>
 		</collision>
@@ -365,10 +365,10 @@
 		<child link="wall_11" />
 	</joint>
-<!-- wall_12 -->
+	<!-- wall_12 -->
 	<link name="wall_12">
 		<inertial>
 			<origin xyz="0 0 0" />
 			<mass value="5.0" />
-			<inertia  ixx="0.0" ixy="0.0"  ixz="0.0"  iyy="0.0"  iyz="0.0"  izz="0.0" />
+			<inertia ixx="0.0" ixy="0.0" ixz="0.0" iyy="0.0" iyz="0.0" izz="0.0" />
 		</inertial>
 		<visual>
@@ -381,5 +381,5 @@
 			<origin xyz="0 0 0" />
 			<geometry>
-				<box size="0.83 0.04 0.53" />
+				<box size="0.87 0.08 0.57" />
 			</geometry>
 		</collision>
@@ -393,10 +393,10 @@
 		<child link="wall_12" />
 	</joint>
-<!-- wall_13 -->
+	<!-- wall_13 -->
 	<link name="wall_13">
 		<inertial>
 			<origin xyz="0 0 0" />
 			<mass value="5.0" />
-			<inertia  ixx="0.0" ixy="0.0"  ixz="0.0"  iyy="0.0"  iyz="0.0"  izz="0.0" />
+			<inertia ixx="0.0" ixy="0.0" ixz="0.0" iyy="0.0" iyz="0.0" izz="0.0" />
 		</inertial>
 		<visual>
@@ -409,5 +409,5 @@
 			<origin xyz="0 0 0" />
 			<geometry>
-				<box size="0.13 0.04 2.58" />
+				<box size="0.17 0.08 2.62" />
 			</geometry>
 		</collision>
@@ -421,10 +421,10 @@
 		<child link="wall_13" />
 	</joint>
-<!-- wall_14 -->
+	<!-- wall_14 -->
 	<link name="wall_14">
 		<inertial>
 			<origin xyz="0 0 0" />
 			<mass value="5.0" />
-			<inertia  ixx="0.0" ixy="0.0"  ixz="0.0"  iyy="0.0"  iyz="0.0"  izz="0.0" />
+			<inertia ixx="0.0" ixy="0.0" ixz="0.0" iyy="0.0" iyz="0.0" izz="0.0" />
 		</inertial>
 		<visual>
@@ -437,5 +437,5 @@
 			<origin xyz="0 0 0" />
 			<geometry>
-				<box size="0.04 0.52 0.73" />
+				<box size="0.08 0.56 0.77" />
 			</geometry>
 		</collision>
@@ -449,10 +449,10 @@
 		<child link="wall_14" />
 	</joint>
-<!-- wall_15 -->
+	<!-- wall_15 -->
 	<link name="wall_15">
 		<inertial>
 			<origin xyz="0 0 0" />
 			<mass value="5.0" />
-			<inertia  ixx="0.0" ixy="0.0"  ixz="0.0"  iyy="0.0"  iyz="0.0"  izz="0.0" />
+			<inertia ixx="0.0" ixy="0.0" ixz="0.0" iyy="0.0" iyz="0.0" izz="0.0" />
 		</inertial>
 		<visual>
@@ -465,5 +465,5 @@
 			<origin xyz="0 0 0" />
 			<geometry>
-				<box size="0.04 0.52 0.53" />
+				<box size="0.08 0.56 0.57" />
 			</geometry>
 		</collision>
@@ -477,10 +477,10 @@
 		<child link="wall_15" />
 	</joint>
-<!-- wall_16 -->
+	<!-- wall_16 -->
 	<link name="wall_16">
 		<inertial>
 			<origin xyz="0 0 0" />
 			<mass value="5.0" />
-			<inertia  ixx="0.0" ixy="0.0"  ixz="0.0"  iyy="0.0"  iyz="0.0"  izz="0.0" />
+			<inertia ixx="0.0" ixy="0.0" ixz="0.0" iyy="0.0" iyz="0.0" izz="0.0" />
 		</inertial>
 		<visual>
@@ -493,5 +493,5 @@
 			<origin xyz="0 0 0" />
 			<geometry>
-				<box size="0.04 0.04 2.58" />
+				<box size="0.08 0.08 2.62" />
 			</geometry>
 		</collision>
@@ -505,10 +505,10 @@
 		<child link="wall_16" />
 	</joint>
-<!-- wall_17 -->
+	<!-- wall_17 -->
 	<link name="wall_17">
 		<inertial>
 			<origin xyz="0 0 0" />
 			<mass value="5.0" />
-			<inertia  ixx="0.0" ixy="0.0"  ixz="0.0"  iyy="0.0"  iyz="0.0"  izz="0.0" />
+			<inertia ixx="0.0" ixy="0.0" ixz="0.0" iyy="0.0" iyz="0.0" izz="0.0" />
 		</inertial>
 		<visual>
@@ -521,5 +521,5 @@
 			<origin xyz="0 0 0" />
 			<geometry>
-				<box size="1.61 0.04 0.73" />
+				<box size="1.65 0.08 0.77" />
 			</geometry>
 		</collision>
@@ -533,10 +533,10 @@
 		<child link="wall_17" />
 	</joint>
-<!-- wall_18 -->
+	<!-- wall_18 -->
 	<link name="wall_18">
 		<inertial>
 			<origin xyz="0 0 0" />
 			<mass value="5.0" />
-			<inertia  ixx="0.0" ixy="0.0"  ixz="0.0"  iyy="0.0"  iyz="0.0"  izz="0.0" />
+			<inertia ixx="0.0" ixy="0.0" ixz="0.0" iyy="0.0" iyz="0.0" izz="0.0" />
 		</inertial>
 		<visual>
@@ -549,5 +549,5 @@
 			<origin xyz="0 0 0" />
 			<geometry>
-				<box size="1.61 0.04 0.53" />
+				<box size="1.65 0.08 0.57" />
 			</geometry>
 		</collision>
@@ -561,10 +561,10 @@
 		<child link="wall_18" />
 	</joint>
-<!-- wall_19 -->
+	<!-- wall_19 -->
 	<link name="wall_19">
 		<inertial>
 			<origin xyz="0 0 0" />
 			<mass value="5.0" />
-			<inertia  ixx="0.0" ixy="0.0"  ixz="0.0"  iyy="0.0"  iyz="0.0"  izz="0.0" />
+			<inertia ixx="0.0" ixy="0.0" ixz="0.0" iyy="0.0" iyz="0.0" izz="0.0" />
 		</inertial>
 		<visual>
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
Commit message: modifications to world

File: cob_gazebo_worlds/common/worlds/ipa-kitchen.urdf.xacro (robot description, xacro)
@@ -78,5 +78,5 @@
 	</link>
 	<gazebo reference="wall_01">
-		<material>IPA/Wall</material>
+		<material>IPA/Wall3</material>
 	</gazebo>
 	<joint name="joint_wall_01" type="fixed">
@@ -1311,4 +1311,145 @@
 		<child link="cabinet_back_left" />
 	</joint>
+<!-- pictures -->
+	<!-- picture_00 -->
+	<link name="picture_00">
+		<inertial>
+			<origin xyz="0 0 0" />
+			<mass value="5.0" />
+			<inertia ixx="0.0" ixy="0.0" ixz="0.0" iyy="0.0" iyz="0.0" izz="0.0" />
+		</inertial>
+		<visual>
+			<origin xyz="0 0 0" />
+			<geometry>
+				<box size="0.56 0.02 0.40" />
+			</geometry>
+		</visual>
+		<collision>
+			<origin xyz="0 0 0" />
+			<geometry>
+				<box size="0.56 0.02 0.40" />
+			</geometry>
+		</collision>
+	</link>
+	<gazebo reference="picture_00">
+		<material>IPA/Comic</material>
+	</gazebo>
+	<joint name="joint_picture_00" type="fixed">
+		<origin xyz="3.009 -2.189 1.450" rpy="0 0 0" />
+		<parent link="dummy_link" />
+		<child link="picture_00" />
+	</joint>
+	<!-- picture_01 -->
+	<link name="picture_01">
+		<inertial>
+			<origin xyz="0 0 0" />
+			<mass value="5.0" />
+			<inertia ixx="0.0" ixy="0.0" ixz="0.0" iyy="0.0" iyz="0.0" izz="0.0" />
+		</inertial>
+		<visual>
+			<origin xyz="0 0 0" />
+			<geometry>
+				<box size="0.02 0.44 0.56" />
+			</geometry>
+		</visual>
+		<collision>
+			<origin xyz="0 0 0" />
+			<geometry>
+				<box size="0.02 0.44 0.56" />
+			</geometry>
+		</collision>
+	</link>
+	<gazebo reference="picture_01">
+		<material>IPA/Care-O-bot</material>
+	</gazebo>
+	<joint name="joint_picture_01" type="fixed">
+		<origin xyz="-3.521 4.451 2.200" rpy="0 0 0" />
+		<parent link="dummy_link" />
+		<child link="picture_01" />
+	</joint>
+	<!-- picture_02 -->
+	<link name="picture_02">
+		<inertial>
+			<origin xyz="0 0 0" />
+			<mass value="5.0" />
+			<inertia ixx="0.0" ixy="0.0" ixz="0.0" iyy="0.0" iyz="0.0" izz="0.0" />
+		</inertial>
+		<visual>
+			<origin xyz="0 0 0" />
+			<geometry>
+				<box size="0.02 2.33 0.64" />
+			</geometry>
+		</visual>
+		<collision>
+			<origin xyz="0 0 0" />
+			<geometry>
+				<box size="0.02 2.33 0.64" />
+			</geometry>
+		</collision>
+	</link>
+	<gazebo reference="picture_02">
+		<material>IPA/FraunhoferIPA</material>
+	</gazebo>
+	<joint name="joint_picture_02" type="fixed">
+		<origin xyz="-3.521 0.055 2.200" rpy="0 0 0" />
+		<parent link="dummy_link" />
+		<child link="picture_02" />
+	</joint>
+	<!-- picture_03 -->
+	<link name="picture_03">
+		<inertial>
+			<origin xyz="0 0 0" />
+			<mass value="5.0" />
+			<inertia ixx="0.0" ixy="0.0" ixz="0.0" iyy="0.0" iyz="0.0" izz="0.0" />
+		</inertial>
+		<visual>
+			<origin xyz="0 0 0" />
+			<geometry>
+				<box size="1.35 0.02 0.62" />
+			</geometry>
+		</visual>
+		<collision>
+			<origin xyz="0 0 0" />
+			<geometry>
+				<box size="1.35 0.02 0.62" />
+			</geometry>
+		</collision>
+	</link>
+	<gazebo reference="picture_03">
+		<material>IPA/Future</material>
+	</gazebo>
+	<joint name="joint_picture_03" type="fixed">
+		<origin xyz="-2.000 2.261 2.050" rpy="0 0 0" />
+		<parent link="dummy_link" />
+		<child link="picture_03" />
+	</joint>
+	<!-- picture_04 -->
+	<link name="picture_04">
+		<inertial>
+			<origin xyz="0 0 0" />
+			<mass value="5.0" />
+			<inertia ixx="0.0" ixy="0.0" ixz="0.0" iyy="0.0" iyz="0.0" izz="0.0" />
+		</inertial>
+		<visual>
+			<origin xyz="0 0 0" />
+			<geometry>
+				<box size="0.02 0.44 0.26" />
+			</geometry>
+		</visual>
+		<collision>
+			<origin xyz="0 0 0" />
+			<geometry>
+				<box size="0.02 0.44 0.26" />
+			</geometry>
+		</collision>
+	</link>
+	<gazebo reference="picture_04">
+		<material>IPA/Brics</material>
+	</gazebo>
+	<joint name="joint_picture_04" type="fixed">
+		<origin xyz="-1.771 3.301 1.770" rpy="0 0 0" />
+		<parent link="dummy_link" />
+		<child link="picture_04" />
+	</joint>
 </xacro:macro>
 <xacro:ipa-kitchen name="ipa-kitchen" />
