Commit message: modified ipa-kitchen and created seperate table

File: cob_gazebo_worlds/common/worlds/ipa-kitchen.urdf.xacro (robot description, xacro)
@@ -18,11 +18,11 @@
 			<origin xyz="0 0 0" />
 			<geometry>
-				<box size="0.01 0.01 0.01" />
-			</geometry>
-		</visual>
-		<collision>
-			<origin xyz="0 0 0" />
-			<geometry>
-				<box size="0.01 0.01 0.01" />
+				<box size="0.00 0.00 0.00" />
+			</geometry>
+		</visual>
+		<collision>
+			<origin xyz="0 0 0" />
+			<geometry>
+				<box size="0.00 0.00 0.00" />
 			</geometry>
 		</collision>
@@ -151,11 +151,11 @@
 			<origin xyz="0 0 0" />
 			<geometry>
-				<box size="0.06 6.80 0.50" />
-			</geometry>
-		</visual>
-		<collision>
-			<origin xyz="0 0 0" />
-			<geometry>
-				<box size="0.08 6.82 0.52" />
+				<box size="0.06 6.90 0.50" />
+			</geometry>
+		</visual>
+		<collision>
+			<origin xyz="0 0 0" />
+			<geometry>
+				<box size="0.08 6.92 0.52" />
 			</geometry>
 		</collision>
@@ -165,35 +165,7 @@
 	</gazebo>
 	<joint name="joint_wall_04" type="fixed">
-		<origin xyz="3.379 1.321 0.250" rpy="0 0 0" />
+		<origin xyz="3.379 1.271 0.250" rpy="0 0 0" />
 		<parent link="dummy_link" />
 		<child link="wall_04" />
-	</joint>
-	<!-- wall_05 -->
-	<link name="wall_05">
-		<inertial>
-			<origin xyz="0 0 0" />
-			<mass value="5.0" />
-			<inertia ixx="0.0" ixy="0.0" ixz="0.0" iyy="0.0" iyz="0.0" izz="0.0" />
-		</inertial>
-		<visual>
-			<origin xyz="0 0 0" />
-			<geometry>
-				<box size="0.80 0.10 3.20" />
-			</geometry>
-		</visual>
-		<collision>
-			<origin xyz="0 0 0" />
-			<geometry>
-				<box size="0.82 0.12 3.22" />
-			</geometry>
-		</collision>
-	</link>
-	<gazebo reference="wall_05">
-		<material>IPA/Wall</material>
-	</gazebo>
-	<joint name="joint_wall_05" type="fixed">
-		<origin xyz="3.009 -2.129 1.600" rpy="0 0 0" />
-		<parent link="dummy_link" />
-		<child link="wall_05" />
 	</joint>
 	<!-- wall_06 -->
@@ -207,11 +179,11 @@
 			<origin xyz="0 0 0" />
 			<geometry>
-				<box size="6.14 0.06 0.50" />
-			</geometry>
-		</visual>
-		<collision>
-			<origin xyz="0 0 0" />
-			<geometry>
-				<box size="6.16 0.08 0.52" />
+				<box size="6.88 0.06 0.50" />
+			</geometry>
+		</visual>
+		<collision>
+			<origin xyz="0 0 0" />
+			<geometry>
+				<box size="6.90 0.08 0.52" />
 			</geometry>
 		</collision>
@@ -221,5 +193,5 @@
 	</gazebo>
 	<joint name="joint_wall_06" type="fixed">
-		<origin xyz="-0.461 -2.149 0.250" rpy="0 0 0" />
+		<origin xyz="-0.091 -2.149 0.250" rpy="0 0 0" />
 		<parent link="dummy_link" />
 		<child link="wall_06" />
@@ -1002,313 +974,4 @@
 		<child link="right_couch_middle" />
 	</joint>
-<!-- cabinet -->
-	<!-- cabinet_top -->
-	<link name="cabinet_top">
-		<inertial>
-			<origin xyz="0 0 0" />
-			<mass value="5.0" />
-			<inertia ixx="0.0" ixy="0.0" ixz="0.0" iyy="0.0" iyz="0.0" izz="0.0" />
-		</inertial>
-		<visual>
-			<origin xyz="0 0 0" />
-			<geometry>
-				<box size="0.78 0.41 0.02" />
-			</geometry>
-		</visual>
-		<collision>
-			<origin xyz="0 0 0" />
-			<geometry>
-				<box size="0.78 0.41 0.02" />
-			</geometry>
-		</collision>
-	</link>
-	<gazebo reference="cabinet_top">
-		<material>IPA/Cabinet_Wood</material>
-	</gazebo>
-	<joint name="joint_cabinet_top" type="fixed">
-		<origin xyz="1.159 1.416 0.850" rpy="0 0 0" />
-		<parent link="dummy_link" />
-		<child link="cabinet_top" />
-	</joint>
-	<!-- cabinet_middle1 -->
-	<link name="cabinet_middle1">
-		<inertial>
-			<origin xyz="0 0 0" />
-			<mass value="5.0" />
-			<inertia ixx="0.0" ixy="0.0" ixz="0.0" iyy="0.0" iyz="0.0" izz="0.0" />
-		</inertial>
-		<visual>
-			<origin xyz="0 0 0" />
-			<geometry>
-				<box size="0.62 0.37 0.01" />
-			</geometry>
-		</visual>
-		<collision>
-			<origin xyz="0 0 0" />
-			<geometry>
-				<box size="0.62 0.37 0.01" />
-			</geometry>
-		</collision>
-	</link>
-	<gazebo reference="cabinet_middle1">
-		<material>IPA/Cabinet_Wood</material>
-	</gazebo>
-	<joint name="joint_cabinet_middle1" type="fixed">
-		<origin xyz="1.159 1.416 0.585" rpy="0 0 0" />
-		<parent link="dummy_link" />
-		<child link="cabinet_middle1" />
-	</joint>
-	<!-- cabinet_middle2 -->
-	<link name="cabinet_middle2">
-		<inertial>
-			<origin xyz="0 0 0" />
-			<mass value="5.0" />
-			<inertia ixx="0.0" ixy="0.0" ixz="0.0" iyy="0.0" iyz="0.0" izz="0.0" />
-		</inertial>
-		<visual>
-			<origin xyz="0 0 0" />
-			<geometry>
-				<box size="0.62 0.37 0.01" />
-			</geometry>
-		</visual>
-		<collision>
-			<origin xyz="0 0 0" />
-			<geometry>
-				<box size="0.62 0.37 0.01" />
-			</geometry>
-		</collision>
-	</link>
-	<gazebo reference="cabinet_middle2">
-		<material>IPA/Cabinet_Wood</material>
-	</gazebo>
-	<joint name="joint_cabinet_middle2" type="fixed">
-		<origin xyz="1.159 1.416 0.375" rpy="0 0 0" />
-		<parent link="dummy_link" />
-		<child link="cabinet_middle2" />
-	</joint>
-	<!-- cabinet_bottom -->
-	<link name="cabinet_bottom">
-		<inertial>
-			<origin xyz="0 0 0" />
-			<mass value="5.0" />
-			<inertia ixx="0.0" ixy="0.0" ixz="0.0" iyy="0.0" iyz="0.0" izz="0.0" />
-		</inertial>
-		<visual>
-			<origin xyz="0 0 0" />
-			<geometry>
-				<box size="0.62 0.37 0.05" />
-			</geometry>
-		</visual>
-		<collision>
-			<origin xyz="0 0 0" />
-			<geometry>
-				<box size="0.62 0.37 0.05" />
-			</geometry>
-		</collision>
-	</link>
-	<gazebo reference="cabinet_bottom">
-		<material>IPA/Cabinet_Wood</material>
-	</gazebo>
-	<joint name="joint_cabinet_bottom" type="fixed">
-		<origin xyz="1.159 1.416 0.175" rpy="0 0 0" />
-		<parent link="dummy_link" />
-		<child link="cabinet_bottom" />
-	</joint>
-	<!-- cabinet_back -->
-	<link name="cabinet_back">
-		<inertial>
-			<origin xyz="0 0 0" />
-			<mass value="5.0" />
-			<inertia ixx="0.0" ixy="0.0" ixz="0.0" iyy="0.0" iyz="0.0" izz="0.0" />
-		</inertial>
-		<visual>
-			<origin xyz="0 0 0" />
-			<geometry>
-				<box size="0.62 0.02 0.69" />
-			</geometry>
-		</visual>
-		<collision>
-			<origin xyz="0 0 0" />
-			<geometry>
-				<box size="0.62 0.02 0.69" />
-			</geometry>
-		</collision>
-	</link>
-	<gazebo reference="cabinet_back">
-		<material>Gazebo/Grey</material>
-	</gazebo>
-	<joint name="joint_cabinet_back" type="fixed">
-		<origin xyz="1.159 1.611 0.495" rpy="0 0 0" />
-		<parent link="dummy_link" />
-		<child link="cabinet_back" />
-	</joint>
-	<!-- cabinet_right -->
-	<link name="cabinet_right">
-		<inertial>
-			<origin xyz="0 0 0" />
-			<mass value="5.0" />
-			<inertia ixx="0.0" ixy="0.0" ixz="0.0" iyy="0.0" iyz="0.0" izz="0.0" />
-		</inertial>
-		<visual>
-			<origin xyz="0 0 0" />
-			<geometry>
-				<box size="0.02 0.29 0.69" />
-			</geometry>
-		</visual>
-		<collision>
-			<origin xyz="0 0 0" />
-			<geometry>
-				<box size="0.02 0.29 0.69" />
-			</geometry>
-		</collision>
-	</link>
-	<gazebo reference="cabinet_right">
-		<material>Gazebo/Grey</material>
-	</gazebo>
-	<joint name="joint_cabinet_right" type="fixed">
-		<origin xyz="1.479 1.436 0.495" rpy="0 0 0" />
-		<parent link="dummy_link" />
-		<child link="cabinet_right" />
-	</joint>
-	<!-- cabinet_left -->
-	<link name="cabinet_left">
-		<inertial>
-			<origin xyz="0 0 0" />
-			<mass value="5.0" />
-			<inertia ixx="0.0" ixy="0.0" ixz="0.0" iyy="0.0" iyz="0.0" izz="0.0" />
-		</inertial>
-		<visual>
-			<origin xyz="0 0 0" />
-			<geometry>
-				<box size="0.02 0.29 0.69" />
-			</geometry>
-		</visual>
-		<collision>
-			<origin xyz="0 0 0" />
-			<geometry>
-				<box size="0.02 0.29 0.69" />
-			</geometry>
-		</collision>
-	</link>
-	<gazebo reference="cabinet_left">
-		<material>Gazebo/Grey</material>
-	</gazebo>
-	<joint name="joint_cabinet_left" type="fixed">
-		<origin xyz="0.839 1.436 0.495" rpy="0 0 0" />
-		<parent link="dummy_link" />
-		<child link="cabinet_left" />
-	</joint>
-	<!-- cabinet_front_right -->
-	<link name="cabinet_front_right">
-		<inertial>
-			<origin xyz="0 0 0" />
-			<mass value="5.0" />
-			<inertia ixx="0.0" ixy="0.0" ixz="0.0" iyy="0.0" iyz="0.0" izz="0.0" />
-		</inertial>
-		<visual>
-			<origin xyz="0 0 0" />
-			<geometry>
-				<box size="0.04 0.04 0.84" />
-			</geometry>
-		</visual>
-		<collision>
-			<origin xyz="0 0 0" />
-			<geometry>
-				<box size="0.04 0.04 0.84" />
-			</geometry>
-		</collision>
-	</link>
-	<gazebo reference="cabinet_front_right">
-		<material>Gazebo/Grey</material>
-	</gazebo>
-	<joint name="joint_cabinet_front_right" type="fixed">
-		<origin xyz="1.489 1.271 0.420" rpy="0 0 0" />
-		<parent link="dummy_link" />
-		<child link="cabinet_front_right" />
-	</joint>
-	<!-- cabinet_front_left -->
-	<link name="cabinet_front_left">
-		<inertial>
-			<origin xyz="0 0 0" />
-			<mass value="5.0" />
-			<inertia ixx="0.0" ixy="0.0" ixz="0.0" iyy="0.0" iyz="0.0" izz="0.0" />
-		</inertial>
-		<visual>
-			<origin xyz="0 0 0" />
-			<geometry>
-				<box size="0.04 0.04 0.84" />
-			</geometry>
-		</visual>
-		<collision>
-			<origin xyz="0 0 0" />
-			<geometry>
-				<box size="0.04 0.04 0.84" />
-			</geometry>
-		</collision>
-	</link>
-	<gazebo reference="cabinet_front_left">
-		<material>Gazebo/Grey</material>
-	</gazebo>
-	<joint name="joint_cabinet_front_left" type="fixed">
-		<origin xyz="0.829 1.271 0.420" rpy="0 0 0" />
-		<parent link="dummy_link" />
-		<child link="cabinet_front_left" />
-	</joint>
-	<!-- cabinet_back_right -->
-	<link name="cabinet_back_right">
-		<inertial>
-			<origin xyz="0 0 0" />
-			<mass value="5.0" />
-			<inertia ixx="0.0" ixy="0.0" ixz="0.0" iyy="0.0" iyz="0.0" izz="0.0" />
-		</inertial>
-		<visual>
-			<origin xyz="0 0 0" />
-			<geometry>
-				<box size="0.04 0.04 0.84" />
-			</geometry>
-		</visual>
-		<collision>
-			<origin xyz="0 0 0" />
-			<geometry>
-				<box size="0.04 0.04 0.84" />
-			</geometry>
-		</collision>
-	</link>
-	<gazebo reference="cabinet_back_right">
-		<material>Gazebo/Grey</material>
-	</gazebo>
-	<joint name="joint_cabinet_back_right" type="fixed">
-		<origin xyz="1.489 1.601 0.420" rpy="0 0 0" />
-		<parent link="dummy_link" />
-		<child link="cabinet_back_right" />
-	</joint>
-	<!-- cabinet_back_left -->
-	<link name="cabinet_back_left">
-		<inertial>
-			<origin xyz="0 0 0" />
-			<mass value="5.0" />
-			<inertia ixx="0.0" ixy="0.0" ixz="0.0" iyy="0.0" iyz="0.0" izz="0.0" />
-		</inertial>
-		<visual>
-			<origin xyz="0 0 0" />
-			<geometry>
-				<box size="0.04 0.04 0.84" />
-			</geometry>
-		</visual>
-		<collision>
-			<origin xyz="0 0 0" />
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
Commit message: speed up simulation by modifying textures in kitchen-world

File: cob_gazebo_worlds/common/worlds/ipa-kitchen.urdf.xacro (robot description, xacro)
@@ -134,5 +134,5 @@
 	</link>
 	<gazebo reference="wall_03">
-		<material>IPA/Wall</material>
+		<material>IPA/Grey</material>
 	</gazebo>
 	<joint name="joint_wall_03" type="fixed">
@@ -218,5 +218,5 @@
 	</link>
 	<gazebo reference="wall_07">
-		<material>IPA/Wall</material>
+		<material>IPA/Grey</material>
 	</gazebo>
 	<joint name="joint_wall_07" type="fixed">
@@ -246,5 +246,5 @@
 	</link>
 	<gazebo reference="wall_08">
-		<material>IPA/Wall</material>
+		<material>IPA/Grey</material>
 	</gazebo>
 	<joint name="joint_wall_08" type="fixed">
@@ -274,5 +274,5 @@
 	</link>
 	<gazebo reference="wall_09">
-		<material>IPA/Wall</material>
+		<material>IPA/Grey</material>
 	</gazebo>
 	<joint name="joint_wall_09" type="fixed">
@@ -302,5 +302,5 @@
 	</link>
 	<gazebo reference="wall_10">
-		<material>IPA/Wall</material>
+		<material>IPA/Grey</material>
 	</gazebo>
 	<joint name="joint_wall_10" type="fixed">
@@ -330,5 +330,5 @@
 	</link>
 	<gazebo reference="wall_11">
-		<material>IPA/Wall</material>
+		<material>IPA/Grey</material>
 	</gazebo>
 	<joint name="joint_wall_11" type="fixed">
@@ -358,5 +358,5 @@
 	</link>
 	<gazebo reference="wall_12">
-		<material>IPA/Wall</material>
+		<material>IPA/Grey</material>
 	</gazebo>
 	<joint name="joint_wall_12" type="fixed">
@@ -386,5 +386,5 @@
 	</link>
 	<gazebo reference="wall_13">
-		<material>IPA/Wall</material>
+		<material>IPA/Grey</material>
 	</gazebo>
 	<joint name="joint_wall_13" type="fixed">
@@ -414,5 +414,5 @@
 	</link>
 	<gazebo reference="wall_14">
-		<material>IPA/Wall</material>
+		<material>IPA/Grey</material>
 	</gazebo>
 	<joint name="joint_wall_14" type="fixed">
@@ -442,5 +442,5 @@
 	</link>
 	<gazebo reference="wall_15">
-		<material>IPA/Wall</material>
+		<material>IPA/Grey</material>
 	</gazebo>
 	<joint name="joint_wall_15" type="fixed">
@@ -470,5 +470,5 @@
 	</link>
 	<gazebo reference="wall_16">
-		<material>IPA/Wall</material>
+		<material>IPA/Grey</material>
 	</gazebo>
 	<joint name="joint_wall_16" type="fixed">
@@ -498,5 +498,5 @@
 	</link>
 	<gazebo reference="wall_17">
-		<material>IPA/Wall</material>
+		<material>IPA/Grey</material>
 	</gazebo>
 	<joint name="joint_wall_17" type="fixed">
@@ -526,5 +526,5 @@
 	</link>
 	<gazebo reference="wall_18">
-		<material>IPA/Wall</material>
+		<material>IPA/Grey</material>
 	</gazebo>
 	<joint name="joint_wall_18" type="fixed">
@@ -554,5 +554,5 @@
 	</link>
 	<gazebo reference="wall_19">
-		<material>IPA/Wall</material>
+		<material>IPA/Grey</material>
 	</gazebo>
 	<joint name="joint_wall_19" type="fixed">
@@ -582,5 +582,5 @@
 	</link>
 	<gazebo reference="wall_20">
-		<material>IPA/Wall</material>
+		<material>IPA/Grey</material>
 	</gazebo>
 	<joint name="joint_wall_20" type="fixed">
@@ -610,5 +610,5 @@
 	</link>
 	<gazebo reference="wall_21">
-		<material>IPA/Wall</material>
+		<material>IPA/Grey</material>
 	</gazebo>
 	<joint name="joint_wall_21" type="fixed">
@@ -638,5 +638,5 @@
 	</link>
 	<gazebo reference="wall_22">
-		<material>IPA/Wall</material>
+		<material>IPA/Grey</material>
 	</gazebo>
 	<joint name="joint_wall_22" type="fixed">
@@ -666,5 +666,5 @@
 	</link>
 	<gazebo reference="wall_23">
-		<material>IPA/Wall</material>
+		<material>IPA/Grey</material>
 	</gazebo>
 	<joint name="joint_wall_23" type="fixed">
@@ -694,5 +694,5 @@
 	</link>
 	<gazebo reference="wall_24">
-		<material>IPA/Wall</material>
+		<material>IPA/Grey</material>
 	</gazebo>
 	<joint name="joint_wall_24" type="fixed">
@@ -722,5 +722,5 @@
 	</link>
 	<gazebo reference="wall_25">
-		<material>IPA/Wall</material>
+		<material>IPA/Grey</material>
 	</gazebo>
 	<joint name="joint_wall_25" type="fixed">

Commit message: new version of kitchen with freezer door

File: cob_gazebo_worlds/common/worlds/ipa-kitchen.urdf.xacro (robot description, xacro)
@@ -785,5 +785,5 @@
 		<child link="kitchen_middle" />
 	</joint>
-	<!-- kitchen_right -->
+	<!-- kitchen_right
 	<link name="kitchen_right">
 		<inertial>
@@ -811,5 +811,5 @@
 		<parent link="dummy_link" />
 		<child link="kitchen_right" />
-	</joint>
+	</joint>-->
 <!-- couch -->
 	<!-- left couch back -->
@@ -1172,4 +1172,154 @@
 		<child link="picture_06" />
 	</joint>
+ <!-- Start simulated freezer door -->
+	<link name="freezer_left">
+    <inertial>
+      <origin xyz="0 0 0" />
+      <mass value="100.0" />
+      <inertia  ixx="1.0" ixy="0.0"  ixz="0.0"  iyy="100.0"  iyz="0.0"  izz="1.0" />
+    </inertial>
+    <visual>
+      <origin xyz="0 0 0"/>
+      <geometry>
+        <box size="0.6 0.01 1.4" />
+      </geometry>
+    </visual>
+    <collision>
+      <origin xyz="0 0 0"/>
+      <geometry>
+        <box size="0.55 0.005 1.38" />
+      </geometry>
+    </collision>
+  </link>
+  <gazebo reference="freezer_left">
+    <material>Gazebo/White</material>
+  </gazebo>
+   <joint name="joint_freezer_lefft" type="fixed">
+    <origin xyz="-3.15 1.06 0.7" rpy="0 0 0"/>
+    <parent link="dummy_link"/>
+    <child link="freezer_left"/>
+ </joint>
+    <link name="freezer_right">
+    <inertial>
+      <origin xyz="0 0 0" />
+      <mass value="100.0" />
+      <inertia  ixx="1.0" ixy="0.0"  ixz="0.0"  iyy="100.0"  iyz="0.0"  izz="1.0" />
+    </inertial>
+    <visual>
+      <origin xyz="0 0 0"/>
+      <geometry>
+        <box size="0.6 0.01 1.4" />
+      </geometry>
+    </visual>
+    <collision>
+      <origin xyz="0 0 0"/>
+      <geometry>
+        <box size="0.55 0.005 1.38" />
+      </geometry>
+    </collision>
+  </link>
+  <gazebo reference="freezer_right">
+    <material>Gazebo/White</material>
+  </gazebo>
+   <joint name="joint_freezer_right" type="fixed">
+    <origin xyz="-3.15 1.66 0.7" rpy="0 0 0"/>
+    <parent link="dummy_link"/>
+    <child link="freezer_right"/>
+ </joint>
+  <gazebo reference="door_link">
+    <latchJoint>handle_joint</latchJoint>
+    <latchAngle>-1.57</latchAngle>
+    <doorClosedAngle>0.0</doorClosedAngle>
+    <latchKp>200.0</latchKp>
+    <latchKd>0.0</latchKd>
+    <latchFMax>1000.0</latchFMax>
+  </gazebo>
+  <joint name="door_joint" type="revolute" >
+    <origin xyz="0.305 0 0.02" rpy="0 0 0" />
+    <axis xyz="0 0 1" />
+    <limit lower="${-M_PI}" upper="${M_PI}" effort="1000" velocity="10" />
+    <safety_controller soft_lower_limit="${-M_PI+0.1}" soft_upper_limit="${M_PI-0.1}"
+           k_position="100.0" k_velocity="10.0" />
+    <dynamics damping="100" friction="0.0" />
+    <parent link="freezer_right" />
+    <child link="door_link" />
+  </joint>
+  <link name="door_link">
+    <inertial >
+      <mass value="30" />
+      <origin xyz="0 0 0" />
+      <inertia  ixx="1.0" ixy="0.0"  ixz="0.0"
+                iyy="1.0" iyz="0.0"
+                izz="3.0" />
+    </inertial>
+    <visual >
+      <origin xyz="0 -0.305 0" rpy="0 0 ${M_PI}" />
+      <geometry name="sholder_roll_mesh_file">
+        <box size="0.01 0.59 1.36" />
+      </geometry>
+    </visual>
+    <collision >
+      <origin xyz="0 -0.305 0" rpy="0 0 ${M_PI}" />
+      <geometry name="door_collision_geom">
+        <box size="0.01 0.59 1.36" />
+      </geometry>
+    </collision>
+  </link>
+  <gazebo reference="door_link">
+    <material>Gazebo/White</material>
+    <laserRetro>2000</laserRetro>
+    <turnGravityOff>true</turnGravityOff>
+    <selfCollide>false</selfCollide>
+    <dampingFactor>0.01</dampingFactor>
+  </gazebo>
+   <link name="handle">
+    <inertial>
+      <origin xyz="0 0 0" />
+      <mass value="1.0" />
+      <inertia  ixx="1.0" ixy="0.0"  ixz="0.0"  iyy="100.0"  iyz="0.0"  izz="1.0" />
+    </inertial>
+    <visual>
+      <origin xyz="0 0 0"/>
+      <geometry>
+        <box size="0.08 0.01 0.3" />
+      </geometry>
+    </visual>
+    <collision>
+      <origin xyz="0 0 0"/>
+      <geometry>
+        <box size="0.07 0.005 0.25" />
+      </geometry>
+    </collision>
+  </link>
+  <gazebo reference="handle">
+    <material>Gazebo/Blue</material>
+  </gazebo>
+   <joint name="joint_handle" type="fixed">
+    <origin xyz="0.051 -0.55  0.0" rpy="0 0 0"/>
+    <parent link="door_link"/>
+    <child link="handle"/>
+ </joint>
+  <gazebo>
+    <controller:gazebo_ros_p3d name="p3d_door_controller" plugin="libgazebo_ros_p3d.so">
+        <alwaysOn>true</alwaysOn>
+        <updateRate>100.0</updateRate>
+        <bodyName>door_link</bodyName>
+        <topicName>door_pose</topicName>
+        <frameName>/map</frameName>
+        <interface:position name="p3d_door_position"/>
+    </controller:gazebo_ros_p3d>
+    <controller:gazebo_ros_controller_manager name="door_controller_manager" plugin="libgazebo_ros_controller_manager.so">
+      <alwaysOn>true</alwaysOn>
+      <updateRate>1000.0</updateRate>
+      <robotParam>/world_description</robotParam>
+      <robotNamespace>/world</robotNamespace>
+      <interface:audio name="gazebo_ros_controller_manager_dummy_iface" />
+    </controller:gazebo_ros_controller_manager>
+  </gazebo>
+  <transmission type="pr2_mechanism_model/SimpleTransmission" name="door_trans">
+    <actuator name="door_motor" />
+    <joint name="door_joint" />
+    <mechanicalReduction>100</mechanicalReduction>
+  </transmission>
 </xacro:macro>
 <xacro:ipa-kitchen name="ipa-kitchen" />
