Commit message: small changes to ipa-kitchen

File: cob_gazebo_worlds/common/worlds/ipa-kitchen.urdf.xacro (robot description, xacro)
@@ -134,5 +134,5 @@
 	</link>
 	<gazebo reference="wall_03">
-		<material>IPA/Grey</material>
+		<material>IPA/Wall</material>
 	</gazebo>
 	<joint name="joint_wall_03" type="fixed">
@@ -218,5 +218,5 @@
 	</link>
 	<gazebo reference="wall_07">
-		<material>IPA/Grey</material>
+		<material>IPA/Wall</material>
 	</gazebo>
 	<joint name="joint_wall_07" type="fixed">
@@ -246,5 +246,5 @@
 	</link>
 	<gazebo reference="wall_08">
-		<material>IPA/Grey</material>
+		<material>IPA/Wall</material>
 	</gazebo>
 	<joint name="joint_wall_08" type="fixed">
@@ -274,5 +274,5 @@
 	</link>
 	<gazebo reference="wall_09">
-		<material>IPA/Grey</material>
+		<material>IPA/Wall</material>
 	</gazebo>
 	<joint name="joint_wall_09" type="fixed">
@@ -302,5 +302,5 @@
 	</link>
 	<gazebo reference="wall_10">
-		<material>IPA/Grey</material>
+		<material>IPA/Wall</material>
 	</gazebo>
 	<joint name="joint_wall_10" type="fixed">
@@ -330,5 +330,5 @@
 	</link>
 	<gazebo reference="wall_11">
-		<material>IPA/Grey</material>
+		<material>IPA/Wall</material>
 	</gazebo>
 	<joint name="joint_wall_11" type="fixed">
@@ -337,4 +337,35 @@
 		<child link="wall_11" />
 	</joint>
+	<link name="door">
+		<inertial>
+			<origin xyz="0 0 0" />
+			<mass value="10.0" />
+			<inertia ixx="0.0" ixy="0.0" ixz="0.0" iyy="0.0" iyz="0.0" izz="10.0" />
+		</inertial>
+		<visual>
+			<origin xyz="0.425 0 0" />
+			<geometry>
+				<box size="0.85 0.06 2.05" />
+			</geometry>
+		</visual>
+		<collision>
+			<origin xyz="0.425 0 0" />
+			<geometry>
+				<box size="0.75 0.06 2.01" />
+			</geometry>
+		</collision>
+	</link>
+	<gazebo reference="door">
+		<material>IPA/Wall2</material>
+	</gazebo>
+	<joint name="door_joint" type="revolute" >
+		<origin xyz="0.375 0.0 -0.275" rpy="0 0 0" />
+		<axis xyz="0 0 1" />
+		<limit lower="-1.8" upper="1.8" effort="1000" velocity="10" />
+		<safety_controller soft_lower_limit="-1.7" soft_upper_limit="1.7" k_position="100.0" k_velocity="10.0" />
+		<dynamics damping="60" friction="2000.0" />
+		<parent link="wall_11" />
+		<child link="door" />
+	</joint>
 	<!-- wall_12 -->
 	<link name="wall_12">
@@ -358,5 +389,5 @@
 	</link>
 	<gazebo reference="wall_12">
-		<material>IPA/Grey</material>
+		<material>IPA/Wall</material>
 	</gazebo>
 	<joint name="joint_wall_12" type="fixed">
@@ -386,5 +417,5 @@
 	</link>
 	<gazebo reference="wall_13">
-		<material>IPA/Grey</material>
+		<material>IPA/Wall</material>
 	</gazebo>
 	<joint name="joint_wall_13" type="fixed">
@@ -414,5 +445,5 @@
 	</link>
 	<gazebo reference="wall_14">
-		<material>IPA/Grey</material>
+		<material>IPA/Wall</material>
 	</gazebo>
 	<joint name="joint_wall_14" type="fixed">
@@ -442,5 +473,5 @@
 	</link>
 	<gazebo reference="wall_15">
-		<material>IPA/Grey</material>
+		<material>IPA/Wall</material>
 	</gazebo>
 	<joint name="joint_wall_15" type="fixed">
@@ -470,5 +501,5 @@
 	</link>
 	<gazebo reference="wall_16">
-		<material>IPA/Grey</material>
+		<material>IPA/Wall</material>
 	</gazebo>
 	<joint name="joint_wall_16" type="fixed">
@@ -498,5 +529,5 @@
 	</link>
 	<gazebo reference="wall_17">
-		<material>IPA/Grey</material>
+		<material>IPA/Wall</material>
 	</gazebo>
 	<joint name="joint_wall_17" type="fixed">
@@ -526,5 +557,5 @@
 	</link>
 	<gazebo reference="wall_18">
-		<material>IPA/Grey</material>
+		<material>IPA/Wall</material>
 	</gazebo>
 	<joint name="joint_wall_18" type="fixed">
@@ -554,5 +585,5 @@
 	</link>
 	<gazebo reference="wall_19">
-		<material>IPA/Grey</material>
+		<material>IPA/Wall</material>
 	</gazebo>
 	<joint name="joint_wall_19" type="fixed">
@@ -582,5 +613,5 @@
 	</link>
 	<gazebo reference="wall_20">
-		<material>IPA/Grey</material>
+		<material>IPA/Wall</material>
 	</gazebo>
 	<joint name="joint_wall_20" type="fixed">
@@ -610,5 +641,5 @@
 	</link>
 	<gazebo reference="wall_21">
-		<material>IPA/Grey</material>
+		<material>IPA/Wall</material>
 	</gazebo>
 	<joint name="joint_wall_21" type="fixed">
@@ -638,5 +669,5 @@
 	</link>
 	<gazebo reference="wall_22">
-		<material>IPA/Grey</material>
+		<material>IPA/Wall</material>
 	</gazebo>
 	<joint name="joint_wall_22" type="fixed">
@@ -666,5 +697,5 @@
 	</link>
 	<gazebo reference="wall_23">
-		<material>IPA/Grey</material>
+		<material>IPA/Wall</material>
 	</gazebo>
 	<joint name="joint_wall_23" type="fixed">
@@ -694,5 +725,5 @@
 	</link>
 	<gazebo reference="wall_24">
-		<material>IPA/Grey</material>
+		<material>IPA/Wall</material>
 	</gazebo>
 	<joint name="joint_wall_24" type="fixed">
@@ -722,5 +753,5 @@
 	</link>
 	<gazebo reference="wall_25">
-		<material>IPA/Grey</material>
+		<material>IPA/Wall</material>
 	</gazebo>
 	<joint name="joint_wall_25" type="fixed">

Commit message: revert freezer door

File: cob_gazebo_worlds/common/worlds/ipa-kitchen.urdf.xacro (robot description, xacro)
@@ -7,5 +7,4 @@
 	name="ipa-kitchen"
 >
-  <property name="M_PI" value="3.1415926535897931" />
 <xacro:macro name="ipa-kitchen" params="name">
 <!-- dummy_link -->
@@ -135,5 +134,5 @@
 	</link>
 	<gazebo reference="wall_03">
-		<material>IPA/Grey</material>
+		<material>IPA/Wall</material>
 	</gazebo>
 	<joint name="joint_wall_03" type="fixed">
@@ -219,5 +218,5 @@
 	</link>
 	<gazebo reference="wall_07">
-		<material>IPA/Grey</material>
+		<material>IPA/Wall</material>
 	</gazebo>
 	<joint name="joint_wall_07" type="fixed">
@@ -247,5 +246,5 @@
 	</link>
 	<gazebo reference="wall_08">
-		<material>IPA/Grey</material>
+		<material>IPA/Wall</material>
 	</gazebo>
 	<joint name="joint_wall_08" type="fixed">
@@ -275,5 +274,5 @@
 	</link>
 	<gazebo reference="wall_09">
-		<material>IPA/Grey</material>
+		<material>IPA/Wall</material>
 	</gazebo>
 	<joint name="joint_wall_09" type="fixed">
@@ -303,5 +302,5 @@
 	</link>
 	<gazebo reference="wall_10">
-		<material>IPA/Grey</material>
+		<material>IPA/Wall</material>
 	</gazebo>
 	<joint name="joint_wall_10" type="fixed">
@@ -331,5 +330,5 @@
 	</link>
 	<gazebo reference="wall_11">
-		<material>IPA/Grey</material>
+		<material>IPA/Wall</material>
 	</gazebo>
 	<joint name="joint_wall_11" type="fixed">
@@ -359,5 +358,5 @@
 	</link>
 	<gazebo reference="wall_12">
-		<material>IPA/Grey</material>
+		<material>IPA/Wall</material>
 	</gazebo>
 	<joint name="joint_wall_12" type="fixed">
@@ -387,5 +386,5 @@
 	</link>
 	<gazebo reference="wall_13">
-		<material>IPA/Grey</material>
+		<material>IPA/Wall</material>
 	</gazebo>
 	<joint name="joint_wall_13" type="fixed">
@@ -415,5 +414,5 @@
 	</link>
 	<gazebo reference="wall_14">
-		<material>IPA/Grey</material>
+		<material>IPA/Wall</material>
 	</gazebo>
 	<joint name="joint_wall_14" type="fixed">
@@ -443,5 +442,5 @@
 	</link>
 	<gazebo reference="wall_15">
-		<material>IPA/Grey</material>
+		<material>IPA/Wall</material>
 	</gazebo>
 	<joint name="joint_wall_15" type="fixed">
@@ -471,5 +470,5 @@
 	</link>
 	<gazebo reference="wall_16">
-		<material>IPA/Grey</material>
+		<material>IPA/Wall</material>
 	</gazebo>
 	<joint name="joint_wall_16" type="fixed">
@@ -499,5 +498,5 @@
 	</link>
 	<gazebo reference="wall_17">
-		<material>IPA/Grey</material>
+		<material>IPA/Wall</material>
 	</gazebo>
 	<joint name="joint_wall_17" type="fixed">
@@ -527,5 +526,5 @@
 	</link>
 	<gazebo reference="wall_18">
-		<material>IPA/Grey</material>
+		<material>IPA/Wall</material>
 	</gazebo>
 	<joint name="joint_wall_18" type="fixed">
@@ -555,5 +554,5 @@
 	</link>
 	<gazebo reference="wall_19">
-		<material>IPA/Grey</material>
+		<material>IPA/Wall</material>
 	</gazebo>
 	<joint name="joint_wall_19" type="fixed">
@@ -583,5 +582,5 @@
 	</link>
 	<gazebo reference="wall_20">
-		<material>IPA/Grey</material>
+		<material>IPA/Wall</material>
 	</gazebo>
 	<joint name="joint_wall_20" type="fixed">
@@ -611,5 +610,5 @@
 	</link>
 	<gazebo reference="wall_21">
-		<material>IPA/Grey</material>
+		<material>IPA/Wall</material>
 	</gazebo>
 	<joint name="joint_wall_21" type="fixed">
@@ -639,5 +638,5 @@
 	</link>
 	<gazebo reference="wall_22">
-		<material>IPA/Grey</material>
+		<material>IPA/Wall</material>
 	</gazebo>
 	<joint name="joint_wall_22" type="fixed">
@@ -667,5 +666,5 @@
 	</link>
 	<gazebo reference="wall_23">
-		<material>IPA/Grey</material>
+		<material>IPA/Wall</material>
 	</gazebo>
 	<joint name="joint_wall_23" type="fixed">
@@ -695,5 +694,5 @@
 	</link>
 	<gazebo reference="wall_24">
-		<material>IPA/Grey</material>
+		<material>IPA/Wall</material>
 	</gazebo>
 	<joint name="joint_wall_24" type="fixed">
@@ -723,5 +722,5 @@
 	</link>
 	<gazebo reference="wall_25">
-		<material>IPA/Grey</material>
+		<material>IPA/Wall</material>
 	</gazebo>
 	<joint name="joint_wall_25" type="fixed">
@@ -786,5 +785,4 @@
 	</joint>
 	<!-- kitchen_right -->
-	<!--
 	<link name="kitchen_right">
 		<inertial>
@@ -812,33 +810,5 @@
 		<parent link="dummy_link" />
 		<child link="kitchen_right" />
-	</joint>-->
-  <link name="freezer_top">
-    <inertial>
-      <origin xyz="0 0 0" />
-      <mass value="1.0" />
-      <inertia  ixx="1.0" ixy="0.0"  ixz="0.0"  iyy="100.0"  iyz="0.0"  izz="1.0" />
-    </inertial>
-    <visual>
-      <origin xyz="0 0 0"/>
-      <geometry>
-        <box size="0.6 0.6 0.01" />
-      </geometry>
-    </visual>
-    <collision>
-      <origin xyz="0 0 0"/>
-      <geometry>
-        <box size="0.6 0.6 0.01" />
-      </geometry>
-    </collision>
-  </link>
-  <gazebo reference="freezer_top">
-    <material>Gazebo/Red</material>
-  </gazebo>
-   <joint name="joint_freezer_top" type="fixed">
-    <origin xyz="-3.2 1.36 1.4" rpy="0 0 0"/>
-    <parent link="dummy_link"/>
-    <child link="freezer_top"/>
- </joint>
->>>>>>> review-320
+	</joint>
 <!-- couch -->
 	<!-- left couch back -->
@@ -1201,154 +1171,4 @@
 		<child link="picture_06" />
 	</joint>
- <!-- Start simulated freezer door -->
-	<link name="freezer_left">
-    <inertial>
-      <origin xyz="0 0 0" />
-      <mass value="100.0" />
-      <inertia  ixx="1.0" ixy="0.0"  ixz="0.0"  iyy="100.0"  iyz="0.0"  izz="1.0" />
-    </inertial>
-    <visual>
-      <origin xyz="0 0 0"/>
-      <geometry>
-        <box size="0.6 0.01 1.4" />
-      </geometry>
-    </visual>
-    <collision>
-      <origin xyz="0 0 0"/>
-      <geometry>
-        <box size="0.55 0.005 1.38" />
-      </geometry>
-    </collision>
-  </link>
-  <gazebo reference="freezer_left">
-    <material>Gazebo/White</material>
-  </gazebo>
-   <joint name="joint_freezer_lefft" type="fixed">
-    <origin xyz="-3.15 1.06 0.7" rpy="0 0 0"/>
-    <parent link="dummy_link"/>
-    <child link="freezer_left"/>
- </joint>
-    <link name="freezer_right">
-    <inertial>
-      <origin xyz="0 0 0" />
-      <mass value="100.0" />
-      <inertia  ixx="1.0" ixy="0.0"  ixz="0.0"  iyy="100.0"  iyz="0.0"  izz="1.0" />
-    </inertial>
-    <visual>
-      <origin xyz="0 0 0"/>
-      <geometry>
-        <box size="0.6 0.01 1.4" />
-      </geometry>
-    </visual>
-    <collision>
-      <origin xyz="0 0 0"/>
-      <geometry>
-        <box size="0.55 0.005 1.38" />
-      </geometry>
-    </collision>
-  </link>
-  <gazebo reference="freezer_right">
-    <material>Gazebo/White</material>
-  </gazebo>
-   <joint name="joint_freezer_right" type="fixed">
-    <origin xyz="-3.15 1.66 0.7" rpy="0 0 0"/>
-    <parent link="dummy_link"/>
-    <child link="freezer_right"/>
- </joint>
-  <gazebo reference="door_link">
-    <latchJoint>handle_joint</latchJoint>
-    <latchAngle>-1.57</latchAngle>
-    <doorClosedAngle>0.0</doorClosedAngle>
-    <latchKp>200.0</latchKp>
-    <latchKd>0.0</latchKd>
-    <latchFMax>1000.0</latchFMax>
-  </gazebo>
-  <joint name="door_joint" type="revolute" >
-    <origin xyz="0.305 0 0.02" rpy="0 0 0" />
-    <axis xyz="0 0 1" />
-    <limit lower="${-M_PI}" upper="${M_PI}" effort="1000" velocity="10" />
-    <safety_controller soft_lower_limit="${-M_PI+0.1}" soft_upper_limit="${M_PI-0.1}"
-           k_position="100.0" k_velocity="10.0" />
-    <dynamics damping="100" friction="0.0" />
-    <parent link="freezer_right" />
-    <child link="door_link" />
-  </joint>
-  <link name="door_link">
-    <inertial >
-      <mass value="30" />
-      <origin xyz="0 0 0" />
-      <inertia  ixx="1.0" ixy="0.0"  ixz="0.0"
-                iyy="1.0" iyz="0.0"
-                izz="3.0" />
-    </inertial>
-    <visual >
-      <origin xyz="0 -0.305 0" rpy="0 0 ${M_PI}" />
-      <geometry name="sholder_roll_mesh_file">
-        <box size="0.01 0.59 1.36" />
-      </geometry>
-    </visual>
-    <collision >
-      <origin xyz="0 -0.305 0" rpy="0 0 ${M_PI}" />
-      <geometry name="door_collision_geom">
-        <box size="0.01 0.59 1.36" />
-      </geometry>
-    </collision>
-  </link>
-  <gazebo reference="door_link">
-    <material>Gazebo/White</material>
-    <laserRetro>2000</laserRetro>
-    <turnGravityOff>true</turnGravityOff>
-    <selfCollide>false</selfCollide>
-    <dampingFactor>0.01</dampingFactor>
-  </gazebo>
-   <link name="handle">
-    <inertial>
-      <origin xyz="0 0 0" />
-      <mass value="1.0" />
-      <inertia  ixx="1.0" ixy="0.0"  ixz="0.0"  iyy="100.0"  iyz="0.0"  izz="1.0" />
-    </inertial>
-    <visual>
-      <origin xyz="0 0 0"/>
-      <geometry>
-        <box size="0.08 0.01 0.3" />
-      </geometry>
-    </visual>
-    <collision>
-      <origin xyz="0 0 0"/>
-      <geometry>
-        <box size="0.08 0.01 0.3" />
-      </geometry>
-    </collision>
-  </link>
-  <gazebo reference="handle">
-    <material>Gazebo/Blue</material>
-  </gazebo>
-   <joint name="joint_handle" type="fixed">
-    <origin xyz="0.051 -0.55  0.0" rpy="0 0 0"/>
-    <parent link="door_link"/>
-    <child link="handle"/>
- </joint>
-  <gazebo>
-    <controller:gazebo_ros_p3d name="p3d_door_controller" plugin="libgazebo_ros_p3d.so">
-        <alwaysOn>true</alwaysOn>
-        <updateRate>100.0</updateRate>
-        <bodyName>door_link</bodyName>
-        <topicName>door_pose</topicName>
-        <frameName>/map</frameName>
-        <interface:position name="p3d_door_position"/>
-    </controller:gazebo_ros_p3d>
-    <controller:gazebo_ros_controller_manager name="door_controller_manager" plugin="libgazebo_ros_controller_manager.so">
-      <alwaysOn>true</alwaysOn>
-      <updateRate>1000.0</updateRate>
-      <robotParam>/world_description</robotParam>
-      <robotNamespace>/world</robotNamespace>
-      <interface:audio name="gazebo_ros_controller_manager_dummy_iface" />
-    </controller:gazebo_ros_controller_manager>
-  </gazebo>
-  <transmission type="pr2_mechanism_model/SimpleTransmission" name="door_trans">
-    <actuator name="door_motor" />
-    <joint name="door_joint" />
-    <mechanicalReduction>100</mechanicalReduction>
-  </transmission>
 </xacro:macro>
 <xacro:ipa-kitchen name="ipa-kitchen" />
