Commit message: modified gazebo world to fit new navi map

File: cob_gazebo_worlds/common/worlds/raw-exhibition.urdf.xacro (robot description, xacro)
@@ -162,8 +162,8 @@
 	</link>
 	<gazebo reference="regal_links">
-		<material>IPA/Wall2</material>
+		<material>IPA/Wall3</material>
 	</gazebo>
 	<joint name="joint_regal_links" type="fixed">
-		<origin xyz="-1.4 1.1 0.72" rpy="0 0 0.2" />
+		<origin xyz="-1.45 1.6 0.72" rpy="0 0 1.08" />
 		<parent link="dummy_link" />
 		<child link="regal_links" />
@@ -189,5 +189,5 @@
 	</link>
 	<gazebo reference="regal_rechts">
-		<material>IPA/Wall2</material>
+		<material>IPA/Wall3</material>
 	</gazebo>
 	<joint name="joint_regal_rechts" type="fixed">
@@ -216,5 +216,5 @@
 	</link>
 	<gazebo reference="regal_fach1">
-		<material>IPA/Wall2</material>
+		<material>IPA/Wall3</material>
 	</gazebo>
 	<joint name="joint_regal_fach1" type="fixed">
@@ -243,5 +243,5 @@
 	</link>
 	<gazebo reference="regal_fach2">
-		<material>IPA/Wall2</material>
+		<material>IPA/Wall3</material>
 	</gazebo>
 	<joint name="joint_regal_fach2" type="fixed">
@@ -271,8 +271,8 @@
 	</link>
 	<gazebo reference="arbeitsplatz1">
-		<material>IPA/Wall2</material>
+		<material>IPA/Wall3</material>
 	</gazebo>
 	<joint name="joint_arbeitsplatz1" type="fixed">
-		<origin xyz="1.1 -1.1 0.72" rpy="0 0 0" />
+		<origin xyz="1.25 -1.1 0.72" rpy="0 0 0" />
 		<parent link="dummy_link" />
 		<child link="arbeitsplatz1" />
@@ -298,5 +298,5 @@
 	</link>
 	<gazebo reference="arbeitsplatz2">
-		<material>IPA/Wall2</material>
+		<material>IPA/Wall3</material>
 	</gazebo>
 	<joint name="joint_arbeitsplatz2" type="fixed">
