Commit message: new ipa-apartment worldcob_gazebo_objects/config/ipa-apartment/object_locations.yaml

File: cob_gazebo_worlds/common/worlds/ipa-apartment.urdf.xacro (robot description, xacro)
@@ -6,9 +6,23 @@
 	xmlns:xacro="http://playerstage.sourceforge.net/gazebo/xmlschema/#interface"
 	name="ipa-apartment">
-  <property name="size_x" value="6" /> <!--this parameter is not real-->
-  <property name="size_y" value="4.3" />
+<!--- Translation: [-1.577, 4.350, 0.000]
+- Rotation: in Quaternion [0.000, 0.000, -0.042, 0.999]
+            in RPY [0.000, 0.000, -0.084]
+Setting pose: 1.969 -4.262 0.087
+1.998 -4.081 0.030
+[1.969, -4.070, 0.000]-->
+  <property name="dist_axis_x" value="1.969" />
+  <property name="dist_axis_y" value="4.070" />
+  <property name="dist_axis_yall" value="0"/> <!--0.015-->
+  <property name="size_total_x" value="8.0" />
+  <property name="size_total_y" value="11.2" />
+  <property name="size_a" value="4.7" />
+  <property name="size_b" value="8.2" />
+  <property name="size_c" value="1.8" />
+  <property name="size_d" value="4.16" />
   <property name="wall_depth" value="0.06" />
-  <property name="size_z_wall1" value="3.20" />
-  <property name="size_z_wall2" value="0.5" />
+  <property name="window_depth" value="0.15" />
+  <property name="size_z_wall1" value="2.8" />
+  <property name="size_z_wall2" value="0.92" />
 <xacro:macro name="ipa-apartment" params="name">
 <!-- dummy_link -->
@@ -32,115 +46,447 @@
 		</collision>
 	</link>
-	<!-- wall_1 -->
-	<link name="wall_1">
-		<inertial>
-			<origin xyz="0 0 0" />
-			<mass value="5.0" />
-			<inertia ixx="0.0" ixy="0.0" ixz="0.0" iyy="0.0" iyz="0.0" izz="0.0" />
-		</inertial>
-		<visual>
-			<origin xyz="0 0 0" />
-			<geometry>
-				<box size="${wall_depth} ${size_y} ${size_z_wall2}" />
-			</geometry>
-		</visual>
-		<collision>
-			<origin xyz="0 0 0" />
-			<geometry>
-				<box size="${wall_depth+0.02} ${size_y} ${size_z_wall2}" />
-			</geometry>
-		</collision>
-	</link>
-	<gazebo reference="wall_1">
+	<!-- wall_00 -->
+	<link name="wall_00">
+		<inertial>
+			<origin xyz="0 0 0" />
+			<mass value="5.0" />
+			<inertia ixx="0.0" ixy="0.0" ixz="0.0" iyy="0.0" iyz="0.0" izz="0.0" />
+		</inertial>
+		<visual>
+			<origin xyz="0 0 0" />
+			<geometry>
+				<box size="${wall_depth} ${size_d} ${size_z_wall1}" />
+			</geometry>
+		</visual>
+		<collision>
+			<origin xyz="0 0 0" />
+			<geometry>
+				<box size="${wall_depth} ${size_d} ${size_z_wall1}" />
+			</geometry>
+		</collision>
+	</link>
+	<gazebo reference="wall_00">
+		<material>IPA/WallApartment</material>
+	</gazebo>
+	<joint name="joint_wall_00" type="fixed">
+		<origin xyz="${-size_total_x/2+dist_axis_x-wall_depth} ${size_total_y/2-size_d/2+0.1-dist_axis_y} ${size_z_wall1/2}" rpy="0 0 ${-dist_axis_yall}" />
+		<parent link="dummy_link" />
+		<child link="wall_00" />
+	</joint>
+	<!-- wall_01 -->
+	<link name="wall_01">
+		<inertial>
+			<origin xyz="0 0 0" />
+			<mass value="5.0" />
+			<inertia ixx="0.0" ixy="0.0" ixz="0.0" iyy="0.0" iyz="0.0" izz="0.0" />
+		</inertial>
+		<visual>
+			<origin xyz="0 0 0" />
+			<geometry>
+				<box size=" ${size_b} ${window_depth} ${size_z_wall2}" />
+			</geometry>
+		</visual>
+		<collision>
+			<origin xyz="0 0 0" />
+			<geometry>
+				<box size="${size_b} ${window_depth} ${size_z_wall2}" />
+			</geometry>
+		</collision>
+	</link>
+	<gazebo reference="wall_01">
+		<material>IPA/WallApartment</material>
+	</gazebo>
+	<joint name="joint_wall_01" type="fixed">
+		<origin xyz="${dist_axis_x} ${size_total_y/2-dist_axis_y+window_depth} ${size_z_wall2/2}" rpy="0 0 ${-dist_axis_yall}" />
+		<parent link="dummy_link" />
+		<child link="wall_01" />
+	</joint>
+	<!-- wall_02 -->
+	<link name="wall_02">
+		<inertial>
+			<origin xyz="0 0 0" />
+			<mass value="5.0" />
+			<inertia ixx="0.0" ixy="0.0" ixz="0.0" iyy="0.0" iyz="0.0" izz="0.0" />
+		</inertial>
+		<visual>
+			<origin xyz="0 0 0" />
+			<geometry>
+				<box size="${wall_depth} ${size_a} ${size_z_wall2}" />
+			</geometry>
+		</visual>
+		<collision>
+			<origin xyz="0 0 0" />
+			<geometry>
+				<box size="${wall_depth} ${size_a} ${size_z_wall2}" />
+			</geometry>
+		</collision>
+	</link>
+	<gazebo reference="wall_02">
+		<material>IPA/WallApartment</material>
+	</gazebo>
+	<joint name="joint_wall_02" type="fixed">
+		<origin xyz="${size_total_x/2+dist_axis_x+wall_depth} ${size_total_y/2-size_a/2+0.15-dist_axis_y} ${size_z_wall2/2}" rpy="0 0 ${-dist_axis_yall}" />
+		<parent link="dummy_link" />
+		<child link="wall_02" />
+	</joint>
+	<!-- wall_03 -->
+	<link name="wall_03">
+		<inertial>
+			<origin xyz="0 0 0" />
+			<mass value="5.0" />
+			<inertia ixx="0.0" ixy="0.0" ixz="0.0" iyy="0.0" iyz="0.0" izz="0.0" />
+		</inertial>
+		<visual>
+			<origin xyz="0 0 0" />
+			<geometry>
+				<box size=" ${window_depth} 1.6 ${size_z_wall2}" />
+			</geometry>
+		</visual>
+		<collision>
+			<origin xyz="0 0 0" />
+			<geometry>
+				<box size="${window_depth} 1.5 ${size_z_wall2}" />
+			</geometry>
+		</collision>
+	</link>
+	<gazebo reference="wall_03">
+		<material>IPA/WallApartment</material>
+	</gazebo>
+	<joint name="joint_wall_03" type="fixed">
+		<origin xyz="${size_total_x/2+dist_axis_x+0.561+window_depth/2} ${0.5-dist_axis_y} ${size_z_wall2/2}" rpy="0 0 ${-dist_axis_yall+0.785398}" />
+		<parent link="dummy_link" />
+		<child link="wall_03" />
+	</joint>
+	<!-- wall_04 -->
+	<link name="wall_04">
+		<inertial>
+			<origin xyz="0 0 0" />
+			<mass value="5.0" />
+			<inertia ixx="0.0" ixy="0.0" ixz="0.0" iyy="0.0" iyz="0.0" izz="0.0" />
+		</inertial>
+		<visual>
+			<origin xyz="0 0 0" />
+			<geometry>
+				<box size="${window_depth} 1.55 ${size_z_wall2}" />
+			</geometry>
+		</visual>
+		<collision>
+			<origin xyz="0 0 0" />
+			<geometry>
+				<box size="${window_depth} 1.5 ${size_z_wall2}" />
+			</geometry>
+		</collision>
+	</link>
+	<gazebo reference="wall_04">
+		<material>IPA/WallApartment</material>
+	</gazebo>
+	<joint name="joint_wall_04" type="fixed">
+		<origin xyz="${size_total_x/2+dist_axis_x+0.561+window_depth/2} ${-0.5-dist_axis_y} ${size_z_wall2/2}" rpy="0 0 ${-dist_axis_yall-0.785398}" />
+		<parent link="dummy_link" />
+		<child link="wall_04" />
+	</joint>
+	<!-- wall_05 -->
+	<link name="wall_05">
+		<inertial>
+			<origin xyz="0 0 0" />
+			<mass value="5.0" />
+			<inertia ixx="0.0" ixy="0.0" ixz="0.0" iyy="0.0" iyz="0.0" izz="0.0" />
+		</inertial>
+		<visual>
+			<origin xyz="0 0 0" />
+			<geometry>
+				<box size="${wall_depth} ${size_a} ${size_z_wall2}" />
+			</geometry>
+		</visual>
+		<collision>
+			<origin xyz="0 0 0" />
+			<geometry>
+				<box size="${wall_depth} ${size_a} ${size_z_wall2}" />
+			</geometry>
+		</collision>
+	</link>
+	<gazebo reference="wall_05">
+		<material>IPA/WallApartment</material>
+	</gazebo>
+	<joint name="joint_wall_05" type="fixed">
+		<origin xyz="${size_total_x/2+dist_axis_x+wall_depth} ${-size_total_y/2+size_a/2-0.15-dist_axis_y} ${size_z_wall2/2}" rpy="0 0 ${-dist_axis_yall}" />
+		<parent link="dummy_link" />
+		<child link="wall_05" />
+	</joint>
+	<!-- wall_06 -->
+	<link name="wall_06">
+		<inertial>
+			<origin xyz="0 0 0" />
+			<mass value="5.0" />
+			<inertia ixx="0.0" ixy="0.0" ixz="0.0" iyy="0.0" iyz="0.0" izz="0.0" />
+		</inertial>
+		<visual>
+			<origin xyz="0 0 0" />
+			<geometry>
+				<box size=" ${size_b} ${window_depth} ${size_z_wall2}" />
+			</geometry>
+		</visual>
+		<collision>
+			<origin xyz="0 0 0" />
+			<geometry>
+				<box size="${size_b} ${window_depth+0.02} ${size_z_wall2}" />
+			</geometry>
+		</collision>
+	</link>
+	<gazebo reference="wall_06">
+		<material>IPA/WallApartment</material>
+	</gazebo>
+	<joint name="joint_wall_06" type="fixed">
+		<origin xyz="${+dist_axis_x-0.05} ${-size_total_y/2-dist_axis_y-window_depth} ${size_z_wall2/2}" rpy="0 0 ${-dist_axis_yall}" />
+		<parent link="dummy_link" />
+		<child link="wall_06" />
+	</joint>
+	<!-- wall_07 -->
+	<link name="wall_07">
+		<inertial>
+			<origin xyz="0 0 0" />
+			<mass value="5.0" />
+			<inertia ixx="0.0" ixy="0.0" ixz="0.0" iyy="0.0" iyz="0.0" izz="0.0" />
+		</inertial>
+		<visual>
+			<origin xyz="0 0 0" />
+			<geometry>
+				<box size="${wall_depth} ${size_a} ${size_z_wall1}" />
+			</geometry>
+		</visual>
+		<collision>
+			<origin xyz="0 0 0" />
+			<geometry>
+				<box size="${wall_depth} ${size_a} ${size_z_wall1}" />
+			</geometry>
+		</collision>
+	</link>
+	<gazebo reference="wall_07">
+		<material>IPA/WallApartment</material>
+	</gazebo>
+	<joint name="joint_wall_07" type="fixed">
+		<origin xyz="${-size_total_x/2+dist_axis_x-wall_depth} ${-size_total_y/2+size_a/2-0.1-dist_axis_y} ${size_z_wall1/2}" rpy="0 0 ${-dist_axis_yall}" />
+		<parent link="dummy_link" />
+		<child link="wall_07" />
+	</joint>
+	<!-- wall_08 -->
+	<link name="wall_08">
+		<inertial>
+			<origin xyz="0 0 0" />
+			<mass value="5.0" />
+			<inertia ixx="0.0" ixy="0.0" ixz="0.0" iyy="0.0" iyz="0.0" izz="0.0" />
+		</inertial>
+		<visual>
+			<origin xyz="0 0 0" />
+			<geometry>
+				<box size="${wall_depth} 1.9 ${size_z_wall2}" />
+			</geometry>
+		</visual>
+		<collision>
+			<origin xyz="0 0 0" />
+			<geometry>
+				<box size="${wall_depth} 1.9 ${size_z_wall2}" />
+			</geometry>
+		</collision>
+	</link>
+	<gazebo reference="wall_08">
+		<material>IPA/WallApartment</material>
+	</gazebo>
+	<joint name="joint_wall_08" type="fixed">
+		<origin xyz="${size_total_x/2-1.8+dist_axis_x+wall_depth} ${size_total_y/2-3.6+0.1-dist_axis_y} ${size_z_wall2/2}" rpy="0 0 ${-dist_axis_yall}" />
+		<parent link="dummy_link" />
+		<child link="wall_08" />
+	</joint>
+	<!-- door_00 -->
+	<link name="door_00">
+		<inertial>
+			<origin xyz="0 0 0" />
+			<mass value="5.0" />
+			<inertia ixx="0.0" ixy="0.0" ixz="0.0" iyy="0.0" iyz="0.0" izz="0.0" />
+		</inertial>
+		<visual>
+			<origin xyz="0 0 0" />
+			<geometry>
+				<box size="0.04 0.62 ${size_z_wall1}" />
+			</geometry>
+		</visual>
+		<collision>
+			<origin xyz="0 0 0" />
+			<geometry>
+				<box size="0.04 0.62 ${size_z_wall1}" />
+			</geometry>
+		</collision>
+	</link>
+	<gazebo reference="door_00">
 		<material>IPA/Wall2</material>
 	</gazebo>
-	<joint name="joint_wall_1" type="fixed">
-		<origin xyz="${size_x/2} 0 ${size_z_wall2/2}" rpy="0 0 0" />
-		<parent link="dummy_link" />
-		<child link="wall_1" />
-	</joint>
-	<!-- wall_2 -->
-	<link name="wall_2">
-		<inertial>
-			<origin xyz="0 0 0" />
-			<mass value="5.0" />
-			<inertia ixx="0.0" ixy="0.0" ixz="0.0" iyy="0.0" iyz="0.0" izz="0.0" />
-		</inertial>
-		<visual>
-			<origin xyz="0 0 0" />
-			<geometry>
-				<box size=" ${size_x} ${wall_depth} ${size_z_wall2}" />
-			</geometry>
-		</visual>
-		<collision>
-			<origin xyz="0 0 0" />
-			<geometry>
-				<box size="${size_x} ${wall_depth+0.02} ${size_z_wall2}" />
-			</geometry>
-		</collision>
-	</link>
-	<gazebo reference="wall_2">
+	<joint name="joint_door_00" type="fixed">
+		<origin xyz="${-size_total_x/2+dist_axis_x-wall_depth} ${1.22-dist_axis_y} ${size_z_wall1/2}" rpy="0 0 ${-dist_axis_yall}" />
+		<parent link="dummy_link" />
+		<child link="door_00" />
+	</joint>
+	<!-- door_01 -->
+	<link name="door_01">
+		<inertial>
+			<origin xyz="0 0 0" />
+			<mass value="5.0" />
+			<inertia ixx="0.0" ixy="0.0" ixz="0.0" iyy="0.0" iyz="0.0" izz="0.0" />
+		</inertial>
+		<visual>
+			<origin xyz="0 0 0" />
+			<geometry>
+				<box size="0.04 0.62 ${size_z_wall1}" />
+			</geometry>
+		</visual>
+		<collision>
+			<origin xyz="0 0 0" />
+			<geometry>
+				<box size="0.04 0.62 ${size_z_wall1}" />
+			</geometry>
+		</collision>
+	</link>
+	<gazebo reference="door_01">
 		<material>IPA/Wall2</material>
 	</gazebo>
-	<joint name="joint_wall_2" type="fixed">
-		<origin xyz="0 ${-size_y/2} ${size_z_wall2/2}" rpy="0 0 0" />
-		<parent link="dummy_link" />
-		<child link="wall_2" />
-	</joint>
-	<!-- wall_3 -->
-	<link name="wall_3">
-		<inertial>
-			<origin xyz="0 0 0" />
-			<mass value="5.0" />
-			<inertia ixx="0.0" ixy="0.0" ixz="0.0" iyy="0.0" iyz="0.0" izz="0.0" />
-		</inertial>
-		<visual>
-			<origin xyz="0 0 0" />
-			<geometry>
-				<box size="${wall_depth} ${size_y} ${size_z_wall1}" />
-			</geometry>
-		</visual>
-		<collision>
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