Commit message: wimicare project: simulation test with objects

File: cob_gazebo_worlds/objects/person.urdf.xacro (robot description, xacro)
@@ -16,10 +16,10 @@
 		<visual>
 			<geometry>
-				<cylinder length="1.6" radius="0.2"/>
+				<cylinder length="1.2" radius="0.2"/>
 			</geometry>
 		</visual>
 		<collision>
 			<geometry>
-				<cylinder length="1.6" radius="0.2"/>
+				<cylinder length="1.2" radius="0.2"/>
 			</geometry>
 		</collision>
