Commit message: added image_proc and changed furniture color

File: cob_gazebo_worlds/objects/bookcase.urdf.xacro (robot description, xacro)
@@ -64,5 +64,5 @@
 	</link>
 	<gazebo reference="bookcase_top_link">
-		<material>IPA/White</material>
+		<material>Gazebo/White</material>
 	</gazebo>
 	<joint name="joint_bookcase_top" type="fixed">
@@ -92,5 +92,5 @@
 	</link>
 	<gazebo reference="bookcase_bottom_link">
-		<material>IPA/White</material>
+		<material>Gazebo/White</material>
 	</gazebo>
 	<joint name="joint_bookcase_bottom" type="fixed">
@@ -120,5 +120,5 @@
 	</link>
 	<gazebo reference="bookcase_middle">
-		<material>IPA/White</material>
+		<material>Gazebo/White</material>
 	</gazebo>
 	<joint name="joint_bookcase_middle" type="fixed">
@@ -148,5 +148,5 @@
 	</link>
 	<gazebo reference="bookcase_right">
-		<material>IPA/White</material>
+		<material>Gazebo/White</material>
 	</gazebo>
 	<joint name="joint_bookcase_right" type="fixed">
@@ -176,5 +176,5 @@
 	</link>
 	<gazebo reference="bookcase_left">
-		<material>IPA/White</material>
+		<material>Gazebo/White</material>
 	</gazebo>
 	<joint name="joint_bookcase_left" type="fixed">

File: cob_gazebo_worlds/objects/cabinet_with_door.urdf.xacro (robot description, xacro)
@@ -62,5 +62,5 @@
 	</link>
 	<gazebo reference="cabinet_structure">
-		<material>IPA/White</material>
+		<material>Gazebo/White</material>
 	</gazebo>
 	<joint name="joint_structure" type="fixed">
@@ -90,5 +90,5 @@
 	</link>
 	<gazebo reference="cabinet_door">
-		<material>IPA/White</material>
+		<material>Gazebo/White</material>
 	</gazebo>
 	<joint name="joint_door" type="fixed">
@@ -118,5 +118,5 @@
 	</link>
 	<gazebo reference="knob1_link">
-		<material>IPA/Grey</material>
+		<material>Gazebo/Grey</material>
 	</gazebo>
 	<joint name="joint_knob1" type="fixed">
@@ -146,5 +146,5 @@
 	</link>
 	<gazebo reference="knob2_link">
-		<material>IPA/Grey</material>
+		<material>Gazebo/Grey</material>
 	</gazebo>
 	<joint name="joint_knob2" type="fixed">
@@ -174,5 +174,5 @@
 	</link>
 	<gazebo reference="knob3_link">
-		<material>IPA/Grey</material>
+		<material>Gazebo/Grey</material>
 	</gazebo>
 	<joint name="joint_knob3" type="fixed">
