Commit message: Fixed jumping milk box bug

File: cob_gazebo_worlds/objects/milk_box.urdf (robot description, URDF)
Before this commit: robot milk_box, 1 links, 0 joints
Links:
- link base_link: geometry collision box size=0.06 0.095 0.2; visual mesh filename=package://cob_gazebo_worlds/Media/models/milk_box.dae
