Commit message: New urdf models of the objects

File: cob_gazebo_objects/objects/jodsalz.urdf (robot description, URDF)
Before this commit: robot jodsalz, 1 links, 0 joints
Links:
- link base_link: geometry collision box size=0.061 0.046 0.144; visual mesh filename=package://cob_gazebo_objects/Media/models/jodsalz.dae

File: cob_gazebo_objects/objects/kraeuter.urdf (robot description, URDF)
Before this commit: robot kraeuter, 1 links, 0 joints
Links:
- link base_link: geometry collision box size=0.076 0.047 0.11; visual mesh filename=package://cob_gazebo_objects/Media/models/kraeuter.dae

File: cob_gazebo_objects/objects/tomaten_suppe.urdf (robot description, URDF)
Before this commit: robot tomaten_suppe, 1 links, 0 joints
Links:
- link base_link: geometry collision box size=0.093 0.032 0.126; visual mesh filename=package://cob_gazebo_objects/Media/models/tomaten_suppe.dae

File: cob_gazebo_objects/objects/zwieback.urdf (robot description, URDF)
Before this commit: robot zwieback, 1 links, 0 joints
Links:
- link base_link: geometry collision box size=0.142 0.076 0.144; visual mesh filename=package://cob_gazebo_objects/Media/models/zwieback.dae
