Commit message: New script spawn_object.py and config files

File: cob_gazebo_objects/objects/milk.urdf (robot description, URDF)
Before this commit: robot milk_box, 1 links, 0 joints
Links:
- link base_link: geometry collision box size=0.06 0.095 0.2; visual mesh filename=package://cob_gazebo_objects/Media/models/milk_box.dae

Commit message: Modifications in spawn_object.py, now support urdf.xacro files and rpy parameters

File: cob_gazebo_objects/objects/milk.urdf (robot description, URDF)
Before this commit: robot milk_box, 1 links, 0 joints
Links:
- removed link base_link
- added link box_body, mass 5.0; collision box size=0.06 0.095 0.2; visual mesh filename=package://cob_gazebo_objects/Media/models/milk_box.dae

Commit message: Rename objects

File: cob_gazebo_objects/objects/milk.urdf (robot description, URDF)
Before this commit: robot milk, 1 links, 0 joints
Links:
- link box_body: geometry collision box size=0.06 0.095 0.2; visual mesh filename=package://cob_gazebo_objects/Media/models/milk.dae

File: cob_gazebo_objects/objects/salt.urdf (robot description, URDF)
Before this commit: robot jodsalz, 1 links, 0 joints
Links:
- link base_link: geometry collision box size=0.061 0.046 0.144; visual mesh filename=package://cob_gazebo_objects/Media/models/salt.dae

File: cob_gazebo_objects/objects/tomato_sauce.urdf (robot description, URDF)
Before this commit: robot kraeuter, 1 links, 0 joints
Links:
- link base_link: geometry collision box size=0.076 0.047 0.11; visual mesh filename=package://cob_gazebo_objects/Media/models/tomato_sauce.dae

File: cob_gazebo_objects/objects/tomato_soup.urdf (robot description, URDF)
Before this commit: robot tomaten_suppe, 1 links, 0 joints
Links:
- link base_link: geometry collision box size=0.093 0.032 0.126; visual mesh filename=package://cob_gazebo_objects/Media/models/tomato_soup.dae

Commit message: Updated mass value for milk model

File: cob_gazebo_objects/objects/milk.urdf (robot description, URDF)
Before this commit: robot milk, 1 links, 0 joints
Links:
- link box_body: mass 5.0 -> 1.0
