Commit message: tomato_soup now uses mesh in collision tag

File: cob_gazebo_objects/objects/tomato_soup.urdf (robot description, URDF)
Before this commit: robot tomaten_suppe, 1 links, 0 joints
Links:
- link base_link: geometry collision mesh filename=package://cob_gazebo_objects/Media/models/tomato_soup.dae; visual mesh filename=package://cob_gazebo_objects/Media/models/tomato_soup.dae
