Commit message: Changed name medication_prospan to medicine_prospan and moved the default camera position

File: cob_gazebo_objects/objects/medicine_prospan.urdf (robot description, URDF)
Before this commit: robot my_object, 1 links, 0 joints
Links:
- link base_link: geometry collision box size=0.12 0.056 0.12; visual mesh filename=package://cob_gazebo_objects/Media/models/medicine_prospan.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
