Commit message: added people, move.py and changed model names

File: cob_gazebo_objects/objects/man_arm_raised.urdf (robot description, URDF)
Before this commit: robot my_object, 1 links, 0 joints
Links:
- link base_link: geometry collision mesh filename=package://cob_gazebo_objects/Media/models/man_arm_raised.dae; visual mesh filename=package://cob_gazebo_objects/Media/models/man_arm_raised.dae

File: cob_gazebo_objects/objects/man_resting_side.urdf (robot description, URDF)
Before this commit: robot my_object, 1 links, 0 joints
Links:
- link base_link: geometry collision mesh filename=package://cob_gazebo_objects/Media/models/man_resting_side.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; visual mesh filename=package://cob_gazebo_objects/Media/models/man_resting_side.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

File: cob_gazebo_objects/objects/man_walking.urdf (robot description, URDF)
Before this commit: robot my_object, 1 links, 0 joints
Links:
- link base_link: geometry collision mesh filename=package://cob_gazebo_objects/Media/models/man_walking.dae; visual mesh filename=package://cob_gazebo_objects/Media/models/man_walking.dae

Commit message: fix man urdfs

File: cob_gazebo_objects/objects/man_arm_raised.urdf (robot description, URDF)
Before this commit: robot my_object, 1 links, 0 joints
Links:
- link base_link: mass 1.37 -> 0.01; geometry collision mesh filename=package://cob_gazebo_objects/Media/models/man_arm_raised.stl; visual mesh filename=package://cob_gazebo_objects/Media/models/man_arm_raised.dae

File: cob_gazebo_objects/objects/man_resting_side.urdf (robot description, URDF)
Before this commit: robot my_object, 1 links, 0 joints
Links:
- link base_link: mass 1.37 -> 0.01

File: cob_gazebo_objects/objects/man_walking.urdf (robot description, URDF)
Before this commit: robot my_object, 1 links, 0 joints
Links:
- link base_link: mass 1.37 -> 0.01; geometry collision mesh filename=package://cob_gazebo_objects/Media/models/man_walking.stl; visual mesh filename=package://cob_gazebo_objects/Media/models/man_walking.dae
