Commit message: Added more objects and commented old object-spawning out for ipa-production-plant

File: cob_gazebo_objects/objects/machine4.urdf (robot description, URDF)
Before this commit: robot refridgerator, 1 links, 0 joints
Links:
- link base_link: geometry collision mesh filename=package://cob_gazebo_objects/Media/models/machine4.dae scale=1 1 1; visual mesh filename=package://cob_gazebo_objects/Media/models/machine4.dae scale=1 1 1

File: cob_gazebo_objects/objects/machine5.urdf (robot description, URDF)
Before this commit: robot refridgerator, 1 links, 0 joints
Links:
- link base_link: geometry collision mesh filename=package://cob_gazebo_objects/Media/models/machine5.dae scale=1 1 1; visual mesh filename=package://cob_gazebo_objects/Media/models/machine5.dae scale=1 1 1

File: cob_gazebo_worlds/urdf/ipa-production-plant/ipa-production-plant.urdf.xacro (robot description, xacro)
@@ -9,9 +9,9 @@
   <xacro:include filename="$(find cob_gazebo_worlds)/urdf/ipa-production-plant/warehouse.urdf.xacro" />
   <!-- machine-room -->
-  <xacro:include filename="$(find cob_gazebo_worlds)/urdf/ipa-production-plant/machine-room.urdf.xacro" />
+  <!-- <xacro:include filename="$(find cob_gazebo_worlds)/urdf/ipa-production-plant/machine-room.urdf.xacro" /> -->
   <!-- super-market -->
   <xacro:include filename="$(find cob_gazebo_worlds)/urdf/ipa-production-plant/super-market.urdf.xacro" />
   <!-- work-area -->
-  <xacro:include filename="$(find cob_gazebo_worlds)/urdf/ipa-production-plant/work-area.urdf.xacro" />
+  <!-- <xacro:include filename="$(find cob_gazebo_worlds)/urdf/ipa-production-plant/work-area.urdf.xacro" /> -->
   <!--macros-->
   <xacro:macro name="object" params="object_num *mesh *origin">
