Commit message: Updated the machine room of ipa-production-plant

File: cob_gazebo_objects/objects/assembly_area.urdf (robot description, URDF)
Before this commit: robot robot_arm, 1 links, 0 joints
Links:
- link base_link: geometry collision mesh filename=package://cob_gazebo_objects/Media/models/assembly_area.dae scale=1 1 1; visual mesh filename=package://cob_gazebo_objects/Media/models/assembly_area.dae scale=1 1 1

File: cob_gazebo_objects/objects/conveyor.urdf (robot description, URDF)
Before this commit: robot robot_arm, 1 links, 0 joints
Links:
- link base_link: geometry collision mesh filename=package://cob_gazebo_objects/Media/models/conveyor.dae scale=1 1 1; visual mesh filename=package://cob_gazebo_objects/Media/models/conveyor.dae scale=0.75 0.75 0.75

File: cob_gazebo_objects/objects/kanban.urdf (robot description, URDF)
Before this commit: robot robot_arm, 1 links, 0 joints
Links:
- link base_link: geometry collision mesh filename=package://cob_gazebo_objects/Media/models/kanban.dae scale=0.5 0.5 0.5; visual mesh filename=package://cob_gazebo_objects/Media/models/kanban.dae scale=0.5 0.5 0.5

File: cob_gazebo_objects/objects/robot_arm_mounted.urdf (robot description, URDF)
Before this commit: robot robot_arm, 1 links, 0 joints
Links:
- link base_link: geometry collision box size=1 1 0.5; collision mesh filename=package://cob_gazebo_objects/Media/models/robot_arm.dae scale=0.15 0.15 0.15
