Commit message: Changed some objects

File: cob_gazebo_objects/objects/conveyor.urdf (robot description, URDF)
Before this commit: robot conveyor, 1 links, 0 joints
Links:
- link base_link: geometry collision mesh filename=package://cob_gazebo_objects/Media/models/conveyor.dae scale=0.75 0.75 0.75; visual mesh filename=package://cob_gazebo_objects/Media/models/conveyor.dae scale=0.75 0.75 0.75
