Commit message: Updated model of ipa-office_walls

File: cob_gazebo_objects/objects/ipa-office_walls.urdf (robot description, URDF)
Before this commit: robot ipa-office_walls, 1 links, 0 joints
Links:
- link base_link: geometry collision mesh filename=package://cob_gazebo_objects/Media/models/ipa-office_walls.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; visual mesh filename=package://cob_gazebo_objects/Media/models/ipa-office_walls.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

Commit message: Set correct origin/scale for ipa-office_walls and added walls for stairway

File: cob_gazebo_objects/objects/ipa-office_walls.urdf (robot description, URDF)
Before this commit: robot ipa-office_walls, 1 links, 0 joints
Links:
- link base_link: geometry collision mesh filename=package://cob_gazebo_objects/Media/models/ipa-office_walls.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 scale=0.97 0.97 0.97; visual mesh filename=package://cob_gazebo_objects/Media/models/ipa-office_walls.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 scale=0.97 0.97 0.97
