Commit message: use latest xacro syntax

File: cob_gazebo_objects/objects/bookcase.urdf.xacro (robot description, xacro)
@@ -1,4 +1,5 @@
 <?xml version="1.0"?>
 <robot name="bookcase"
+	xmlns:xacro="http://www.ros.org/wiki/xacro"
 	xmlns:xi="http://www.w3.org/2001/XInclude"
 	xmlns:gazebo="http://playerstage.sourceforge.net/gazebo/xmlschema/#gz"
@@ -14,12 +15,12 @@
 	xmlns:physics="http://playerstage.sourceforge.net/gazebo/xmlschema/#physics"
 >
-  <property name="bookcase_height" value="0.79" />
-  <property name="bookcase_width" value="0.39" />
-  <property name="bookcase_depth" value="1.49" />
-  <property name="bookcase_x" value="0.98" />
-  <property name="bookcase_y" value="0.0" />
-  <property name="bookcase_z" value="0.0" />
-  <property name="bookcase_thickness_min" value="0.015"/>
-  <property name="bookcase_thickness_max" value="0.05"/>
+  <xacro:property name="bookcase_height" value="0.79" />
+  <xacro:property name="bookcase_width" value="0.39" />
+  <xacro:property name="bookcase_depth" value="1.49" />
+  <xacro:property name="bookcase_x" value="0.98" />
+  <xacro:property name="bookcase_y" value="0.0" />
+  <xacro:property name="bookcase_z" value="0.0" />
+  <xacro:property name="bookcase_thickness_min" value="0.015"/>
+  <xacro:property name="bookcase_thickness_max" value="0.05"/>
 <!-- dummy_link -->
 	<link name="dummy_link">
@@ -184,5 +185,5 @@
 	</joint>
 	<!--Separations-->
-    <macro name="separations" params="suffix parent pos">
+    <xacro:macro name="separations" params="suffix parent pos">
         <link name="separation_${suffix}_link">
             <inertial>
@@ -215,5 +216,5 @@
         <child link="separation_${suffix}_link" />
       </joint>
-  </macro>
+  </xacro:macro>
 	<separations suffix="1" parent="bookcase_top_link" pos="0 -${bookcase_thickness_min/2+0.3375} -${bookcase_thickness_max/2+0.3375/2}"/>
 	<separations suffix="2" parent="bookcase_top_link" pos="0 0 -${bookcase_thickness_max/2+0.3375/2}"/>

File: cob_gazebo_objects/objects/cabinet_with_door.urdf.xacro (robot description, xacro)
@@ -1,4 +1,5 @@
 <?xml version="1.0"?>
 <robot name="cabinet"
+	xmlns:xacro="http://www.ros.org/wiki/xacro"
 	xmlns:xi="http://www.w3.org/2001/XInclude"
 	xmlns:gazebo="http://playerstage.sourceforge.net/gazebo/xmlschema/#gz"
@@ -14,10 +15,10 @@
 	xmlns:physics="http://playerstage.sourceforge.net/gazebo/xmlschema/#physics"
 >
-  <property name="cabinet_height" value="1.06" />
-  <property name="cabinet_width" value="0.28" />
-  <property name="cabinet_depth" value="0.40" />
-  <property name="cabinet_x" value="1.5" />
-  <property name="cabinet_y" value="0.0" />
-  <property name="cabinet_z" value="0.0" />
+  <xacro:property name="cabinet_height" value="1.06" />
+  <xacro:property name="cabinet_width" value="0.28" />
+  <xacro:property name="cabinet_depth" value="0.40" />
+  <xacro:property name="cabinet_x" value="1.5" />
+  <xacro:property name="cabinet_y" value="0.0" />
+  <xacro:property name="cabinet_z" value="0.0" />
 <!-- dummy_link -->
 	<link name="dummy_link">

File: cob_gazebo_objects/objects/chair.urdf.xacro (robot description, xacro)
@@ -1,4 +1,5 @@
 <?xml version="1.0"?>
 <robot name="chair"
+       xmlns:xacro="http://www.ros.org/wiki/xacro"
        xmlns:xi="http://www.w3.org/2001/XInclude"
        xmlns:gazebo="http://playerstage.sourceforge.net/gazebo/xmlschema/#gz"
@@ -13,12 +14,12 @@
        xmlns:controller="http://playerstage.sourceforge.net/gazebo/xmlschema/#controller"
        xmlns:physics="http://playerstage.sourceforge.net/gazebo/xmlschema/#physics">
-  <property name="chair_height" value="0.45" />
-  <property name="chair_width" value="0.4" />
-  <property name="chair_depth" value="0.4" />
-  <property name="chair_y" value="0.0" />
-  <property name="chair_z" value="0.0" />
-  <property name="rest_height" value="0.5" />
-  <property name="chair_top_thickness" value="0.02"/>
-  <property name="M_PI" value="3.1415926535897931" />
+  <xacro:property name="chair_height" value="0.45" />
+  <xacro:property name="chair_width" value="0.4" />
+  <xacro:property name="chair_depth" value="0.4" />
+  <xacro:property name="chair_y" value="0.0" />
+  <xacro:property name="chair_z" value="0.0" />
+  <xacro:property name="rest_height" value="0.5" />
+  <xacro:property name="chair_top_thickness" value="0.02"/>
+  <xacro:property name="M_PI" value="3.1415926535897931" />
   <link name="chair_top_link">
     <inertial>
@@ -82,5 +83,5 @@
         <child link="chair_rest_link" />
       </joint>
-    <macro name="legs" params="suffix parent pos1 pos2">
+    <xacro:macro name="legs" params="suffix parent pos1 pos2">
         <link name="leg_${suffix}_link">
             <inertial>
@@ -113,5 +114,5 @@
         <child link="leg_${suffix}_link" />
       </joint>
-  </macro>
+  </xacro:macro>
         <legs suffix="left_front" parent="chair_top_link"  pos1="1" pos2="1"/>
 	<legs suffix="left_back" parent="chair_top_link"  pos1="-1" pos2="1"/>
@@ -149,5 +150,5 @@
         <child link="lath_${suffix}_link" />
       </joint>
-  </macro>
+  </xacro:macro>
         <structure_lath suffix="left_front" parent="chair_top_link"  pos1="1" pos2="0" box_size="0.02 0.77 0.07"/>
 	<structure_lath suffix="left_back" parent="chair_top_link"  pos1="-1" pos2="0" box_size="0.02 0.77 0.07"/>

File: cob_gazebo_objects/objects/table_ikea_bjursta.urdf.xacro (robot description, xacro)
@@ -1,4 +1,5 @@
 <?xml version="1.0"?>
 <robot name="table"
+       xmlns:xacro="http://www.ros.org/wiki/xacro"
        xmlns:xi="http://www.w3.org/2001/XInclude"
        xmlns:gazebo="http://playerstage.sourceforge.net/gazebo/xmlschema/#gz"
@@ -13,12 +14,12 @@
        xmlns:controller="http://playerstage.sourceforge.net/gazebo/xmlschema/#controller"
        xmlns:physics="http://playerstage.sourceforge.net/gazebo/xmlschema/#physics">
-  <property name="table_height" value="0.74" />
-  <property name="table_width" value="0.9" />
-  <property name="table_depth" value="0.9" />
-  <property name="table_x" value="0.98" />
-  <property name="table_y" value="0.0" />
-  <property name="table_z" value="0.0" />
-  <property name="table_top_thickness" value="0.04"/>
-  <property name="M_PI" value="3.1415926535897931" />
+  <xacro:property name="table_height" value="0.74" />
+  <xacro:property name="table_width" value="0.9" />
+  <xacro:property name="table_depth" value="0.9" />
+  <xacro:property name="table_x" value="0.98" />
+  <xacro:property name="table_y" value="0.0" />
+  <xacro:property name="table_z" value="0.0" />
+  <xacro:property name="table_top_thickness" value="0.04"/>
+  <xacro:property name="M_PI" value="3.1415926535897931" />
   <link name="table_top_link">
     <inertial>
@@ -49,5 +50,5 @@
     <kd>1.0</kd>
   </gazebo>
-    <macro name="legs" params="suffix parent pos1 pos2">
+    <xacro:macro name="legs" params="suffix parent pos1 pos2">
         <link name="leg_${suffix}_link">
             <inertial>
@@ -80,10 +81,10 @@
         <child link="leg_${suffix}_link" />
       </joint>
-  </macro>
+  </xacro:macro>
         <legs suffix="left_front" parent="table_top_link"  pos1="1" pos2="1"/>
 	<legs suffix="left_back" parent="table_top_link"  pos1="-1" pos2="1"/>
         <legs suffix="right_front" parent="table_top_link"  pos1="1" pos2="-1"/>
 	<legs suffix="right_back" parent="table_top_link"  pos1="-1" pos2="-1"/>
- <macro name="structure_lath" params="suffix parent pos1 pos2 box_size">
+ <xacro:macro name="structure_lath" params="suffix parent pos1 pos2 box_size">
         <link name="lath_${suffix}_link">
             <inertial>
@@ -116,5 +117,5 @@
         <child link="lath_${suffix}_link" />
       </joint>
-  </macro>
+  </xacro:macro>
         <structure_lath suffix="left_front" parent="table_top_link"  pos1="1" pos2="0" box_size="0.02 0.77 0.07"/>
 	<structure_lath suffix="left_back" parent="table_top_link"  pos1="-1" pos2="0" box_size="0.02 0.77 0.07"/>

File: cob_gazebo_worlds/urdf/automotive-assembly-line/automotive-assembly-line.urdf.xacro (robot description, xacro)
@@ -21,5 +21,5 @@
     <inertial>
       <mass value="${mass}" />
-      <insert_block name="origin" />
+      <xacro:insert_block name="origin" />
       <inertia ixx="${0.0833333 * mass * (y*y + z*z)}" ixy="0.0" ixz="0.0"
           iyy="${0.0833333 * mass * (x*x + z*z)}" iyz="0.0"
@@ -57,5 +57,5 @@
         <origin xyz="0 0 0" rpy="0 0 0"/>
         <geometry>
-          <insert_block name = "mesh"/>
+          <xacro:insert_block name = "mesh"/>
         </geometry>
       </visual>
@@ -63,5 +63,5 @@
         <origin xyz="0 0 0" rpy="0 0 0"/>
         <geometry>
-          <insert_block name = "mesh"/>
+          <xacro:insert_block name = "mesh"/>
         </geometry>
       </collision>
@@ -72,5 +72,5 @@
     </gazebo>
     <joint name="bin_joint_${new_object_num}" type="fixed">
-       <insert_block name="origin"/>
+       <xacro:insert_block name="origin"/>
        <parent link="belt_base_link"/>
        <child link="world_object_${new_object_num}"/>

File: cob_gazebo_worlds/urdf/common.xacro (robot description, xacro)
@@ -1,10 +1,10 @@
 <?xml version="1.0"?>
 <robot xmlns:xacro="http://www.ros.org/wiki/xacro">
-  <property name="M_PI" value="3.1415926535897931" />
+  <xacro:property name="M_PI" value="3.1415926535897931" />
   <!-- see https://secure.wikimedia.org/wikipedia/en/wiki/List_of_moment_of_inertia_tensors -->
   <xacro:macro name="sphere_inertial" params="radius mass *origin">
     <inertial>
       <mass value="${mass}" />
-      <insert_block name="origin" />
+      <xacro:insert_block name="origin" />
       <inertia ixx="${0.4 * mass * radius * radius}" ixy="0.0" ixz="0.0"
         iyy="${0.4 * mass * radius * radius}" iyz="0.0"
@@ -15,5 +15,5 @@
     <inertial>
       <mass value="${mass}" />
-      <insert_block name="origin" />
+      <xacro:insert_block name="origin" />
       <inertia ixx="${0.0833333 * mass * (3 * radius * radius + length * length)}" ixy="0.0" ixz="0.0"
         iyy="${0.0833333 * mass * (3 * radius * radius + length * length)}" iyz="0.0"
@@ -24,5 +24,5 @@
     <inertial>
       <mass value="${mass}" />
-      <insert_block name="origin" />
+      <xacro:insert_block name="origin" />
       <inertia ixx="${0.0833333 * mass * (y*y + z*z)}" ixy="0.0" ixz="0.0"
         iyy="${0.0833333 * mass * (x*x + z*z)}" iyz="0.0"

File: cob_gazebo_worlds/urdf/ipa-apartment/ipa-apartment.urdf.xacro (robot description, xacro)
@@ -19,17 +19,17 @@
   <xacro:include filename="$(find cob_gazebo_worlds)/urdf/ipa-apartment/wall_ipa.urdf.xacro" />
   <!--Parameters-->
-  <property name="dist_axis_x" value="1.969" />
-  <property name="dist_axis_y" value="4.070" />
-  <property name="size_total_x" value="8.0" />
-  <property name="size_total_y" value="11.2" />
-  <property name="size_a" value="4.7" />
-  <property name="size_b" value="8.2" />
-  <property name="size_c" value="1.8" />
-  <property name="size_d" value="4.16" />
-  <property name="wall_depth" value="0.1" />
-  <property name="window_depth" value="0.15" />
-  <property name="size_z_wall1" value="2.7" />
-  <property name="size_z_wall2" value="2.7" />
-  <property name="size_z_wall3" value="2.7" />
+  <xacro:property name="dist_axis_x" value="1.969" />
+  <xacro:property name="dist_axis_y" value="4.070" />
+  <xacro:property name="size_total_x" value="8.0" />
+  <xacro:property name="size_total_y" value="11.2" />
+  <xacro:property name="size_a" value="4.7" />
+  <xacro:property name="size_b" value="8.2" />
+  <xacro:property name="size_c" value="1.8" />
+  <xacro:property name="size_d" value="4.16" />
+  <xacro:property name="wall_depth" value="0.1" />
+  <xacro:property name="window_depth" value="0.15" />
+  <xacro:property name="size_z_wall1" value="2.7" />
+  <xacro:property name="size_z_wall2" value="2.7" />
+  <xacro:property name="size_z_wall3" value="2.7" />
   <xacro:macro name="ipa-apartment" params="name">
     <gazebo>

File: cob_gazebo_worlds/urdf/ipa-apartment/landing.urdf.xacro (robot description, xacro)
@@ -6,5 +6,5 @@
   </link>
   <joint name="joint_origin_landing" type="fixed">
-    <insert_block name="origin" />
+    <xacro:insert_block name="origin" />
     <parent link="${parent}"/>
     <child link="origin_landing" />

File: cob_gazebo_worlds/urdf/ipa-production-plant/ipa-production-plant.property.xacro (robot description, xacro)
@@ -2,30 +2,30 @@
 <robot xmlns:xacro="http://www.ros.org/wiki/xacro">
   <!--properties-->
-  <property name="wall_depth" value="0.1" />
-  <property name="wall_height" value="5" />
-  <property name="gate_size" value="3" />
-  <property name="room1_w1" value="9.5" />
-  <property name="room1_w2" value="9.5" />
-  <property name="room1_w3" value="24" />
-  <property name="room2_w1" value="22.5" />
-  <property name="room2_w2" value="21" />
-  <property name="room3_w1" value="24" />
-  <property name="room3_w2" value="22" />
-  <property name="room4_w1" value="36" />
-  <property name="room4_w2" value="21" /> 24
-  <property name="room4_w3" value="11.25" />
-  <property name="room4_w4" value="7.5" />
-  <property name="room1_room2_w1" value="10.5" />
-  <property name="room1_room3_w1" value="9.5" />
-  <property name="room2_room4_w1" value="11.25" />
-  <property name="room3_room4_w1" value="17" />
-  <property name="room3_room4_w2" value="4" />
-  <property name="hallway_w1" value="26" />
-  <property name="hallway_w2" value="58" />
-  <property name="hallway_w3" value="5" />
-  <property name="hallway2_w1" value="3" />
-  <property name="hallway2_w2" value="53" />
-  <property name="position_offset_x" value="-20" />
-  <property name="position_offset_y" value="-35" />
-  <property name="position_offset_z" value="0" />
+  <xacro:property name="wall_depth" value="0.1" />
+  <xacro:property name="wall_height" value="5" />
+  <xacro:property name="gate_size" value="3" />
+  <xacro:property name="room1_w1" value="9.5" />
+  <xacro:property name="room1_w2" value="9.5" />
+  <xacro:property name="room1_w3" value="24" />
+  <xacro:property name="room2_w1" value="22.5" />
+  <xacro:property name="room2_w2" value="21" />
+  <xacro:property name="room3_w1" value="24" />
+  <xacro:property name="room3_w2" value="22" />
+  <xacro:property name="room4_w1" value="36" />
+  <xacro:property name="room4_w2" value="21" /> 24
+  <xacro:property name="room4_w3" value="11.25" />
+  <xacro:property name="room4_w4" value="7.5" />
+  <xacro:property name="room1_room2_w1" value="10.5" />
+  <xacro:property name="room1_room3_w1" value="9.5" />
+  <xacro:property name="room2_room4_w1" value="11.25" />
+  <xacro:property name="room3_room4_w1" value="17" />
+  <xacro:property name="room3_room4_w2" value="4" />
+  <xacro:property name="hallway_w1" value="26" />
+  <xacro:property name="hallway_w2" value="58" />
+  <xacro:property name="hallway_w3" value="5" />
+  <xacro:property name="hallway2_w1" value="3" />
+  <xacro:property name="hallway2_w2" value="53" />
+  <xacro:property name="position_offset_x" value="-20" />
+  <xacro:property name="position_offset_y" value="-35" />
+  <xacro:property name="position_offset_z" value="0" />
 </robot>
