Commit message: Fixed some walls in ipa_office

File: cob_gazebo_worlds/urdf/ipa-apartment/office.urdf.xacro (robot description, xacro)
@@ -97,12 +97,12 @@
 			<origin xyz="0 0 0" />
 			<geometry>
-				<box size="${wall_depth} 8.2 ${size_z_wall3}" />
-			</geometry>
-			<material name="Grey"/>
-		</visual>
-		<collision>
-			<origin xyz="0 0 0" />
-			<geometry>
-				<box size="${wall_depth} 8.2 ${size_z_wall3}" />
+				<box size="${wall_depth} 8.2 ${size_z_wall2}" />
+			</geometry>
+			<material name="Grey"/>
+		</visual>
+		<collision>
+			<origin xyz="0 0 0" />
+			<geometry>
+				<box size="${wall_depth} 8.2 ${size_z_wall2}" />
 			</geometry>
 		</collision>
@@ -112,5 +112,5 @@
 	</gazebo>
 	<joint name="joint_wall_office_02" type="fixed">
-		<origin xyz="5.6 0 ${size_z_wall3/2}" rpy="0 0 0" />
+		<origin xyz="5.6 0 ${size_z_wall2/2}" rpy="0 0 0" />
 		<parent link="origin_office" />
 		<child link="wall_office_02" />
@@ -126,12 +126,12 @@
 			<origin xyz="0 0 0" />
 			<geometry>
-				<box size="${wall_depth} 8.2 ${size_z_wall3}" />
-			</geometry>
-			<material name="Grey"/>
-		</visual>
-		<collision>
-			<origin xyz="0 0 0" />
-			<geometry>
-				<box size="${wall_depth} 8.2 ${size_z_wall3}" />
+				<box size="${wall_depth} 8.2 ${size_z_wall2}" />
+			</geometry>
+			<material name="Grey"/>
+		</visual>
+		<collision>
+			<origin xyz="0 0 0" />
+			<geometry>
+				<box size="${wall_depth} 8.2 ${size_z_wall2}" />
 			</geometry>
 		</collision>
@@ -141,5 +141,5 @@
 	</gazebo>
 	<joint name="joint_wall_office_03" type="fixed">
-		<origin xyz="-5.6 0 ${size_z_wall3/2}" rpy="0 0 0" />
+		<origin xyz="-5.6 0 ${size_z_wall2/2}" rpy="0 0 0" />
 		<parent link="origin_office" />
 		<child link="wall_office_03" />
@@ -155,12 +155,12 @@
 			<origin xyz="0 0 0" />
 			<geometry>
-				<box size="11.2 ${wall_depth} ${size_z_wall3}" />
-			</geometry>
-			<material name="Grey"/>
-		</visual>
-		<collision>
-			<origin xyz="0 0 0" />
-			<geometry>
-				<box size="11.2 ${wall_depth} ${size_z_wall3}" />
+				<box size="11.2 ${wall_depth} ${size_z_wall2}" />
+			</geometry>
+			<material name="Grey"/>
+		</visual>
+		<collision>
+			<origin xyz="0 0 0" />
+			<geometry>
+				<box size="11.2 ${wall_depth} ${size_z_wall2}" />
 			</geometry>
 		</collision>
@@ -170,5 +170,5 @@
 	</gazebo>
 	<joint name="joint_wall_office_04" type="fixed">
-		<origin xyz="0 4 ${size_z_wall3/2}" rpy="0 0 0" />
+		<origin xyz="0 4 ${size_z_wall2/2}" rpy="0 0 0" />
 		<parent link="origin_office" />
 		<child link="wall_office_04" />
@@ -184,12 +184,12 @@
 			<origin xyz="0 0 0" />
 			<geometry>
-				<box size="${wall_depth} 4.51 ${size_z_wall3}" />
-			</geometry>
-			<material name="Grey"/>
-		</visual>
-		<collision>
-			<origin xyz="0 0 0" />
-			<geometry>
-				<box size="${wall_depth} 4.51 ${size_z_wall3}" />
+				<box size="${wall_depth} 4.51 ${size_z_wall1}" />
+			</geometry>
+			<material name="Grey"/>
+		</visual>
+		<collision>
+			<origin xyz="0 0 0" />
+			<geometry>
+				<box size="${wall_depth} 4.51 ${size_z_wall1}" />
 			</geometry>
 		</collision>
@@ -199,5 +199,5 @@
 	</gazebo>
 	<joint name="joint_wall_office_05" type="fixed">
-		<origin xyz="1.09 -0.615 ${size_z_wall3/2}" rpy="0 0 0" />
+		<origin xyz="1.09 -0.615 ${size_z_wall1/2}" rpy="0 0 0" />
 		<parent link="origin_office" />
 		<child link="wall_office_05" />
@@ -213,12 +213,12 @@
 			<origin xyz="0 0 0" />
 			<geometry>
-				<box size="${wall_depth} 1.23 ${size_z_wall3}" />
-			</geometry>
-			<material name="Grey"/>
-		</visual>
-		<collision>
-			<origin xyz="0 0 0" />
-			<geometry>
-				<box size="${wall_depth} 1.23 ${size_z_wall3}" />
+				<box size="${wall_depth} 1.23 ${size_z_wall1}" />
+			</geometry>
+			<material name="Grey"/>
+		</visual>
+		<collision>
+			<origin xyz="0 0 0" />
+			<geometry>
+				<box size="${wall_depth} 1.23 ${size_z_wall1}" />
 			</geometry>
 		</collision>
@@ -228,5 +228,5 @@
 	</gazebo>
 	<joint name="joint_wall_office_06" type="fixed">
-		<origin xyz="1.09 3.385 ${size_z_wall3/2}" rpy="0 0 0" />
+		<origin xyz="1.09 3.385 ${size_z_wall1/2}" rpy="0 0 0" />
 		<parent link="origin_office" />
 		<child link="wall_office_06" />
@@ -242,12 +242,12 @@
 			<origin xyz="0 0 0" />
 			<geometry>
-				<box size="${wall_depth} 4.01 ${size_z_wall3}" />
-			</geometry>
-			<material name="Grey"/>
-		</visual>
-		<collision>
-			<origin xyz="0 0 0" />
-			<geometry>
-				<box size="${wall_depth} 4.01 ${size_z_wall3}" />
+				<box size="${wall_depth} 4.01 ${size_z_wall1}" />
+			</geometry>
+			<material name="Grey"/>
+		</visual>
+		<collision>
+			<origin xyz="0 0 0" />
+			<geometry>
+				<box size="${wall_depth} 4.01 ${size_z_wall1}" />
 			</geometry>
 		</collision>
@@ -257,5 +257,5 @@
 	</gazebo>
 	<joint name="joint_wall_office_07" type="fixed">
-		<origin xyz="-1.09 2 ${size_z_wall3/2}" rpy="0 0 0" />
+		<origin xyz="-1.09 2 ${size_z_wall1/2}" rpy="0 0 0" />
 		<parent link="origin_office" />
 		<child link="wall_office_07" />
@@ -271,12 +271,12 @@
 			<origin xyz="0 0 0" />
 			<geometry>
-				<box size="${wall_depth} 1.73 ${size_z_wall3}" />
-			</geometry>
-			<material name="Grey"/>
-		</visual>
-		<collision>
-			<origin xyz="0 0 0" />
-			<geometry>
-				<box size="${wall_depth} 1.73 ${size_z_wall3}" />
+				<box size="${wall_depth} 1.73 ${size_z_wall1}" />
+			</geometry>
+			<material name="Grey"/>
+		</visual>
+		<collision>
+			<origin xyz="0 0 0" />
+			<geometry>
+				<box size="${wall_depth} 1.73 ${size_z_wall1}" />
 			</geometry>
 		</collision>
@@ -286,5 +286,5 @@
 	</gazebo>
 	<joint name="joint_wall_office_08" type="fixed">
-		<origin xyz="-1.09 -2 ${size_z_wall3/2}" rpy="0 0 0" />
+		<origin xyz="-1.09 -2 ${size_z_wall1/2}" rpy="0 0 0" />
 		<parent link="origin_office" />
 		<child link="wall_office_08" />
@@ -300,12 +300,12 @@
 			<origin xyz="0 0 0" />
 			<geometry>
-				<box size="4.5 ${wall_depth} ${size_z_wall3}" />
-			</geometry>
-			<material name="Grey"/>
-		</visual>
-		<collision>
-			<origin xyz="0 0 0" />
-			<geometry>
-				<box size="4.5 ${wall_depth} ${size_z_wall3}" />
+				<box size="4.5 ${wall_depth} ${size_z_wall1}" />
+			</geometry>
+			<material name="Grey"/>
+		</visual>
+		<collision>
+			<origin xyz="0 0 0" />
+			<geometry>
+				<box size="4.5 ${wall_depth} ${size_z_wall1}" />
 			</geometry>
 		</collision>
@@ -315,5 +315,5 @@
 	</gazebo>
 	<joint name="joint_wall_office_09" type="fixed">
-		<origin xyz="3.35 1.64 ${size_z_wall3/2}" rpy="0 0 0" />
+		<origin xyz="3.35 1.64 ${size_z_wall1/2}" rpy="0 0 0" />
 		<parent link="origin_office" />
 		<child link="wall_office_09" />
@@ -329,12 +329,12 @@
 			<origin xyz="0 0 0" />
 			<geometry>
-				<box size="4.5 ${wall_depth} ${size_z_wall3}" />
-			</geometry>
-			<material name="Grey"/>
-		</visual>
-		<collision>
-			<origin xyz="0 0 0" />
-			<geometry>
-				<box size="4.5 ${wall_depth} ${size_z_wall3}" />
+				<box size="4.5 ${wall_depth} ${size_z_wall1}" />
+			</geometry>
+			<material name="Grey"/>
+		</visual>
+		<collision>
+			<origin xyz="0 0 0" />
+			<geometry>
+				<box size="4.5 ${wall_depth} ${size_z_wall1}" />
 			</geometry>
 		</collision>
@@ -344,5 +344,5 @@
 	</gazebo>
 	<joint name="joint_wall_office_10" type="fixed">
-		<origin xyz="-3.35 -1.14 ${size_z_wall3/2}" rpy="0 0 0" />
+		<origin xyz="-3.35 -1.14 ${size_z_wall1/2}" rpy="0 0 0" />
 		<parent link="origin_office" />
 		<child link="wall_office_10" />
