Commit message: Simulation model for 3rd flor and visualiced in rviz

File: cob_gazebo_worlds/urdf/ipa-apartment/apartment.urdf.xacro (robot description, xacro)
@@ -17,4 +17,5 @@
 				<box size="${wall_depth} ${size_d} ${size_z_wall1}" />
 			</geometry>
+			<material name="Grey"/>
 		</visual>
 		<collision>
@@ -45,4 +46,5 @@
 				<box size=" ${size_b} ${window_depth} ${size_z_wall2}" />
 			</geometry>
+			<material name="Grey"/>
 		</visual>
 		<collision>
@@ -73,4 +75,5 @@
 				<box size="${wall_depth} ${size_a} ${size_z_wall2}" />
 			</geometry>
+			<material name="Grey"/>
 		</visual>
 		<collision>
@@ -101,4 +104,5 @@
 				<box size=" ${window_depth} 1.6 ${size_z_wall2}" />
 			</geometry>
+			<material name="Grey"/>
 		</visual>
 		<collision>
@@ -129,4 +133,5 @@
 				<box size="${window_depth} 1.55 ${size_z_wall2}" />
 			</geometry>
+			<material name="Grey"/>
 		</visual>
 		<collision>
@@ -157,4 +162,5 @@
 				<box size="${wall_depth} ${size_a} ${size_z_wall2}" />
 			</geometry>
+			<material name="Grey"/>
 		</visual>
 		<collision>
@@ -185,4 +191,5 @@
 				<box size=" ${size_b} ${window_depth} ${size_z_wall2}" />
 			</geometry>
+			<material name="Grey"/>
 		</visual>
 		<collision>
@@ -213,4 +220,5 @@
 				<box size="${wall_depth} ${size_a} ${size_z_wall1}" />
 			</geometry>
+			<material name="Grey"/>
 		</visual>
 		<collision>
@@ -241,4 +249,5 @@
 				<box size="${wall_depth} 1.9 ${size_z_wall2}" />
 			</geometry>
+			<material name="Grey"/>
 		</visual>
 		<collision>
@@ -269,4 +278,5 @@
 				<box size="0.04 0.62 ${size_z_wall1}" />
 			</geometry>
+			<material name="Transparent"/>
 		</visual>
 		<collision>
@@ -297,4 +307,5 @@
 				<box size="0.04 0.62 ${size_z_wall1}" />
 			</geometry>
+			<material name="Transparent"/>
 		</visual>
 		<collision>

File: cob_gazebo_worlds/urdf/ipa-apartment/cabinets.urdf.xacro (robot description, xacro)
@@ -17,4 +17,5 @@
 				<box size="1.15 0.55 2.40" />
 			</geometry>
+			<material name="LightBlue"/>
 		</visual>
 		<collision>
@@ -44,4 +45,5 @@
 				<box size="1.15 0.55 2.40" />
 			</geometry>
+			<material name="LightBlue"/>
 		</visual>
 		<collision>
@@ -71,4 +73,5 @@
 				<box size="1.15 0.55 2.40" />
 			</geometry>
+			<material name="LightBlue"/>
 		</visual>
 		<collision>
@@ -98,4 +101,5 @@
 				<box size="0.36 0.36 ${size_z_wall1}" />
 			</geometry>
+			<material name="LightBlue"/>
 		</visual>
 		<collision>

File: cob_gazebo_worlds/urdf/ipa-apartment/elevator.urdf.xacro (robot description, xacro)
@@ -5,4 +5,28 @@
        xmlns:xacro="http://ros.org/wiki/xacro">
         <xacro:macro name="elevator" params="name">
+	<link name="origin_elevator">
+		<inertial>
+			<origin xyz="0 0 0" />
+			<mass value="0.0" />
+			<inertia ixx="0.0" ixy="0.0" ixz="0.0" iyy="0.0" iyz="0.0" izz="0.0" />
+		</inertial>
+		<visual>
+			<origin xyz="0 0 0" />
+			<geometry>
+				<box size="0 0 0" />
+			</geometry>
+		</visual>
+		<collision>
+			<origin xyz="0 0 0" />
+			<geometry>
+				<box size="0 0 0" />
+			</geometry>
+		</collision>
+	</link>
+	<joint name="joint_origin_elevator" type="fixed">
+		<origin xyz="3.15 -3.15 ${size_z_wall1/2}" rpy="0 0 -0.7853981" />
+        <parent link="origin_landing"/>
+		<child link="origin_elevator" />
+	</joint>
 	<!-- elevator 1 -->
 	<link name="elevator_left">
@@ -17,4 +41,5 @@
 				<box size="0.04 0.87 ${size_z_wall1}" />
 			</geometry>
+			<material name="LightBlue"/>
 		</visual>
 		<collision>
@@ -28,13 +53,13 @@
 		<material>IPA/Wall2</material>
 	</gazebo>
-	<joint name="joint_elevator_left" type="prismatic">
+	<joint name="elevator_left_joint" type="prismatic">
+		<origin xyz="0 1.085 0" rpy="0 0 0" />
+		<parent link="origin_elevator" />
+		<child link="elevator_left" />
 		<axis xyz = "0 1 0"/>
-		<origin xyz="${-size_total_x/2+dist_axis_x-wall_depth-4.6-1.6} ${-0.68-dist_axis_y-1.68} ${size_z_wall1/2}" rpy="0 0 -0.7853" />
-		<parent link="dummy_link" />
-		<child link="elevator_left" />
 		<calibration rising="0.0"/>
 		<dynamics damping="0.0" friction="0.0"/>
 		<limit effort="100" velocity="1.0" lower="0" upper="0.87" />
-		<safety_controller k_velocity="10"/>
+		<!--safety_controller k_velocity="10"/-->
 	</joint>
          <transmission name="elevator_left_trans" type="pr2_mechanism_model/SimpleTransmission">
@@ -42,60 +67,62 @@
                    <joint name="elevator_left_joint"/>
                    <mechanicalReduction>1</mechanicalReduction>
-                </transmission>
-	<!-- wall ext5 -->
-	<link name="wall_ext5">
-		<inertial>
-			<origin xyz="0 0 0" />
-			<mass value="5.0" />
-			<inertia ixx="0.0" ixy="0.0" ixz="0.0" iyy="0.0" iyz="0.0" izz="0.0" />
-		</inertial>
-		<visual>
-			<origin xyz="0 0 0" />
-			<geometry>
-				<box size="2.4 0.04 ${size_z_wall1}" />
-			</geometry>
-		</visual>
-		<collision>
-			<origin xyz="0 0 0" />
-			<geometry>
-				<box size="2.4 0.04 ${size_z_wall1}" />
-			</geometry>
-		</collision>
-	</link>
-	<gazebo reference="wall_ext5">
-		<material>IPA/WallApartment</material>
-	</gazebo>
-	<joint name="joint_wall_ext5" type="fixed">
-		<origin xyz="${-size_total_x/2+dist_axis_x-wall_depth-5.1} ${-0.68-dist_axis_y-0.65-1.5} ${size_z_wall1/2}" rpy="0 0 -0.7853" />
-		<parent link="dummy_link" />
-		<child link="wall_ext5" />
-	</joint>
-	<!-- wall ext6 -->
-	<link name="wall_ext6">
-		<inertial>
-			<origin xyz="0 0 0" />
-			<mass value="5.0" />
-			<inertia ixx="0.0" ixy="0.0" ixz="0.0" iyy="0.0" iyz="0.0" izz="0.0" />
-		</inertial>
-		<visual>
-			<origin xyz="0 0 0" />
-			<geometry>
-				<box size="2.4 0.04 ${size_z_wall1}" />
-			</geometry>
-		</visual>
-		<collision>
-			<origin xyz="0 0 0" />
-			<geometry>
-				<box size="2.4 0.04 ${size_z_wall1}" />
-			</geometry>
-		</collision>
-	</link>
-	<gazebo reference="wall_ext6">
-		<material>IPA/WallApartment</material>
-	</gazebo>
-	<joint name="joint_wall_ext6" type="fixed">
-		<origin xyz="${-size_total_x/2+dist_axis_x-wall_depth-5.1-0.615} ${-0.68-dist_axis_y-0.65-1.5-0.615} ${size_z_wall1/2}" rpy="0 0 -0.7853" />
-		<parent link="dummy_link" />
-		<child link="wall_ext6" />
+         </transmission>
+	<!-- wall elv5 -->
+	<link name="wall_elv5">
+		<inertial>
+			<origin xyz="0 0 0" />
+			<mass value="5.0" />
+			<inertia ixx="0.0" ixy="0.0" ixz="0.0" iyy="0.0" iyz="0.0" izz="0.0" />
+		</inertial>
+		<visual>
+			<origin xyz="0 0 0" />
+			<geometry>
+				<box size="2.4 0.04 ${size_z_wall1}" />
+			</geometry>
+			<material name="Grey"/>
+		</visual>
+		<collision>
+			<origin xyz="0 0 0" />
+			<geometry>
+				<box size="2.4 0.04 ${size_z_wall1}" />
+			</geometry>
+		</collision>
+	</link>
+	<gazebo reference="wall_elv5">
+		<material>IPA/WallApartment</material>
+	</gazebo>
+	<joint name="joint_wall_elv5" type="fixed">
+		<origin xyz="1.2 1.52 0" rpy="0 0 0" />
+		<parent link="origin_elevator" />
+		<child link="wall_elv5" />
+	</joint>
+	<!-- wall elv6 -->
+	<link name="wall_elv6">
+		<inertial>
+			<origin xyz="0 0 0" />
+			<mass value="5.0" />
+			<inertia ixx="0.0" ixy="0.0" ixz="0.0" iyy="0.0" iyz="0.0" izz="0.0" />
+		</inertial>
+		<visual>
+			<origin xyz="0 0 0" />
+			<geometry>
+				<box size="2.4 0.04 ${size_z_wall1}" />
+			</geometry>
+			<material name="Grey"/>
+		</visual>
+		<collision>
+			<origin xyz="0 0 0" />
+			<geometry>
+				<box size="2.4 0.04 ${size_z_wall1}" />
+			</geometry>
+		</collision>
+	</link>
+	<gazebo reference="wall_elv6">
+		<material>IPA/WallApartment</material>
+	</gazebo>
+	<joint name="joint_wall_elv6" type="fixed">
+		<origin xyz="1.2 0.65 0" rpy="0 0 0" />
+		<parent link="origin_elevator" />
+		<child link="wall_elv6" />
 	</joint>
 	<!-- elevator_left2  -->
@@ -111,4 +138,5 @@
 				<box size="0.04 0.87 ${size_z_wall1}" />
 			</geometry>
+			<material name="Grey"/>
 		</visual>
 		<collision>
@@ -123,6 +151,6 @@
 	</gazebo>
 	<joint name="joint_elevator_left2" type="fixed">
-		<origin xyz="${-size_total_x/2+dist_axis_x-wall_depth-1.6-3} ${-0.68-dist_axis_y-1.68-1.6} ${size_z_wall1/2}" rpy="0 0 -0.7853" />
-		<parent link="dummy_link" />
+		<origin xyz="2.4 1.085 0" rpy="0 0 0" />
+		<parent link="origin_elevator" />
 		<child link="elevator_left2" />
 	</joint>
@@ -139,4 +167,5 @@
 				<box size="0.04 0.87 ${size_z_wall1}" />
 			</geometry>
+			<material name="LightBlue"/>
 		</visual>
 		<collision>
@@ -150,8 +179,8 @@
 		<material>IPA/Wall2</material>
 	</gazebo>
-	<joint name="joint_elevator_right" type="prismatic">
+	<joint name="elevator_right_joint" type="prismatic">
 		<axis xyz = "0 -1 0"/>
-		<origin xyz="${-size_total_x/2+dist_axis_x-wall_depth-4.6-1.6-1.15} ${-0.68-dist_axis_y-1.68-1.15} ${size_z_wall1/2}" rpy="0 0 -0.7853" />
-		<parent link="dummy_link" />
+		<origin xyz="0 -1.085 0" rpy="0 0 0" />
+		<parent link="origin_elevator" />
 		<child link="elevator_right" />
 		<calibration rising="0.0"/>
@@ -164,60 +193,62 @@
                    <joint name="elevator_right_joint"/>
                    <mechanicalReduction>1</mechanicalReduction>
-                </transmission>
-	<!-- wall ext7 -->
-	<link name="wall_ext7">
-		<inertial>
-			<origin xyz="0 0 0" />
-			<mass value="5.0" />
-			<inertia ixx="0.0" ixy="0.0" ixz="0.0" iyy="0.0" iyz="0.0" izz="0.0" />
-		</inertial>
-		<visual>
-			<origin xyz="0 0 0" />
-			<geometry>
-				<box size="2.4 0.04 ${size_z_wall1}" />
-			</geometry>
-		</visual>
-		<collision>
-			<origin xyz="0 0 0" />
-			<geometry>
-				<box size="2.4 0.04 ${size_z_wall1}" />
-			</geometry>
-		</collision>
-	</link>
-	<gazebo reference="wall_ext7">
-		<material>IPA/WallApartment</material>
-	</gazebo>
-	<joint name="joint_wall_ext7" type="fixed">
-		<origin xyz="${-size_total_x/2+dist_axis_x-wall_depth-5.1-1.15} ${-0.68-dist_axis_y-0.65-1.5-1.15} ${size_z_wall1/2}" rpy="0 0 -0.7853" />
-		<parent link="dummy_link" />
-		<child link="wall_ext7" />
-	</joint>
-	<!-- wall ext8 -->
-	<link name="wall_ext8">
-		<inertial>
-			<origin xyz="0 0 0" />
-			<mass value="5.0" />
-			<inertia ixx="0.0" ixy="0.0" ixz="0.0" iyy="0.0" iyz="0.0" izz="0.0" />
-		</inertial>
-		<visual>
-			<origin xyz="0 0 0" />
-			<geometry>
-				<box size="2.4 0.04 ${size_z_wall1}" />
-			</geometry>
-		</visual>
-		<collision>
-			<origin xyz="0 0 0" />
-			<geometry>
-				<box size="2.4 0.04 ${size_z_wall1}" />
-			</geometry>
-		</collision>
-	</link>
-	<gazebo reference="wall_ext8">
-		<material>IPA/WallApartment</material>
-	</gazebo>
-	<joint name="joint_wall_ext8" type="fixed">
-		<origin xyz="${-size_total_x/2+dist_axis_x-wall_depth-5.1-1.78} ${-0.68-dist_axis_y-0.65-1.5-1.78} ${size_z_wall1/2}" rpy="0 0 -0.7853" />
-		<parent link="dummy_link" />
-		<child link="wall_ext8" />
+        </transmission>
+	<!-- wall elv7 -->
+	<link name="wall_elv7">
+		<inertial>
+			<origin xyz="0 0 0" />
+			<mass value="5.0" />
+			<inertia ixx="0.0" ixy="0.0" ixz="0.0" iyy="0.0" iyz="0.0" izz="0.0" />
+		</inertial>
+		<visual>
+			<origin xyz="0 0 0" />
+			<geometry>
+				<box size="2.4 0.04 ${size_z_wall1}" />
+			</geometry>
+			<material name="Grey"/>
+		</visual>
+		<collision>
+			<origin xyz="0 0 0" />
+			<geometry>
+				<box size="2.4 0.04 ${size_z_wall1}" />
+			</geometry>
+		</collision>
+	</link>
+	<gazebo reference="wall_elv7">
+		<material>IPA/WallApartment</material>
+	</gazebo>
+	<joint name="joint_wall_elv7" type="fixed">
+		<origin xyz="1.2 -0.65 0" rpy="0 0 0" />
+		<parent link="origin_elevator" />
+		<child link="wall_elv7" />
+	</joint>
+	<!-- wall elv8 -->
+	<link name="wall_elv8">
+		<inertial>
+			<origin xyz="0 0 0" />
+			<mass value="5.0" />
+			<inertia ixx="0.0" ixy="0.0" ixz="0.0" iyy="0.0" iyz="0.0" izz="0.0" />
+		</inertial>
+		<visual>
+			<origin xyz="0 0 0" />
+			<geometry>
+				<box size="2.4 0.04 ${size_z_wall1}" />
+			</geometry>
+			<material name="Grey"/>
+		</visual>
+		<collision>
+			<origin xyz="0 0 0" />
+			<geometry>
+				<box size="2.4 0.04 ${size_z_wall1}" />
+			</geometry>
+		</collision>
+	</link>
+	<gazebo reference="wall_elv8">
+		<material>IPA/WallApartment</material>
+	</gazebo>
+	<joint name="joint_wall_elv8" type="fixed">
+		<origin xyz="1.2 -1.52 0" rpy="0 0 0" />
+		<parent link="origin_elevator" />
+		<child link="wall_elv8" />
 	</joint>
 	<!-- elevator 22 -->
@@ -233,4 +264,5 @@
 				<box size="0.04 0.87 ${size_z_wall1}" />
 			</geometry>
+			<material name="Grey"/>
 		</visual>
 		<collision>
@@ -245,6 +277,6 @@
 	</gazebo>
 	<joint name="joint_elevator_right2" type="fixed">
-		<origin xyz="${-size_total_x/2+dist_axis_x-wall_depth-1.6-1.15-3} ${-0.68-dist_axis_y-1.68-1.15-1.6} ${size_z_wall1/2}" rpy="0 0 -0.7853" />
-		<parent link="dummy_link" />
+		<origin xyz="2.4 -1.085 0" rpy="0 0 0" />
+		<parent link="origin_elevator" />
 		<child link="elevator_right2" />
 	</joint>
@@ -261,4 +293,5 @@
 				<box size="0.01 0.05 0.05" />
 			</geometry>
+			<material name="Red"/>
 		</visual>
 		<collision>
@@ -270,6 +303,6 @@
 	</link>
 	<joint name="joint_elevator_button1" type="prismatic">
-		<origin xyz="${-0.025} ${0.025} ${-size_z_wall1/2+1.035}" rpy="0 0 0" />
-		<parent link="wall_ext4" />
+		<origin xyz="-0.04 0 ${-size_z_wall1/2+1.035}" rpy="0 0 0" />
+		<parent link="origin_elevator" />
 		<child link="elevator_button1" />
 		<calibration rising="0.0"/>
@@ -292,5 +325,4 @@
                         </sensor:contact>
                         <material>Gazebo/Red</material>
-                        <!--turnGravityOff>false</turnGravityOff-->
                 </gazebo>
 	<link name="elevator_button2">
@@ -305,4 +337,5 @@
 				<box size="0.01 0.05 0.05" />
 			</geometry>
+			<material name="Red"/>
 		</visual>
 		<collision>
@@ -314,6 +347,6 @@
 	</link>
 	<joint name="joint_elevator_button2" type="prismatic">
-		<origin xyz="${-0.025} ${0.025} ${-size_z_wall1/2+1.095}" rpy="0 0 0" />
-		<parent link="wall_ext4" />
+		<origin xyz="-0.04 0 ${-size_z_wall1/2+1.095}" rpy="0 0 0" />
+		<parent link="origin_elevator" />
 		<child link="elevator_button2" />
 		<calibration rising="0.0"/>
@@ -338,4 +371,88 @@
                         <turnGravityOff>false</turnGravityOff>
                 </gazebo>
+<link name="wall_ext18">
+		<inertial>
+			<origin xyz="0 0 0" />
+			<mass value="5.0" />
+			<inertia ixx="0.0" ixy="0.0" ixz="0.0" iyy="0.0" iyz="0.0" izz="0.0" />
+		</inertial>
+		<visual>
+			<origin xyz="0 0 0" />
+			<geometry>
+				<box size="0.04 1.74 ${size_z_wall1}" />
+			</geometry>
+			<material name="Grey"/>
+		</visual>
+		<collision>
+			<origin xyz="0 0 0" />
+			<geometry>
+				<box size="0.04 1.74 ${size_z_wall1}" />
+			</geometry>
+		</collision>
+	</link>
+	<gazebo reference="wall_ext18">
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
File: cob_gazebo_worlds/urdf/ipa-apartment/ipa-apartment.urdf.xacro (robot description, xacro)
@@ -6,6 +6,9 @@
 	xmlns:xacro="http://playerstage.sourceforge.net/gazebo/xmlschema/#interface"
 	name="ipa-apartment">
+  	  <include filename="$(find cob_description)/urdf/materials.urdf.xacro" />
 	  <!-- apartment -->
 	  <include filename="$(find cob_gazebo_worlds)/urdf/ipa-apartment/apartment.urdf.xacro" />
+	  <!-- office-->
+	  <include filename="$(find cob_gazebo_worlds)/urdf/ipa-apartment/office.urdf.xacro" />
 	  <!-- landing-->
 	  <include filename="$(find cob_gazebo_worlds)/urdf/ipa-apartment/landing.urdf.xacro" />
@@ -29,6 +32,7 @@
 	  <property name="wall_depth" value="0.06" />
 	  <property name="window_depth" value="0.15" />
-	  <property name="size_z_wall1" value="2.8" />
+	  <property name="size_z_wall1" value="2" />
 	  <property name="size_z_wall2" value="0.92" />
+	  <property name="size_z_wall3" value="1.4" />
 <xacro:macro name="ipa-apartment" params="name">
 	<!-- dummy_link -->
@@ -54,6 +58,9 @@
 	  <xacro:apartment name="apartment">
 	  </xacro:apartment>
-	  <xacro:landing name="landing">
+	  <xacro:landing name="landing" parent="dummy_link">
+		<origin xyz="${-13.9+dist_axis_x} ${-dist_axis_y} 0" rpy="0 0 0" />
 	  </xacro:landing>
+	  <xacro:office name="office">
+	  </xacro:office>
 	  <xacro:elevator name="elevator">
 	  </xacro:elevator>
