Commit message: Simulation model for 3rd flor and visualiced in rviz

File: cob_gazebo_worlds/urdf/ipa-apartment/landing.urdf.xacro (robot description, xacro)
@@ -4,33 +4,58 @@
        xmlns:interface="http://playerstage.sourceforge.net/gazebo/xmlschema/#interface"
        xmlns:xacro="http://ros.org/wiki/xacro">
-        <xacro:macro name="landing" params="name">
-	<!-- wall ext -->
-	<link name="wall_ext">
-		<inertial>
-			<origin xyz="0 0 0" />
-			<mass value="5.0" />
-			<inertia ixx="0.0" ixy="0.0" ixz="0.0" iyy="0.0" iyz="0.0" izz="0.0" />
-		</inertial>
-		<visual>
-			<origin xyz="0 0 0" />
-			<geometry>
-				<box size="4.6 0.04 ${size_z_wall1}" />
-			</geometry>
-		</visual>
-		<collision>
-			<origin xyz="0 0 0" />
-			<geometry>
-				<box size="4.6 0.04 ${size_z_wall1}" />
-			</geometry>
-		</collision>
-	</link>
-	<gazebo reference="wall_ext">
-		<material>IPA/WallApartment</material>
-	</gazebo>
-	<joint name="joint_wall_ext" type="fixed">
-		<origin xyz="${-size_total_x/2+dist_axis_x-wall_depth-2.3} ${-0.68-dist_axis_y} ${size_z_wall1/2}" rpy="0 0 0" />
-		<parent link="dummy_link" />
-		<child link="wall_ext" />
-	</joint>
+        <xacro:macro name="landing" params="name parent *origin">
+	<link name="origin_landing">
+		<inertial>
+			<origin xyz="0 0 0" />
+			<mass value="0.0" />
+			<inertia ixx="0.0" ixy="0.0" ixz="0.0" iyy="0.0" iyz="0.0" izz="0.0" />
+		</inertial>
+		<visual>
+			<origin xyz="0 0 0" />
+			<geometry>
+				<box size="0 0 0" />
+			</geometry>
+		</visual>
+		<collision>
+			<origin xyz="0 0 0" />
+			<geometry>
+				<box size="0 0 0" />
+			</geometry>
+		</collision>
+	</link>
+	<joint name="joint_origin_landing" type="fixed">
+		<insert_block name="origin" />
+        <parent link="${parent}"/>
+		<child link="origin_landing" />
+	</joint>
+	<!-- wall ext -->
+	<!--link name="wall_ext1">
+		<inertial>
+			<origin xyz="0 0 0" />
+			<mass value="5.0" />
+			<inertia ixx="0.0" ixy="0.0" ixz="0.0" iyy="0.0" iyz="0.0" izz="0.0" />
+		</inertial>
+		<visual>
+			<origin xyz="0 0 0" />
+			<geometry>
+				<box size="2.1 0.04 ${size_z_wall1}" />
+			</geometry>
+			<material name="Grey"/>
+		</visual>
+		<collision>
+			<origin xyz="0 0 0" />
+			<geometry>
+				<box size="2.1 0.04 ${size_z_wall1}" />
+			</geometry>
+		</collision>
+	</link>
+	<gazebo reference="wall_ext1">
+		<material>IPA/WallApartment</material>
+	</gazebo>
+	<joint name="joint_wall_ext1" type="fixed">
+		<origin xyz="8.8 2.565 ${size_z_wall1/2}" rpy="0 0 0" />
+		<parent link="origin_landing" />
+		<child link="wall_ext1" />
+	</joint-->
 	<!-- wall ext -->
 	<link name="wall_ext2">
@@ -43,11 +68,12 @@
 			<origin xyz="0 0 0" />
 			<geometry>
-				<box size="4.6 0.04 ${size_z_wall1}" />
-			</geometry>
-		</visual>
-		<collision>
-			<origin xyz="0 0 0" />
-			<geometry>
-				<box size="4.6 0.04 ${size_z_wall1}" />
+				<box size="2.1 0.04 ${size_z_wall1}" />
+			</geometry>
+			<material name="Grey"/>
+		</visual>
+		<collision>
+			<origin xyz="0 0 0" />
+			<geometry>
+				<box size="2.1 0.04 ${size_z_wall1}" />
 			</geometry>
 		</collision>
@@ -57,9 +83,9 @@
 	</gazebo>
 	<joint name="joint_wall_ext2" type="fixed">
-		<origin xyz="${-size_total_x/2+dist_axis_x-wall_depth-2.3} ${-0.68-dist_axis_y+1.6} ${size_z_wall1/2}" rpy="0 0 0" />
-		<parent link="dummy_link" />
+		<origin xyz="8.8 -2.565 ${size_z_wall1/2}" rpy="0 0 0" />
+		<parent link="origin_landing" />
 		<child link="wall_ext2" />
 	</joint>
-	<!-- wall ext3 -->
+	<!-- wall ext -->
 	<link name="wall_ext3">
 		<inertial>
@@ -71,11 +97,12 @@
 			<origin xyz="0 0 0" />
 			<geometry>
-				<box size="0.04 1.9 ${size_z_wall1}" />
-			</geometry>
-		</visual>
-		<collision>
-			<origin xyz="0 0 0" />
-			<geometry>
-				<box size="0.04 1.9 ${size_z_wall1}" />
+				<box size="0.04 1.73 ${size_z_wall1}" />
+			</geometry>
+			<material name="Grey"/>
+		</visual>
+		<collision>
+			<origin xyz="0 0 0" />
+			<geometry>
+				<box size="0.04 1.73 ${size_z_wall1}" />
 			</geometry>
 		</collision>
@@ -85,9 +112,9 @@
 	</gazebo>
 	<joint name="joint_wall_ext3" type="fixed">
-		<origin xyz="${-size_total_x/2+dist_axis_x-wall_depth-4.6-0.68} ${-0.68-dist_axis_y-0.65} ${size_z_wall1/2}" rpy="0 0 -0.7853" />
-		<parent link="dummy_link" />
+		<origin xyz="7.75 -1.7 ${size_z_wall1/2}" rpy="0 0 0" />
+		<parent link="origin_landing" />
 		<child link="wall_ext3" />
 	</joint>
-	<!-- wall ext4 -->
+	<!-- wall ext -->
 	<link name="wall_ext4">
 		<inertial>
@@ -99,11 +126,12 @@
 			<origin xyz="0 0 0" />
 			<geometry>
-				<box size="0.04 0.72 ${size_z_wall1}" />
-			</geometry>
-		</visual>
-		<collision>
-			<origin xyz="0 0 0" />
-			<geometry>
-				<box size="0.04 0.72 ${size_z_wall1}" />
+				<box size="0.04 1.73 ${size_z_wall1}" />
+			</geometry>
+			<material name="Grey"/>
+		</visual>
+		<collision>
+			<origin xyz="0 0 0" />
+			<geometry>
+				<box size="0.04 1.73 ${size_z_wall1}" />
 			</geometry>
 		</collision>
@@ -113,8 +141,432 @@
 	</gazebo>
 	<joint name="joint_wall_ext4" type="fixed">
-		<origin xyz="${-size_total_x/2+dist_axis_x-wall_depth-4.6-0.68-1.54} ${-0.68-dist_axis_y-0.65-1.54} ${size_z_wall1/2}" rpy="0 0 -0.7853" />
-		<parent link="dummy_link" />
+		<origin xyz="7.75 1.7 ${size_z_wall1/2}" rpy="0 0 0" />
+		<parent link="origin_landing" />
 		<child link="wall_ext4" />
 	</joint>
+<link name="wall_ext5">
+		<inertial>
+			<origin xyz="0 0 0" />
+			<mass value="5.0" />
+			<inertia ixx="0.0" ixy="0.0" ixz="0.0" iyy="0.0" iyz="0.0" izz="0.0" />
+		</inertial>
+		<visual>
+			<origin xyz="0 0 0" />
+			<geometry>
+				<box size="2.34 0.04 ${size_z_wall1}" />
+			</geometry>
+			<material name="Grey"/>
+		</visual>
+		<collision>
+			<origin xyz="0 0 0" />
+			<geometry>
+				<box size="6.73 0.04 ${size_z_wall1}" />
+			</geometry>
+		</collision>
+	</link>
+	<gazebo reference="wall_ext5">
+		<material>IPA/WallApartment</material>
+	</gazebo>
+	<joint name="joint_wall_ext5" type="fixed">
+		<origin xyz="6.6 -0.85 ${size_z_wall1/2}" rpy="0 0 0" />
+		<parent link="origin_landing" />
+		<child link="wall_ext5" />
+	</joint>
+<link name="wall_ext6">
+		<inertial>
+			<origin xyz="0 0 0" />
+			<mass value="5.0" />
+			<inertia ixx="0.0" ixy="0.0" ixz="0.0" iyy="0.0" iyz="0.0" izz="0.0" />
+		</inertial>
+		<visual>
+			<origin xyz="0 0 0" />
+			<geometry>
+				<box size="2.34 0.04 ${size_z_wall1}" />
+			</geometry>
+			<material name="Grey"/>
+		</visual>
+		<collision>
+			<origin xyz="0 0 0" />
+			<geometry>
+				<box size="2.34 0.04 ${size_z_wall1}" />
+			</geometry>
+		</collision>
+	</link>
+	<gazebo reference="wall_ext6">
+		<material>IPA/WallApartment</material>
+	</gazebo>
+	<joint name="joint_wall_ext6" type="fixed">
+		<origin xyz="6.6 0.85 ${size_z_wall1/2}" rpy="0 0 0" />
+		<parent link="origin_landing" />
+		<child link="wall_ext6" />
+	</joint>
+	<!--office landing-->
+		<!--link name="wall_ext7">
+		<inertial>
+			<origin xyz="0 0 0" />
+			<mass value="5.0" />
+			<inertia ixx="0.0" ixy="0.0" ixz="0.0" iyy="0.0" iyz="0.0" izz="0.0" />
+		</inertial>
+		<visual>
+			<origin xyz="0 0 0" />
+			<geometry>
+				<box size="0.04 2.1 ${size_z_wall1}" />
+			</geometry>
+			<material name="Grey"/>
+		</visual>
+		<collision>
+			<origin xyz="0 0 0" />
+			<geometry>
+				<box size="0.04 2.1 ${size_z_wall1}" />
+			</geometry>
+		</collision>
+	</link>
+	<gazebo reference="wall_ext7">
+		<material>IPA/WallApartment</material>
+	</gazebo>
+	<joint name="joint_wall_ext7" type="fixed">
+		<origin xyz="2.565 8.8 ${size_z_wall1/2}" rpy="0 0 0" />
+		<parent link="origin_landing" />
+		<child link="wall_ext7" />
+	</joint-->
+	<!-- wall ext -->
+	<link name="wall_ext8">
+		<inertial>
+			<origin xyz="0 0 0" />
+			<mass value="5.0" />
+			<inertia ixx="0.0" ixy="0.0" ixz="0.0" iyy="0.0" iyz="0.0" izz="0.0" />
+		</inertial>
+		<visual>
+			<origin xyz="0 0 0" />
+			<geometry>
+				<box size="0.04 2.1 ${size_z_wall1}" />
+			</geometry>
+			<material name="Grey"/>
+		</visual>
+		<collision>
+			<origin xyz="0 0 0" />
+			<geometry>
+				<box size="0.04 2.1 ${size_z_wall1}" />
+			</geometry>
+		</collision>
+	</link>
+	<gazebo reference="wall_ext8">
+		<material>IPA/WallApartment</material>
+	</gazebo>
+	<joint name="joint_wall_ext8" type="fixed">
+		<origin xyz="-2.565 8.8 ${size_z_wall1/2}" rpy="0 0 0" />
+		<parent link="origin_landing" />
+		<child link="wall_ext8" />
+	</joint>
+	<!-- wall ext -->
+	<link name="wall_ext9">
+		<inertial>
+			<origin xyz="0 0 0" />
+			<mass value="5.0" />
+			<inertia ixx="0.0" ixy="0.0" ixz="0.0" iyy="0.0" iyz="0.0" izz="0.0" />
+		</inertial>
+		<visual>
+			<origin xyz="0 0 0" />
+			<geometry>
+				<box size="1.73 0.04 ${size_z_wall1}" />
+			</geometry>
+			<material name="Grey"/>
+		</visual>
+		<collision>
+			<origin xyz="0 0 0" />
+			<geometry>
+				<box size="1.73 0.04 ${size_z_wall1}" />
+			</geometry>
+		</collision>
+	</link>
+	<gazebo reference="wall_ext9">
+		<material>IPA/WallApartment</material>
+	</gazebo>
+	<joint name="joint_wall_ext9" type="fixed">
+		<origin xyz="-1.7 7.75 ${size_z_wall1/2}" rpy="0 0 0" />
+		<parent link="origin_landing" />
+		<child link="wall_ext9" />
+	</joint>
+	<!-- wall ext -->
+	<link name="wall_ext10">
+		<inertial>
+			<origin xyz="0 0 0" />
+			<mass value="5.0" />
+			<inertia ixx="0.0" ixy="0.0" ixz="0.0" iyy="0.0" iyz="0.0" izz="0.0" />
+		</inertial>
+		<visual>
+			<origin xyz="0 0 0" />
+			<geometry>
+				<box size="1.73 0.04 ${size_z_wall1}" />
+			</geometry>
+			<material name="Grey"/>
+		</visual>
+		<collision>
+			<origin xyz="0 0 0" />
+			<geometry>
+				<box size="1.73 0.04 ${size_z_wall1}" />
+			</geometry>
+		</collision>
+	</link>
+	<gazebo reference="wall_ext10">
+		<material>IPA/WallApartment</material>
+	</gazebo>
+	<joint name="joint_wall_ext10" type="fixed">
+		<origin xyz="1.7 7.75 ${size_z_wall1/2}" rpy="0 0 0" />
+		<parent link="origin_landing" />
+		<child link="wall_ext10" />
+	</joint>
+<link name="wall_ext11">
+		<inertial>
+			<origin xyz="0 0 0" />
+			<mass value="5.0" />
+			<inertia ixx="0.0" ixy="0.0" ixz="0.0" iyy="0.0" iyz="0.0" izz="0.0" />
+		</inertial>
+		<visual>
+			<origin xyz="0 0 0" />
+			<geometry>
+				<box size="0.04 2.34 ${size_z_wall1}" />
+			</geometry>
+			<material name="Grey"/>
+		</visual>
+		<collision>
+			<origin xyz="0 0 0" />
+			<geometry>
+				<box size="0.04 2.34 ${size_z_wall1}" />
+			</geometry>
+		</collision>
+	</link>
+	<gazebo reference="wall_ext11">
+		<material>IPA/WallApartment</material>
+	</gazebo>
+	<joint name="joint_wall_ext11" type="fixed">
+		<origin xyz="-0.85 6.6 ${size_z_wall1/2}" rpy="0 0 0" />
+		<parent link="origin_landing" />
+		<child link="wall_ext11" />
+	</joint>
+<link name="wall_ext12">
+		<inertial>
+			<origin xyz="0 0 0" />
+			<mass value="5.0" />
+			<inertia ixx="0.0" ixy="0.0" ixz="0.0" iyy="0.0" iyz="0.0" izz="0.0" />
+		</inertial>
+		<visual>
+			<origin xyz="0 0 0" />
+			<geometry>
+				<box size="0.04 2.34 ${size_z_wall1}" />
+			</geometry>
+			<material name="Grey"/>
+		</visual>
+		<collision>
+			<origin xyz="0 0 0" />
+			<geometry>
+				<box size="0.04 2.34 ${size_z_wall1}" />
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
File: cob_gazebo_worlds/urdf/ipa-apartment/wall_ipa.urdf.xacro (robot description, xacro)
@@ -16,4 +16,5 @@
 				<box size="0.77 0.10 2.40" />
 			</geometry>
+			<material name="Grey"/>
 		</visual>
 		<collision>
