Commit message: :q

File: cob_gazebo_worlds/urdf/ipa-apartment/apartment.urdf.xacro (robot description, xacro)
@@ -17,5 +17,5 @@
 				<box size="${wall_depth} ${size_d} ${size_z_wall1}" />
 			</geometry>
-			<material name="Grey"/>
+			<material name="IPA/Grey"/>
 		</visual>
 		<collision>
@@ -46,5 +46,5 @@
 				<box size=" ${size_b} ${window_depth} ${size_z_wall2}" />
 			</geometry>
-			<material name="Grey"/>
+			<material name="IPA/Grey"/>
 		</visual>
 		<collision>
@@ -75,5 +75,5 @@
 				<box size="${wall_depth} ${size_a} ${size_z_wall2}" />
 			</geometry>
-			<material name="Grey"/>
+			<material name="IPA/Grey"/>
 		</visual>
 		<collision>
@@ -104,5 +104,5 @@
 				<box size=" ${window_depth} 1.6 ${size_z_wall2}" />
 			</geometry>
-			<material name="Grey"/>
+			<material name="IPA/Grey"/>
 		</visual>
 		<collision>
@@ -133,5 +133,5 @@
 				<box size="${window_depth} 1.55 ${size_z_wall2}" />
 			</geometry>
-			<material name="Grey"/>
+			<material name="IPA/Grey"/>
 		</visual>
 		<collision>
@@ -162,5 +162,5 @@
 				<box size="${wall_depth} ${size_a} ${size_z_wall2}" />
 			</geometry>
-			<material name="Grey"/>
+			<material name="IPA/Grey"/>
 		</visual>
 		<collision>
@@ -191,5 +191,5 @@
 				<box size=" ${size_b} ${window_depth} ${size_z_wall2}" />
 			</geometry>
-			<material name="Grey"/>
+			<material name="IPA/Grey"/>
 		</visual>
 		<collision>
@@ -220,5 +220,5 @@
 				<box size="${wall_depth} ${size_a} ${size_z_wall1}" />
 			</geometry>
-			<material name="Grey"/>
+			<material name="IPA/Grey"/>
 		</visual>
 		<collision>
@@ -249,5 +249,5 @@
 				<box size="${wall_depth} 1.9 ${size_z_wall2}" />
 			</geometry>
-			<material name="Grey"/>
+			<material name="IPA/Grey"/>
 		</visual>
 		<collision>
@@ -278,5 +278,5 @@
 				<box size="0.04 0.62 ${size_z_wall1}" />
 			</geometry>
-			<material name="Transparent"/>
+			<material name="IPA/Transparent"/>
 		</visual>
 		<collision>
@@ -307,5 +307,5 @@
 				<box size="0.04 0.62 ${size_z_wall1}" />
 			</geometry>
-			<material name="Transparent"/>
+			<material name="IPA/Transparent"/>
 		</visual>
 		<collision>

File: cob_gazebo_worlds/urdf/ipa-apartment/cabinets.urdf.xacro (robot description, xacro)
@@ -17,5 +17,5 @@
 				<box size="1.15 0.55 2.40" />
 			</geometry>
-			<material name="LightBlue"/>
+			<material name="IPA/LightBlue"/>
 		</visual>
 		<collision>
@@ -45,5 +45,5 @@
 				<box size="1.15 0.55 2.40" />
 			</geometry>
-			<material name="LightBlue"/>
+			<material name="IPA/LightBlue"/>
 		</visual>
 		<collision>
@@ -73,5 +73,5 @@
 				<box size="1.15 0.55 2.40" />
 			</geometry>
-			<material name="LightBlue"/>
+			<material name="IPA/LightBlue"/>
 		</visual>
 		<collision>
@@ -101,5 +101,5 @@
 				<box size="0.36 0.36 ${size_z_wall1}" />
 			</geometry>
-			<material name="LightBlue"/>
+			<material name="IPA/LightBlue"/>
 		</visual>
 		<collision>

File: cob_gazebo_worlds/urdf/ipa-apartment/elevator.urdf.xacro (robot description, xacro)
@@ -41,5 +41,5 @@
 				<box size="0.04 0.87 ${size_z_wall1}" />
 			</geometry>
-			<material name="LightBlue"/>
+			<material name="IPA/LightBlue"/>
 		</visual>
 		<collision>
@@ -80,5 +80,5 @@
 				<box size="2.4 0.04 ${size_z_wall1}" />
 			</geometry>
-			<material name="Grey"/>
+			<material name="IPA/Grey"/>
 		</visual>
 		<collision>
@@ -109,5 +109,5 @@
 				<box size="2.4 0.04 ${size_z_wall1}" />
 			</geometry>
-			<material name="Grey"/>
+			<material name="IPA/Grey"/>
 		</visual>
 		<collision>
@@ -138,5 +138,5 @@
 				<box size="0.04 0.87 ${size_z_wall1}" />
 			</geometry>
-			<material name="Grey"/>
+			<material name="IPA/Grey"/>
 		</visual>
 		<collision>
@@ -167,5 +167,5 @@
 				<box size="0.04 0.87 ${size_z_wall1}" />
 			</geometry>
-			<material name="LightBlue"/>
+			<material name="IPA/LightBlue"/>
 		</visual>
 		<collision>
@@ -206,5 +206,5 @@
 				<box size="2.4 0.04 ${size_z_wall1}" />
 			</geometry>
-			<material name="Grey"/>
+			<material name="IPA/Grey"/>
 		</visual>
 		<collision>
@@ -235,5 +235,5 @@
 				<box size="2.4 0.04 ${size_z_wall1}" />
 			</geometry>
-			<material name="Grey"/>
+			<material name="IPA/Grey"/>
 		</visual>
 		<collision>
@@ -264,5 +264,5 @@
 				<box size="0.04 0.87 ${size_z_wall1}" />
 			</geometry>
-			<material name="Grey"/>
+			<material name="IPA/Grey"/>
 		</visual>
 		<collision>
@@ -293,5 +293,5 @@
 				<box size="0.01 0.05 0.05" />
 			</geometry>
-			<material name="Red"/>
+			<material name="IPA/Red"/>
 		</visual>
 		<collision>
@@ -337,5 +337,5 @@
 				<box size="0.01 0.05 0.05" />
 			</geometry>
-			<material name="Red"/>
+			<material name="IPA/Red"/>
 		</visual>
 		<collision>
@@ -382,5 +382,5 @@
 				<box size="0.04 1.74 ${size_z_wall1}" />
 			</geometry>
-			<material name="Grey"/>
+			<material name="IPA/Grey"/>
 		</visual>
 		<collision>
@@ -410,5 +410,5 @@
 				<box size="0.04 1.74 ${size_z_wall1}" />
 			</geometry>
-			<material name="Grey"/>
+			<material name="IPA/Grey"/>
 		</visual>
 		<collision>
@@ -438,5 +438,5 @@
 				<box size="0.04 1.3 ${size_z_wall1}" />
 			</geometry>
-			<material name="Grey"/>
+			<material name="IPA/Grey"/>
 		</visual>
 		<collision>

File: cob_gazebo_worlds/urdf/ipa-apartment/ipa-apartment.urdf (robot description, URDF)
Before this commit: robot ipa-apartment, 64 links, 63 joints
Links:
- link wall_office_02: geometry collision box size=0.06 8.2 0.92; visual box size=0.06 8.2 0.92
- link wall_office_03: geometry collision box size=0.06 8.2 0.92; visual box size=0.06 8.2 0.92
- link wall_office_04: geometry collision box size=11.2 0.06 0.92; visual box size=11.2 0.06 0.92
- link wall_office_05: geometry collision box size=0.06 4.51 2; visual box size=0.06 4.51 2
- link wall_office_06: geometry collision box size=0.06 1.23 2; visual box size=0.06 1.23 2
- link wall_office_07: geometry collision box size=0.06 4.01 2; visual box size=0.06 4.01 2
- link wall_office_08: geometry collision box size=0.06 1.73 2; visual box size=0.06 1.73 2
- link wall_office_09: geometry collision box size=4.5 0.06 2; visual box size=4.5 0.06 2
- link wall_office_10: geometry collision box size=4.5 0.06 2; visual box size=4.5 0.06 2
Joints:
- joint joint_wall_office_02: origin xyz=5.6 0 0.7 rpy=0 0 0 -> xyz=5.6 0 0.46 rpy=0 0 0
- joint joint_wall_office_03: origin xyz=-5.6 0 0.7 rpy=0 0 0 -> xyz=-5.6 0 0.46 rpy=0 0 0
- joint joint_wall_office_04: origin xyz=0 4 0.7 rpy=0 0 0 -> xyz=0 4 0.46 rpy=0 0 0
- joint joint_wall_office_05: origin xyz=1.09 -0.615 0.7 rpy=0 0 0 -> xyz=1.09 -0.615 1.0 rpy=0 0 0
- joint joint_wall_office_06: origin xyz=1.09 3.385 0.7 rpy=0 0 0 -> xyz=1.09 3.385 1.0 rpy=0 0 0
- joint joint_wall_office_07: origin xyz=-1.09 2 0.7 rpy=0 0 0 -> xyz=-1.09 2 1.0 rpy=0 0 0
- joint joint_wall_office_08: origin xyz=-1.09 -2 0.7 rpy=0 0 0 -> xyz=-1.09 -2 1.0 rpy=0 0 0
- joint joint_wall_office_09: origin xyz=3.35 1.64 0.7 rpy=0 0 0 -> xyz=3.35 1.64 1.0 rpy=0 0 0
- joint joint_wall_office_10: origin xyz=-3.35 -1.14 0.7 rpy=0 0 0 -> xyz=-3.35 -1.14 1.0 rpy=0 0 0

File: cob_gazebo_worlds/urdf/ipa-apartment/landing.urdf.xacro (robot description, xacro)
@@ -41,5 +41,5 @@
 				<box size="2.1 0.04 ${size_z_wall1}" />
 			</geometry>
-			<material name="Grey"/>
+			<material name="IPA/Grey"/>
 		</visual>
 		<collision>
@@ -70,5 +70,5 @@
 				<box size="2.1 0.04 ${size_z_wall1}" />
 			</geometry>
-			<material name="Grey"/>
+			<material name="IPA/Grey"/>
 		</visual>
 		<collision>
@@ -99,5 +99,5 @@
 				<box size="0.04 1.73 ${size_z_wall1}" />
 			</geometry>
-			<material name="Grey"/>
+			<material name="IPA/Grey"/>
 		</visual>
 		<collision>
@@ -128,5 +128,5 @@
 				<box size="0.04 1.73 ${size_z_wall1}" />
 			</geometry>
-			<material name="Grey"/>
+			<material name="IPA/Grey"/>
 		</visual>
 		<collision>
@@ -156,5 +156,5 @@
 				<box size="2.34 0.04 ${size_z_wall1}" />
 			</geometry>
-			<material name="Grey"/>
+			<material name="IPA/Grey"/>
 		</visual>
 		<collision>
@@ -184,5 +184,5 @@
 				<box size="2.34 0.04 ${size_z_wall1}" />
 			</geometry>
-			<material name="Grey"/>
+			<material name="IPA/Grey"/>
 		</visual>
 		<collision>
@@ -213,5 +213,5 @@
 				<box size="0.04 2.1 ${size_z_wall1}" />
 			</geometry>
-			<material name="Grey"/>
+			<material name="IPA/Grey"/>
 		</visual>
 		<collision>
@@ -242,5 +242,5 @@
 				<box size="0.04 2.1 ${size_z_wall1}" />
 			</geometry>
-			<material name="Grey"/>
+			<material name="IPA/Grey"/>
 		</visual>
 		<collision>
@@ -271,5 +271,5 @@
 				<box size="1.73 0.04 ${size_z_wall1}" />
 			</geometry>
-			<material name="Grey"/>
+			<material name="IPA/Grey"/>
 		</visual>
 		<collision>
@@ -300,5 +300,5 @@
 				<box size="1.73 0.04 ${size_z_wall1}" />
 			</geometry>
-			<material name="Grey"/>
+			<material name="IPA/Grey"/>
 		</visual>
 		<collision>
@@ -328,5 +328,5 @@
 				<box size="0.04 2.34 ${size_z_wall1}" />
 			</geometry>
-			<material name="Grey"/>
+			<material name="IPA/Grey"/>
 		</visual>
 		<collision>
@@ -356,5 +356,5 @@
 				<box size="0.04 2.34 ${size_z_wall1}" />
 			</geometry>
-			<material name="Grey"/>
+			<material name="IPA/Grey"/>
 		</visual>
 		<collision>
@@ -384,5 +384,5 @@
 				<box size="0.04 6.6 ${size_z_wall1}" />
 			</geometry>
-			<material name="Grey"/>
+			<material name="IPA/Grey"/>
 		</visual>
 		<collision>
@@ -412,5 +412,5 @@
 				<box size="0.04 6.6 ${size_z_wall1}" />
 			</geometry>
-			<material name="Grey"/>
+			<material name="IPA/Grey"/>
 		</visual>
 		<collision>
@@ -441,5 +441,5 @@
 				<box size="0.04 6.6 ${size_z_wall1}" />
 			</geometry>
-			<material name="Grey"/>
+			<material name="IPA/Grey"/>
 		</visual>
 		<collision>
@@ -469,5 +469,5 @@
 				<box size="0.04 1.8 ${size_z_wall1}" />
 			</geometry>
-			<material name="Grey"/>
+			<material name="IPA/Grey"/>
 		</visual>
 		<collision>
@@ -497,5 +497,5 @@
 				<box size="1.8 0.04 ${size_z_wall1}" />
 			</geometry>
-			<material name="Grey"/>
+			<material name="IPA/Grey"/>
 		</visual>
 		<collision>
@@ -525,5 +525,5 @@
 				<box size="0.04 7.4 ${size_z_wall1}" />
 			</geometry>
-			<material name="Grey"/>
+			<material name="IPA/Grey"/>
 		</visual>
 		<collision>
@@ -553,5 +553,5 @@
 				<box size="0.06 6 ${size_z_wall2}" />
 			</geometry>
-			<material name="Grey"/>
+			<material name="IPA/Grey"/>
 		</visual>
 		<collision>

File: cob_gazebo_worlds/urdf/ipa-apartment/office.urdf.xacro (robot description, xacro)
@@ -41,5 +41,5 @@
 				<box size="4.65 ${wall_depth} ${size_z_wall1}" />
 			</geometry>
-			<material name="Grey"/>
+			<material name="IPA/Grey"/>
 		</visual>
 		<collision>
@@ -70,5 +70,5 @@
 				<box size="4.65 ${wall_depth} ${size_z_wall1}" />
 			</geometry>
-			<material name="Grey"/>
+			<material name="IPA/Grey"/>
 		</visual>
 		<collision>
@@ -99,5 +99,5 @@
 				<box size="${wall_depth} 8.2 ${size_z_wall2}" />
 			</geometry>
-			<material name="Grey"/>
+			<material name="IPA/Grey"/>
 		</visual>
 		<collision>
@@ -128,5 +128,5 @@
 				<box size="${wall_depth} 8.2 ${size_z_wall2}" />
 			</geometry>
-			<material name="Grey"/>
+			<material name="IPA/Grey"/>
 		</visual>
 		<collision>
@@ -157,5 +157,5 @@
 				<box size="11.2 ${wall_depth} ${size_z_wall2}" />
 			</geometry>
-			<material name="Grey"/>
+			<material name="IPA/Grey"/>
 		</visual>
 		<collision>
@@ -186,5 +186,5 @@
 				<box size="${wall_depth} 4.51 ${size_z_wall1}" />
 			</geometry>
-			<material name="Grey"/>
+			<material name="IPA/Grey"/>
 		</visual>
 		<collision>
@@ -215,5 +215,5 @@
 				<box size="${wall_depth} 1.23 ${size_z_wall1}" />
 			</geometry>
-			<material name="Grey"/>
+			<material name="IPA/Grey"/>
 		</visual>
 		<collision>
@@ -244,5 +244,5 @@
 				<box size="${wall_depth} 4.01 ${size_z_wall1}" />
 			</geometry>
-			<material name="Grey"/>
+			<material name="IPA/Grey"/>
 		</visual>
 		<collision>
@@ -273,5 +273,5 @@
 				<box size="${wall_depth} 1.73 ${size_z_wall1}" />
 			</geometry>
-			<material name="Grey"/>
+			<material name="IPA/Grey"/>
 		</visual>
 		<collision>
@@ -302,5 +302,5 @@
 				<box size="4.5 ${wall_depth} ${size_z_wall1}" />
 			</geometry>
-			<material name="Grey"/>
+			<material name="IPA/Grey"/>
 		</visual>
 		<collision>
@@ -331,5 +331,5 @@
 				<box size="4.5 ${wall_depth} ${size_z_wall1}" />
 			</geometry>
-			<material name="Grey"/>
+			<material name="IPA/Grey"/>
 		</visual>
 		<collision>

File: cob_gazebo_worlds/urdf/ipa-apartment/wall_ipa.urdf.xacro (robot description, xacro)
@@ -16,5 +16,5 @@
 				<box size="0.77 0.10 2.40" />
 			</geometry>
-			<material name="Grey"/>
+			<material name="IPA/Grey"/>
 		</visual>
 		<collision>
