Commit message: New wall textures and floor for ipa-apartment environment

File: cob_gazebo_worlds/urdf/ipa-apartment/apartment.urdf.xacro (robot description, xacro)
@@ -15,20 +15,20 @@
 			<origin xyz="0 0 0" />
 			<geometry>
-				<box size="${wall_depth} ${size_d} ${size_z_wall1}" />
-			</geometry>
-			<material name="IPA/Grey"/>
-		</visual>
-		<collision>
-			<origin xyz="0 0 0" />
-			<geometry>
-				<box size="${wall_depth} ${size_d} ${size_z_wall1}" />
+				<box size="${wall_depth} ${size_d+0.18+0.35} ${size_z_wall1}" />
+			</geometry>
+			<material name="IPA/Grey"/>
+		</visual>
+		<collision>
+			<origin xyz="0 0 0" />
+			<geometry>
+				<box size="${wall_depth} ${size_d+0.18+0.35} ${size_z_wall1}" />
 			</geometry>
 		</collision>
 	</link>
 	<gazebo reference="wall_00">
-		<material>IPA/WallApartment</material>
+		<material>wall_floor_05</material>
 	</gazebo>
 	<joint name="joint_wall_00" type="fixed">
-		<origin xyz="${-size_total_x/2+dist_axis_x-wall_depth} ${size_total_y/2-size_d/2+0.1-dist_axis_y} ${size_z_wall1/2}" rpy="0 0 0" />
+		<origin xyz="${-size_total_x/2+dist_axis_x-wall_depth} ${(size_total_y/2-size_d/2+0.1-dist_axis_y)+0.175} ${size_z_wall1/2}" rpy="0 0 0" />
 		<parent link="dummy_link" />
 		<child link="wall_00" />
@@ -44,22 +44,109 @@
 			<origin xyz="0 0 0" />
 			<geometry>
-				<box size=" ${size_b} ${window_depth} ${size_z_wall2}" />
-			</geometry>
-			<material name="IPA/Grey"/>
-		</visual>
-		<collision>
-			<origin xyz="0 0 0" />
-			<geometry>
-				<box size="${size_b} ${window_depth} ${size_z_wall2}" />
+				<box size=" ${size_b} 0.001 0.90" />
+			</geometry>
+			<material name="IPA/Grey"/>
+		</visual>
+		<collision>
+			<origin xyz="0 0 0" />
+			<geometry>
+				<box size="${size_b} 0.001 0.90" />
 			</geometry>
 		</collision>
 	</link>
 	<gazebo reference="wall_01">
-		<material>IPA/WallApartment</material>
+		<material>kitchen_wall_with_heating</material>
 	</gazebo>
 	<joint name="joint_wall_01" type="fixed">
-		<origin xyz="${dist_axis_x} ${size_total_y/2-dist_axis_y+window_depth} ${size_z_wall2/2}" rpy="0 0 0" />
+		<origin xyz="${dist_axis_x} ${size_total_y/2-dist_axis_y+window_depth+0.02} 0.45" rpy="0 0 0" />
 		<parent link="dummy_link" />
 		<child link="wall_01" />
+	</joint>
+	<!-- wall_01_part2 -->
+	<link name="wall_01_part2">
+		<inertial>
+			<origin xyz="0 0 0" />
+			<mass value="5.0" />
+			<inertia ixx="0.0" ixy="0.0" ixz="0.0" iyy="0.0" iyz="0.0" izz="0.0" />
+		</inertial>
+		<visual>
+			<origin xyz="0 0 0" />
+			<geometry>
+				<box size=" ${size_b} 0.35 0.90" />
+			</geometry>
+			<material name="IPA/Grey"/>
+		</visual>
+		<collision>
+			<origin xyz="0 0 0" />
+			<geometry>
+				<box size="${size_b} 0.35 0.90" />
+			</geometry>
+		</collision>
+	</link>
+	<gazebo reference="wall_01_part2">
+		<material>kitchen_window_board</material>
+	</gazebo>
+	<joint name="joint_wall_01_part2" type="fixed">
+		<origin xyz="${dist_axis_x} ${size_total_y/2-dist_axis_y+window_depth+0.195} 0.45" rpy="0 0 0" />
+		<parent link="dummy_link" />
+		<child link="wall_01_part2" />
+	</joint>
+	<!-- wall_01_little_glas -->
+	<link name="wall_01_little_glas">
+		<inertial>
+			<origin xyz="0 0 0" />
+			<mass value="5.0" />
+			<inertia ixx="0.0" ixy="0.0" ixz="0.0" iyy="0.0" iyz="0.0" izz="0.0" />
+		</inertial>
+		<visual>
+			<origin xyz="0 0 0" />
+			<geometry>
+				<box size="0.02 0.35 2.70" />
+			</geometry>
+			<material name="IPA/Grey"/>
+		</visual>
+		<collision>
+			<origin xyz="0 0 0" />
+			<geometry>
+				<box size="0.02 0.35 2.70" />
+			</geometry>
+		</collision>
+	</link>
+	<gazebo reference="wall_01_little_glas">
+		<material>kitchen_wall_with_windows</material>
+	</gazebo>
+	<joint name="joint_wall_01_little_glas" type="fixed">
+		<origin xyz="3.5 ${size_total_y/2-dist_axis_y+window_depth+0.195} 1.35" rpy="0 0 0" />
+		<parent link="dummy_link" />
+		<child link="wall_01_little_glas" />
+	</joint>
+<!-- wall_01_part3 -->
+	<link name="wall_01_part3">
+		<inertial>
+			<origin xyz="0 0 0" />
+			<mass value="5.0" />
+			<inertia ixx="0.0" ixy="0.0" ixz="0.0" iyy="0.0" iyz="0.0" izz="0.0" />
+		</inertial>
+		<visual>
+			<origin xyz="0 0 0" />
+			<geometry>
+				<box size=" ${size_b} ${window_depth} 1.80" />
+			</geometry>
+			<material name="IPA/Grey"/>
+		</visual>
+		<collision>
+			<origin xyz="0 0 0" />
+			<geometry>
+				<box size="${size_b} ${window_depth} 1.80" />
+			</geometry>
+		</collision>
+	</link>
+	<gazebo reference="wall_01_part3">
+		<material>kitchen_wall_with_windows</material>
+	</gazebo>
+	<joint name="joint_wall_01_part3" type="fixed">
+		<origin xyz="${dist_axis_x} ${size_total_y/2-dist_axis_y+window_depth+0.44} 1.80" rpy="0 0 0" />
+		<parent link="dummy_link" />
+		<child link="wall_01_part3" />
 	</joint>
 	<!-- wall_02 -->
@@ -73,20 +160,20 @@
 			<origin xyz="0 0 0" />
 			<geometry>
-				<box size="${wall_depth} ${size_a} ${size_z_wall2}" />
-			</geometry>
-			<material name="IPA/Grey"/>
-		</visual>
-		<collision>
-			<origin xyz="0 0 0" />
-			<geometry>
-				<box size="${wall_depth} ${size_a} ${size_z_wall2}" />
+				<box size="${wall_depth} ${size_a+0.35} ${size_z_wall2}" />
+			</geometry>
+			<material name="IPA/Grey"/>
+		</visual>
+		<collision>
+			<origin xyz="0 0 0" />
+			<geometry>
+				<box size="${wall_depth} ${size_a+0.35} ${size_z_wall2}" />
 			</geometry>
 		</collision>
 	</link>
 	<gazebo reference="wall_02">
-		<material>IPA/WallApartment</material>
+		<material>wall_floor_05</material>
 	</gazebo>
 	<joint name="joint_wall_02" type="fixed">
-		<origin xyz="${size_total_x/2+dist_axis_x+wall_depth} ${size_total_y/2-size_a/2+0.15-dist_axis_y} ${size_z_wall2/2}" rpy="0 0 0" />
+		<origin xyz="${size_total_x/2+dist_axis_x+wall_depth} ${(size_total_y/2-size_a/2+0.15-dist_axis_y)+0.175} ${size_z_wall2/2}" rpy="0 0 0" />
 		<parent link="dummy_link" />
 		<child link="wall_02" />
@@ -102,20 +189,20 @@
 			<origin xyz="0 0 0" />
 			<geometry>
-				<box size=" ${window_depth} 1.6 ${size_z_wall2}" />
-			</geometry>
-			<material name="IPA/Grey"/>
-		</visual>
-		<collision>
-			<origin xyz="0 0 0" />
-			<geometry>
-				<box size="${window_depth} 1.5 ${size_z_wall2}" />
+				<box size=" ${window_depth} 1.55 ${size_z_wall2}" />
+			</geometry>
+			<material name="IPA/Grey"/>
+		</visual>
+		<collision>
+			<origin xyz="0 0 0" />
+			<geometry>
+				<box size="${window_depth} 1.55 ${size_z_wall2}" />
 			</geometry>
 		</collision>
 	</link>
 	<gazebo reference="wall_03">
-		<material>IPA/WallApartment</material>
+		<material>emergencyExit_window_left</material>
 	</gazebo>
 	<joint name="joint_wall_03" type="fixed">
-		<origin xyz="${size_total_x/2+dist_axis_x+0.561+window_depth/2} ${0.5-dist_axis_y} ${size_z_wall2/2}" rpy="0 0 0.785398" />
+		<origin xyz="${size_total_x/2+dist_axis_x+0.55+window_depth/2} ${0.6-dist_axis_y} ${size_z_wall2/2}" rpy="0 0 0.785398" />
 		<parent link="dummy_link" />
 		<child link="wall_03" />
@@ -131,20 +218,20 @@
 			<origin xyz="0 0 0" />
 			<geometry>
-				<box size="${window_depth} 1.55 ${size_z_wall2}" />
-			</geometry>
-			<material name="IPA/Grey"/>
-		</visual>
-		<collision>
-			<origin xyz="0 0 0" />
-			<geometry>
-				<box size="${window_depth} 1.5 ${size_z_wall2}" />
+				<box size="${window_depth} 1.6 ${size_z_wall2}" />
+			</geometry>
+			<material name="IPA/Grey"/>
+		</visual>
+		<collision>
+			<origin xyz="0 0 0" />
+			<geometry>
+				<box size="${window_depth} 1.6 ${size_z_wall2}" />
 			</geometry>
 		</collision>
 	</link>
 	<gazebo reference="wall_04">
-		<material>IPA/WallApartment</material>
+		<material>emergencyExit_window_right</material>
 	</gazebo>
 	<joint name="joint_wall_04" type="fixed">
-		<origin xyz="${size_total_x/2+dist_axis_x+0.561+window_depth/2} ${-0.5-dist_axis_y} ${size_z_wall2/2}" rpy="0 0 -0.785398" />
+		<origin xyz="${size_total_x/2+dist_axis_x+0.61+window_depth/2} ${-0.54-dist_axis_y} ${size_z_wall2/2}" rpy="0 0 -0.785398" />
 		<parent link="dummy_link" />
 		<child link="wall_04" />
@@ -172,5 +259,5 @@
 	</link>
 	<gazebo reference="wall_05">
-		<material>IPA/WallApartment</material>
+		<material>wall_floor_05</material>
 	</gazebo>
 	<joint name="joint_wall_05" type="fixed">
@@ -201,5 +288,5 @@
 	</link>
 	<gazebo reference="wall_06">
-		<material>IPA/WallApartment</material>
+		<material>wall_livingroom1</material>
 	</gazebo>
 	<joint name="joint_wall_06" type="fixed">
@@ -230,5 +317,5 @@
 	</link>
 	<gazebo reference="wall_07">
-		<material>IPA/WallApartment</material>
+		<material>wall_floor_05</material>
 	</gazebo>
 	<joint name="joint_wall_07" type="fixed">
@@ -237,33 +324,4 @@
 		<child link="wall_07" />
 	</joint>
-	<!-- wall_08 -->
-	<link name="wall_08">
-		<inertial>
-			<origin xyz="0 0 0" />
-			<mass value="5.0" />
-			<inertia ixx="0.0" ixy="0.0" ixz="0.0" iyy="0.0" iyz="0.0" izz="0.0" />
-		</inertial>
-		<visual>
-			<origin xyz="0 0 0" />
-			<geometry>
-				<box size="${wall_depth} 1.9 ${size_z_wall2}" />
-			</geometry>
-			<material name="IPA/Grey"/>
-		</visual>
-		<collision>
-			<origin xyz="0 0 0" />
-			<geometry>
-				<box size="${wall_depth} 1.9 ${size_z_wall2}" />
-			</geometry>
-		</collision>
-	</link>
-	<gazebo reference="wall_08">
-		<material>IPA/WallApartment</material>
-	</gazebo>
-	<joint name="joint_wall_08" type="fixed">
-		<origin xyz="${size_total_x/2-1.8+dist_axis_x+wall_depth} ${size_total_y/2-3.6+0.1-dist_axis_y} ${size_z_wall2/2}" rpy="0 0 0" />
-		<parent link="dummy_link" />
-		<child link="wall_08" />
-	</joint>
 	<!-- door_00 -->
 	<link name="door_00">

File: cob_gazebo_worlds/urdf/ipa-apartment/elevator.urdf.xacro (robot description, xacro)
@@ -90,5 +90,5 @@
 	</link>
 	<gazebo reference="wall_elv5">
-		<material>IPA/WallApartment</material>
+		<material>wall_floor_07</material>
 	</gazebo>
 	<joint name="joint_wall_elv5" type="fixed">
@@ -119,5 +119,5 @@
 	</link>
 	<gazebo reference="wall_elv6">
-		<material>IPA/WallApartment</material>
+		<material>wall_floor_07</material>
 	</gazebo>
 	<joint name="joint_wall_elv6" type="fixed">
@@ -148,5 +148,5 @@
 	</link>
 	<gazebo reference="elevator_left2">
-		<material>IPA/WallApartment</material>
+		<material>wall_floor_07</material>
 	</gazebo>
 	<joint name="joint_elevator_left2" type="fixed">
@@ -216,5 +216,5 @@
 	</link>
 	<gazebo reference="wall_elv7">
-		<material>IPA/WallApartment</material>
+		<material>wall_floor_07</material>
 	</gazebo>
 	<joint name="joint_wall_elv7" type="fixed">
@@ -245,5 +245,5 @@
 	</link>
 	<gazebo reference="wall_elv8">
-		<material>IPA/WallApartment</material>
+		<material>wall_floor_07</material>
 	</gazebo>
 	<joint name="joint_wall_elv8" type="fixed">
@@ -274,5 +274,5 @@
 	</link>
 	<gazebo reference="elevator_right2">
-		<material>IPA/WallApartment</material>
+		<material>wall_floor_07</material>
 	</gazebo>
 	<joint name="joint_elevator_right2" type="fixed">
@@ -397,5 +397,5 @@
 	</link>
 	<gazebo reference="wall_ext18">
-		<material>IPA/WallApartment</material>
+		<material>wall_floor_07</material>
 	</gazebo>
 	<joint name="joint_wall_ext18" type="fixed">
@@ -425,5 +425,5 @@
 	</link>
 	<gazebo reference="wall_ext19">
-		<material>IPA/WallApartment</material>
+		<material>wall_floor_07</material>
 	</gazebo>
 	<joint name="joint_wall_ext19" type="fixed">
@@ -453,5 +453,5 @@
 	</link>
 	<gazebo reference="wall_ext20">
-		<material>IPA/WallApartment</material>
+		<material>wall_floor_07</material>
 	</gazebo>
 	<joint name="joint_wall_ext20" type="fixed">

File: cob_gazebo_worlds/urdf/ipa-apartment/ipa-apartment.urdf.xacro (robot description, xacro)
@@ -30,9 +30,9 @@
 	  <property name="size_c" value="1.8" />
 	  <property name="size_d" value="4.16" />
-	  <property name="wall_depth" value="0.06" />
+	  <property name="wall_depth" value="0.1" />
 	  <property name="window_depth" value="0.15" />
-	  <property name="size_z_wall1" value="2" />
-	  <property name="size_z_wall2" value="0.92" />
-	  <property name="size_z_wall3" value="1.4" />
+	  <property name="size_z_wall1" value="2.7" />
+	  <property name="size_z_wall2" value="2.7" />
+	  <property name="size_z_wall3" value="2.7" />
 <xacro:macro name="ipa-apartment" params="name">
 	<!-- dummy_link -->
