Commit message: New wall textures and floor for ipa-apartment environment

File: cob_gazebo_worlds/urdf/ipa-apartment/landing.urdf.xacro (robot description, xacro)
@@ -39,12 +39,12 @@
 			<origin xyz="0 0 0" />
 			<geometry>
-				<box size="2.1 0.04 ${size_z_wall1}" />
-			</geometry>
-			<material name="IPA/Grey"/>
-		</visual>
-		<collision>
-			<origin xyz="0 0 0" />
-			<geometry>
-				<box size="2.1 0.04 ${size_z_wall1}" />
+				<box size="2.1 ${wall_depth} ${size_z_wall1}" />
+			</geometry>
+			<material name="IPA/Grey"/>
+		</visual>
+		<collision>
+			<origin xyz="0 0 0" />
+			<geometry>
+				<box size="2.1 ${wall_depth} ${size_z_wall1}" />
 			</geometry>
 		</collision>
@@ -68,20 +68,20 @@
 			<origin xyz="0 0 0" />
 			<geometry>
-				<box size="2.1 0.04 ${size_z_wall1}" />
-			</geometry>
-			<material name="IPA/Grey"/>
-		</visual>
-		<collision>
-			<origin xyz="0 0 0" />
-			<geometry>
-				<box size="2.1 0.04 ${size_z_wall1}" />
+				<box size="2.2 ${wall_depth} ${size_z_wall1}" />
+			</geometry>
+			<material name="IPA/Grey"/>
+		</visual>
+		<collision>
+			<origin xyz="0 0 0" />
+			<geometry>
+				<box size="2.2 ${wall_depth} ${size_z_wall1}" />
 			</geometry>
 		</collision>
 	</link>
 	<gazebo reference="wall_ext2">
-		<material>IPA/WallApartment</material>
+		<material>door_E334</material>
 	</gazebo>
 	<joint name="joint_wall_ext2" type="fixed">
-		<origin xyz="8.8 -2.565 ${size_z_wall1/2}" rpy="0 0 0" />
+		<origin xyz="8.70 -1.565 ${size_z_wall1/2}" rpy="0 0 0" />
 		<parent link="origin_landing" />
 		<child link="wall_ext2" />
@@ -97,20 +97,20 @@
 			<origin xyz="0 0 0" />
 			<geometry>
-				<box size="0.04 1.73 ${size_z_wall1}" />
-			</geometry>
-			<material name="IPA/Grey"/>
-		</visual>
-		<collision>
-			<origin xyz="0 0 0" />
-			<geometry>
-				<box size="0.04 1.73 ${size_z_wall1}" />
+				<box size="${wall_depth} 1.73 ${size_z_wall1}" />
+			</geometry>
+			<material name="IPA/Grey"/>
+		</visual>
+		<collision>
+			<origin xyz="0 0 0" />
+			<geometry>
+				<box size="${wall_depth} 1.73 ${size_z_wall1}" />
 			</geometry>
 		</collision>
 	</link>
 	<gazebo reference="wall_ext3">
-		<material>IPA/WallApartment</material>
+		<material>wall_floor_07</material>
 	</gazebo>
 	<joint name="joint_wall_ext3" type="fixed">
-		<origin xyz="7.75 -1.7 ${size_z_wall1/2}" rpy="0 0 0" />
+		<origin xyz="7.6 -1.7 ${size_z_wall1/2}" rpy="0 0 0" />
 		<parent link="origin_landing" />
 		<child link="wall_ext3" />
@@ -126,20 +126,20 @@
 			<origin xyz="0 0 0" />
 			<geometry>
-				<box size="0.04 1.73 ${size_z_wall1}" />
-			</geometry>
-			<material name="IPA/Grey"/>
-		</visual>
-		<collision>
-			<origin xyz="0 0 0" />
-			<geometry>
-				<box size="0.04 1.73 ${size_z_wall1}" />
+				<box size="${wall_depth} 1.93 ${size_z_wall1}" />
+			</geometry>
+			<material name="IPA/Grey"/>
+		</visual>
+		<collision>
+			<origin xyz="0 0 0" />
+			<geometry>
+				<box size="${wall_depth} 1.93 ${size_z_wall1}" />
 			</geometry>
 		</collision>
 	</link>
 	<gazebo reference="wall_ext4">
-		<material>IPA/WallApartment</material>
+		<material>wall_floor_07</material>
 	</gazebo>
 	<joint name="joint_wall_ext4" type="fixed">
-		<origin xyz="7.75 1.7 ${size_z_wall1/2}" rpy="0 0 0" />
+		<origin xyz="7.58 1.83 ${size_z_wall1/2}" rpy="0 0 0" />
 		<parent link="origin_landing" />
 		<child link="wall_ext4" />
@@ -154,20 +154,20 @@
 			<origin xyz="0 0 0" />
 			<geometry>
-				<box size="2.34 0.04 ${size_z_wall1}" />
-			</geometry>
-			<material name="IPA/Grey"/>
-		</visual>
-		<collision>
-			<origin xyz="0 0 0" />
-			<geometry>
-				<box size="6.73 0.04 ${size_z_wall1}" />
+				<box size="2.24 0.04 ${size_z_wall1}" />
+			</geometry>
+			<material name="IPA/Grey"/>
+		</visual>
+		<collision>
+			<origin xyz="0 0 0" />
+			<geometry>
+				<box size="2.24 ${wall_depth} ${size_z_wall1}" />
 			</geometry>
 		</collision>
 	</link>
 	<gazebo reference="wall_ext5">
-		<material>IPA/WallApartment</material>
+		<material>door_opposite_of_men_toilet</material>
 	</gazebo>
 	<joint name="joint_wall_ext5" type="fixed">
-		<origin xyz="6.6 -0.85 ${size_z_wall1/2}" rpy="0 0 0" />
+		<origin xyz="6.55 -0.85 ${size_z_wall1/2}" rpy="0 0 0" />
 		<parent link="origin_landing" />
 		<child link="wall_ext5" />
@@ -182,20 +182,20 @@
 			<origin xyz="0 0 0" />
 			<geometry>
-				<box size="2.34 0.04 ${size_z_wall1}" />
-			</geometry>
-			<material name="IPA/Grey"/>
-		</visual>
-		<collision>
-			<origin xyz="0 0 0" />
-			<geometry>
-				<box size="2.34 0.04 ${size_z_wall1}" />
+				<box size="2.24 0.04 ${size_z_wall1}" />
+			</geometry>
+			<material name="IPA/Grey"/>
+		</visual>
+		<collision>
+			<origin xyz="0 0 0" />
+			<geometry>
+				<box size="2.24 0.04 ${size_z_wall1}" />
 			</geometry>
 		</collision>
 	</link>
 	<gazebo reference="wall_ext6">
-		<material>IPA/WallApartment</material>
+		<material>door_toilet_men</material>
 	</gazebo>
 	<joint name="joint_wall_ext6" type="fixed">
-		<origin xyz="6.6 0.85 ${size_z_wall1/2}" rpy="0 0 0" />
+		<origin xyz="6.55 0.85 ${size_z_wall1/2}" rpy="0 0 0" />
 		<parent link="origin_landing" />
 		<child link="wall_ext6" />
@@ -211,12 +211,12 @@
 			<origin xyz="0 0 0" />
 			<geometry>
-				<box size="0.04 2.1 ${size_z_wall1}" />
-			</geometry>
-			<material name="IPA/Grey"/>
-		</visual>
-		<collision>
-			<origin xyz="0 0 0" />
-			<geometry>
-				<box size="0.04 2.1 ${size_z_wall1}" />
+				<box size="${wall_depth} 2.1 ${size_z_wall1}" />
+			</geometry>
+			<material name="IPA/Grey"/>
+		</visual>
+		<collision>
+			<origin xyz="0 0 0" />
+			<geometry>
+				<box size="${wall_depth} 2.1 ${size_z_wall1}" />
 			</geometry>
 		</collision>
@@ -240,20 +240,20 @@
 			<origin xyz="0 0 0" />
 			<geometry>
-				<box size="0.04 2.1 ${size_z_wall1}" />
-			</geometry>
-			<material name="IPA/Grey"/>
-		</visual>
-		<collision>
-			<origin xyz="0 0 0" />
-			<geometry>
-				<box size="0.04 2.1 ${size_z_wall1}" />
+				<box size="${wall_depth} 2.3 ${size_z_wall1}" />
+			</geometry>
+			<material name="IPA/Grey"/>
+		</visual>
+		<collision>
+			<origin xyz="0 0 0" />
+			<geometry>
+				<box size="${wall_depth} 2.3 ${size_z_wall1}" />
 			</geometry>
 		</collision>
 	</link>
 	<gazebo reference="wall_ext8">
-		<material>IPA/WallApartment</material>
+		<material>wall_floor_05</material>
 	</gazebo>
 	<joint name="joint_wall_ext8" type="fixed">
-		<origin xyz="-2.565 8.8 ${size_z_wall1/2}" rpy="0 0 0" />
+		<origin xyz="-2.565 8.7 ${size_z_wall1/2}" rpy="0 0 0" />
 		<parent link="origin_landing" />
 		<child link="wall_ext8" />
@@ -269,20 +269,20 @@
 			<origin xyz="0 0 0" />
 			<geometry>
-				<box size="1.73 0.04 ${size_z_wall1}" />
-			</geometry>
-			<material name="IPA/Grey"/>
-		</visual>
-		<collision>
-			<origin xyz="0 0 0" />
-			<geometry>
-				<box size="1.73 0.04 ${size_z_wall1}" />
+				<box size="1.73 ${wall_depth} ${size_z_wall1}" />
+			</geometry>
+			<material name="IPA/Grey"/>
+		</visual>
+		<collision>
+			<origin xyz="0 0 0" />
+			<geometry>
+				<box size="1.73 ${wall_depth} ${size_z_wall1}" />
 			</geometry>
 		</collision>
 	</link>
 	<gazebo reference="wall_ext9">
-		<material>IPA/WallApartment</material>
+		<material>wall_floor_07</material>
 	</gazebo>
 	<joint name="joint_wall_ext9" type="fixed">
-		<origin xyz="-1.7 7.75 ${size_z_wall1/2}" rpy="0 0 0" />
+		<origin xyz="-1.8 7.50 ${size_z_wall1/2}" rpy="0 0 0" />
 		<parent link="origin_landing" />
 		<child link="wall_ext9" />
@@ -298,20 +298,20 @@
 			<origin xyz="0 0 0" />
 			<geometry>
-				<box size="1.73 0.04 ${size_z_wall1}" />
-			</geometry>
-			<material name="IPA/Grey"/>
-		</visual>
-		<collision>
-			<origin xyz="0 0 0" />
-			<geometry>
-				<box size="1.73 0.04 ${size_z_wall1}" />
+				<box size="1.96 ${wall_depth} ${size_z_wall1}" />
+			</geometry>
+			<material name="IPA/Grey"/>
+		</visual>
+		<collision>
+			<origin xyz="0 0 0" />
+			<geometry>
+				<box size="1.96 ${wall_depth} ${size_z_wall1}" />
 			</geometry>
 		</collision>
 	</link>
 	<gazebo reference="wall_ext10">
-		<material>IPA/WallApartment</material>
+		<material>wall_floor_07</material>
 	</gazebo>
 	<joint name="joint_wall_ext10" type="fixed">
-		<origin xyz="1.7 7.75 ${size_z_wall1/2}" rpy="0 0 0" />
+		<origin xyz="1.89 7.53 ${size_z_wall1/2}" rpy="0 0 0" />
 		<parent link="origin_landing" />
 		<child link="wall_ext10" />
@@ -326,20 +326,20 @@
 			<origin xyz="0 0 0" />
 			<geometry>
-				<box size="0.04 2.34 ${size_z_wall1}" />
-			</geometry>
-			<material name="IPA/Grey"/>
-		</visual>
-		<collision>
-			<origin xyz="0 0 0" />
-			<geometry>
-				<box size="0.04 2.34 ${size_z_wall1}" />
+				<box size="0.04 2.24 ${size_z_wall1}" />
+			</geometry>
+			<material name="IPA/Grey"/>
+		</visual>
+		<collision>
+			<origin xyz="0 0 0" />
+			<geometry>
+				<box size="0.04 2.24 ${size_z_wall1}" />
 			</geometry>
 		</collision>
 	</link>
 	<gazebo reference="wall_ext11">
-		<material>IPA/WallApartment</material>
+		<material>door_women_toilet</material>
 	</gazebo>
 	<joint name="joint_wall_ext11" type="fixed">
-		<origin xyz="-0.85 6.6 ${size_z_wall1/2}" rpy="0 0 0" />
+		<origin xyz="-0.85 6.55 ${size_z_wall1/2}" rpy="0 0 0" />
 		<parent link="origin_landing" />
 		<child link="wall_ext11" />
@@ -354,20 +354,20 @@
 			<origin xyz="0 0 0" />
 			<geometry>
-				<box size="0.04 2.34 ${size_z_wall1}" />
-			</geometry>
-			<material name="IPA/Grey"/>
-		</visual>
-		<collision>
-			<origin xyz="0 0 0" />
-			<geometry>
-				<box size="0.04 2.34 ${size_z_wall1}" />
+				<box size="0.04 2.24 ${size_z_wall1}" />
+			</geometry>
+			<material name="IPA/Grey"/>
+		</visual>
+		<collision>
+			<origin xyz="0 0 0" />
+			<geometry>
+				<box size="0.04 2.24 ${size_z_wall1}" />
 			</geometry>
 		</collision>
 	</link>
 	<gazebo reference="wall_ext12">
-		<material>IPA/WallApartment</material>
+		<material>door_E322</material>
 	</gazebo>
 	<joint name="joint_wall_ext12" type="fixed">
-		<origin xyz="0.85 6.6 ${size_z_wall1/2}" rpy="0 0 0" />
+		<origin xyz="0.85 6.55 ${size_z_wall1/2}" rpy="0 0 0" />
 		<parent link="origin_landing" />
 		<child link="wall_ext12" />
@@ -394,5 +394,5 @@
 	</link>
 	<gazebo reference="wall_ext13">
-		<material>IPA/WallApartment</material>
+		<material>wall_floor_07</material>
 	</gazebo>
 	<joint name="joint_wall_ext13" type="fixed">
@@ -410,17 +410,17 @@
 			<origin xyz="0 0 0" />
 			<geometry>
-				<box size="0.04 6.6 ${size_z_wall1}" />
-			</geometry>
-			<material name="IPA/Grey"/>
-		</visual>
-		<collision>
-			<origin xyz="0 0 0" />
-			<geometry>
-				<box size="0.04 6.6 ${size_z_wall1}" />
+				<box size="${wall_depth} 6.6 ${size_z_wall1}" />
+			</geometry>
+			<material name="IPA/Grey"/>
+		</visual>
+		<collision>
+			<origin xyz="0 0 0" />
+			<geometry>
+				<box size="${wall_depth} 6.6 ${size_z_wall1}" />
 			</geometry>
 		</collision>
 	</link>
 	<gazebo reference="wall_ext14">
-		<material>IPA/WallApartment</material>
+		<material>wall_floor_07</material>
 	</gazebo>
 	<joint name="joint_wall_ext14" type="fixed">
@@ -429,5 +429,4 @@
 		<child link="wall_ext14" />
 	</joint>
-        </xacro:macro>
 <link name="wall_ext15">
 		<inertial>
@@ -451,5 +450,5 @@
 	</link>
 	<gazebo reference="wall_ext15">
-		<material>IPA/WallApartment</material>
+		<material>wall_floor_07</material>
 	</gazebo>
 	<joint name="joint_wall_ext15" type="fixed">
@@ -479,5 +478,5 @@
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
File: cob_gazebo_worlds/urdf/ipa-apartment/office.urdf.xacro (robot description, xacro)
@@ -51,5 +51,5 @@
 	</link>
 	<gazebo reference="wall_office_00">
-		<material>IPA/WallApartment</material>
+		<material>wall_floor_05</material>
 	</gazebo>
 	<joint name="joint_wall_office_00" type="fixed">
@@ -68,20 +68,20 @@
 			<origin xyz="0 0 0" />
 			<geometry>
-				<box size="4.65 ${wall_depth} ${size_z_wall1}" />
-			</geometry>
-			<material name="IPA/Grey"/>
-		</visual>
-		<collision>
-			<origin xyz="0 0 0" />
-			<geometry>
-				<box size="4.65 ${wall_depth} ${size_z_wall1}" />
+				<box size="4.4 ${wall_depth} ${size_z_wall1}" />
+			</geometry>
+			<material name="IPA/Grey"/>
+		</visual>
+		<collision>
+			<origin xyz="0 0 0" />
+			<geometry>
+				<box size="4.4 ${wall_depth} ${size_z_wall1}" />
 			</geometry>
 		</collision>
 	</link>
 	<gazebo reference="wall_office_01">
-		<material>IPA/WallApartment</material>
+		<material>wall_floor_11</material>
 	</gazebo>
 	<joint name="joint_wall_office_01" type="fixed">
-		<origin xyz="-3.25 -4.15 ${size_z_wall1/2}" rpy="0 0 0" />
+		<origin xyz="-3.25 -4.22 ${size_z_wall1/2}" rpy="0 0 0" />
 		<parent link="origin_office" />
 		<child link="wall_office_01" />
@@ -109,5 +109,5 @@
 	</link>
 	<gazebo reference="wall_office_02">
-		<material>IPA/WallApartment</material>
+		<material>wall_livingroom1</material>
 	</gazebo>
 	<joint name="joint_wall_office_02" type="fixed">
@@ -138,8 +138,8 @@
 	</link>
 	<gazebo reference="wall_office_03">
-		<material>IPA/WallApartment</material>
+		<material>wall_livingroom1</material>
 	</gazebo>
 	<joint name="joint_wall_office_03" type="fixed">
-		<origin xyz="-5.6 0 ${size_z_wall2/2}" rpy="0 0 0" />
+		<origin xyz="-5.6 -0.1 ${size_z_wall2/2}" rpy="0 0 0" />
 		<parent link="origin_office" />
 		<child link="wall_office_03" />
@@ -167,5 +167,5 @@
 	</link>
 	<gazebo reference="wall_office_04">
-		<material>IPA/WallApartment</material>
+		<material>wall_livingroom1</material>
 	</gazebo>
 	<joint name="joint_wall_office_04" type="fixed">
@@ -184,20 +184,20 @@
 			<origin xyz="0 0 0" />
 			<geometry>
-				<box size="${wall_depth} 4.51 ${size_z_wall1}" />
-			</geometry>
-			<material name="IPA/Grey"/>
-		</visual>
-		<collision>
-			<origin xyz="0 0 0" />
-			<geometry>
-				<box size="${wall_depth} 4.51 ${size_z_wall1}" />
+				<box size="${wall_depth} 4.21 ${size_z_wall1}" />
+			</geometry>
+			<material name="IPA/Grey"/>
+		</visual>
+		<collision>
+			<origin xyz="0 0 0" />
+			<geometry>
+				<box size="${wall_depth} 4.21 ${size_z_wall1}" />
 			</geometry>
 		</collision>
 	</link>
 	<gazebo reference="wall_office_05">
-		<material>IPA/WallApartment</material>
+		<material>wall_floor_05</material>
 	</gazebo>
 	<joint name="joint_wall_office_05" type="fixed">
-		<origin xyz="1.09 -0.615 ${size_z_wall1/2}" rpy="0 0 0" />
+		<origin xyz="0.95 -0.52 ${size_z_wall1/2}" rpy="0 0 0" />
 		<parent link="origin_office" />
 		<child link="wall_office_05" />
@@ -213,20 +213,20 @@
 			<origin xyz="0 0 0" />
 			<geometry>
-				<box size="${wall_depth} 1.23 ${size_z_wall1}" />
-			</geometry>
-			<material name="IPA/Grey"/>
-		</visual>
-		<collision>
-			<origin xyz="0 0 0" />
-			<geometry>
-				<box size="${wall_depth} 1.23 ${size_z_wall1}" />
+				<box size="${wall_depth} 1.40 ${size_z_wall1}" />
+			</geometry>
+			<material name="IPA/Grey"/>
+		</visual>
+		<collision>
+			<origin xyz="0 0 0" />
+			<geometry>
+				<box size="${wall_depth} 1.40 ${size_z_wall1}" />
 			</geometry>
 		</collision>
 	</link>
 	<gazebo reference="wall_office_06">
-		<material>IPA/WallApartment</material>
+		<material>wall_floor_06</material>
 	</gazebo>
 	<joint name="joint_wall_office_06" type="fixed">
-		<origin xyz="1.09 3.385 ${size_z_wall1/2}" rpy="0 0 0" />
+		<origin xyz="0.95 3.28 ${size_z_wall1/2}" rpy="0 0 0" />
 		<parent link="origin_office" />
 		<child link="wall_office_06" />
@@ -254,5 +254,5 @@
 	</link>
 	<gazebo reference="wall_office_07">
-		<material>IPA/WallApartment</material>
+		<material>wall_floor_07</material>
 	</gazebo>
 	<joint name="joint_wall_office_07" type="fixed">
@@ -283,5 +283,5 @@
 	</link>
 	<gazebo reference="wall_office_08">
-		<material>IPA/WallApartment</material>
+		<material>wall_floor_08</material>
 	</gazebo>
 	<joint name="joint_wall_office_08" type="fixed">
@@ -300,20 +300,20 @@
 			<origin xyz="0 0 0" />
 			<geometry>
-				<box size="4.5 ${wall_depth} ${size_z_wall1}" />
-			</geometry>
-			<material name="IPA/Grey"/>
-		</visual>
-		<collision>
-			<origin xyz="0 0 0" />
-			<geometry>
-				<box size="4.5 ${wall_depth} ${size_z_wall1}" />
+				<box size="4.53 ${wall_depth} ${size_z_wall1}" />
+			</geometry>
+			<material name="IPA/Grey"/>
+		</visual>
+		<collision>
+			<origin xyz="0 0 0" />
+			<geometry>
+				<box size="4.53 ${wall_depth} ${size_z_wall1}" />
 			</geometry>
 		</collision>
 	</link>
 	<gazebo reference="wall_office_09">
-		<material>IPA/WallApartment</material>
+		<material>wall_bedroom1</material>
 	</gazebo>
 	<joint name="joint_wall_office_09" type="fixed">
-		<origin xyz="3.35 1.64 ${size_z_wall1/2}" rpy="0 0 0" />
+		<origin xyz="3.26 1.32 ${size_z_wall1/2}" rpy="0 0 0" />
 		<parent link="origin_office" />
 		<child link="wall_office_09" />
@@ -341,5 +341,5 @@
 	</link>
 	<gazebo reference="wall_office_10">
-		<material>IPA/WallApartment</material>
+		<material>wall_bedroom1</material>
 	</gazebo>
 	<joint name="joint_wall_office_10" type="fixed">
