Commit message: fix environment descriptions according to new gazebo format

File: cob_gazebo_worlds/urdf/ipa-apartment/elevator.urdf.xacro (robot description, xacro)
@@ -313,4 +313,10 @@
                 <gazebo reference="elevator_button1">
                         <selfCollide>true</selfCollide>
+                        <sensor name='elevator_button1_contact_sensor' type='contact'>
+							<contact>
+								<collision>elevator_button1_geom</collision>
+							</contact>
+						</sensor>
+<!--
                         <sensor:contact name="elevator_button1_contact_sensor">
                                 <geom>elevator_button1_geom</geom>
@@ -324,4 +330,5 @@
                                 </controller:gazebo_ros_bumper>
                         </sensor:contact>
+-->
                         <material>Gazebo/Red</material>
                 </gazebo>
@@ -357,4 +364,10 @@
  		<gazebo reference="elevator_button2">
                         <selfCollide>true</selfCollide>
+                        <sensor name='elevator_button2_contact_sensor' type='contact'>
+							<contact>
+								<collision>elevator_button2_geom</collision>
+							</contact>
+						</sensor>
+<!--
                         <sensor:contact name="elevator_button2_contact_sensor">
                                 <geom>elevator_button2_geom</geom>
@@ -368,4 +381,5 @@
                                 </controller:gazebo_ros_bumper>
                         </sensor:contact>
+-->
                         <material>Gazebo/Red</material>
                         <turnGravityOff>false</turnGravityOff>

Commit message: some cleaning up

File: cob_gazebo_worlds/urdf/ipa-apartment/elevator.urdf.xacro (robot description, xacro)
@@ -4,5 +4,5 @@
        xmlns:interface="http://playerstage.sourceforge.net/gazebo/xmlschema/#interface"
        xmlns:xacro="http://ros.org/wiki/xacro">
-        <xacro:macro name="elevator" params="name">
+	<xacro:macro name="elevator" params="name">
 	<link name="origin_elevator">
 		<inertial>
@@ -63,9 +63,9 @@
 		<!--safety_controller k_velocity="10"/-->
 	</joint>
-         <transmission name="elevator_left_trans" type="pr2_mechanism_model/SimpleTransmission">
-                   <actuator name="elevator_left_motor"/>
-                   <joint name="elevator_left_joint"/>
-                   <mechanicalReduction>1</mechanicalReduction>
-         </transmission>
+	<transmission name="elevator_left_trans" type="pr2_mechanism_model/SimpleTransmission">
+		<actuator name="elevator_left_motor"/>
+		<joint name="elevator_left_joint"/>
+		<mechanicalReduction>1</mechanicalReduction>
+	</transmission>
 	<!-- wall elv5 -->
 	<link name="wall_elv5">
@@ -189,9 +189,9 @@
 		<safety_controller k_velocity="10"/>
 	</joint>
-         <transmission name="elevator_right_trans" type="pr2_mechanism_model/SimpleTransmission">
-                   <actuator name="elevator_right_motor"/>
-                   <joint name="elevator_right_joint"/>
-                   <mechanicalReduction>1</mechanicalReduction>
-        </transmission>
+	<transmission name="elevator_right_trans" type="pr2_mechanism_model/SimpleTransmission">
+	   <actuator name="elevator_right_motor"/>
+	   <joint name="elevator_right_joint"/>
+	   <mechanicalReduction>1</mechanicalReduction>
+	</transmission>
 	<!-- wall elv7 -->
 	<link name="wall_elv7">
@@ -311,26 +311,22 @@
 		<safety_controller k_velocity="10"/>
 	</joint>
-                <gazebo reference="elevator_button1">
-                        <selfCollide>true</selfCollide>
-                        <sensor name='elevator_button1_contact_sensor' type='contact'>
-							<contact>
-								<collision>elevator_button1_geom</collision>
-							</contact>
-						</sensor>
-<!--
-                        <sensor:contact name="elevator_button1_contact_sensor">
-                                <geom>elevator_button1_geom</geom>
-                                <updateRate>10</updateRate>
-                                <controller:gazebo_ros_bumper name="elevator_button1_gazebo_ros_bumper_controller" plugin="libgazebo_ros_bumper.so">
-                                        <alwaysOn>true</alwaysOn>
-                                        <updateRate>10</updateRate>
-                                        <frameName>elevator_button1</frameName>
-                                        <bumperTopicName>elevator_button1_bumper</bumperTopicName>
-                                        <interface:bumper name="elevator_button1_bumper_iface" />
-                                </controller:gazebo_ros_bumper>
-                        </sensor:contact>
--->
-                        <material>Gazebo/Red</material>
-                </gazebo>
+	<gazebo reference="elevator_button1">
+		<selfCollide>true</selfCollide>
+        <sensor name='elevator_button1_contact_sensor' type='contact'>
+			<always_on>true</always_on>
+			<update_rate>10</update_rate>
+			<contact>
+				<collision>elevator_button1_geom</collision>
+			</contact>
+			<plugin name="elevator_button1_gazebo_ros_bumper_controller" plugin="libgazebo_ros_bumper.so">
+				<alwaysOn>true</alwaysOn>
+				<updateRate>10</updateRate>
+				<frameName>elevator_button1</frameName>
+				<bumperTopicName>elevator_button1_bumper</bumperTopicName>
+			</plugin>
+		</sensor>
+		<material>Gazebo/Red</material>
+		<turnGravityOff>false</turnGravityOff>
+	</gazebo>
 	<link name="elevator_button2">
 		<inertial>
@@ -362,28 +358,23 @@
 		<safety_controller k_velocity="10"/>
 	</joint>
- 		<gazebo reference="elevator_button2">
-                        <selfCollide>true</selfCollide>
-                        <sensor name='elevator_button2_contact_sensor' type='contact'>
-							<contact>
-								<collision>elevator_button2_geom</collision>
-							</contact>
-						</sensor>
-<!--
-                        <sensor:contact name="elevator_button2_contact_sensor">
-                                <geom>elevator_button2_geom</geom>
-                                <updateRate>10</updateRate>
-                                <controller:gazebo_ros_bumper name="elevator_button2_gazebo_ros_bumper_controller" plugin="libgazebo_ros_bumper.so">
-                                        <alwaysOn>true</alwaysOn>
-                                        <updateRate>10</updateRate>
-                                        <frameName>elevator_button2</frameName>
-                                        <bumperTopicName>elevator_button2_bumper</bumperTopicName>
-                                        <interface:bumper name="elevator_button2_bumper_iface" />
-                                </controller:gazebo_ros_bumper>
-                        </sensor:contact>
--->
-                        <material>Gazebo/Red</material>
-                        <turnGravityOff>false</turnGravityOff>
-                </gazebo>
-<link name="wall_ext18">
+	<gazebo reference="elevator_button2">
+		<selfCollide>true</selfCollide>
+        <sensor name='elevator_button2_contact_sensor' type='contact'>
+			<always_on>true</always_on>
+			<update_rate>10</update_rate>
+			<contact>
+				<collision>elevator_button2_geom</collision>
+			</contact>
+			<plugin name="elevator_button2_gazebo_ros_bumper_controller" plugin="libgazebo_ros_bumper.so">
+				<alwaysOn>true</alwaysOn>
+				<updateRate>10</updateRate>
+				<frameName>elevator_button2</frameName>
+				<bumperTopicName>elevator_button2_bumper</bumperTopicName>
+			</plugin>
+		</sensor>
+		<material>Gazebo/Red</material>
+		<turnGravityOff>false</turnGravityOff>
+	</gazebo>
+	<link name="wall_ext18">
 		<inertial>
 			<origin xyz="0 0 0" />
@@ -413,5 +404,5 @@
 		<child link="wall_ext18" />
 	</joint>
-        <link name="wall_ext19">
+	<link name="wall_ext19">
 		<inertial>
 			<origin xyz="0 0 0" />
@@ -441,5 +432,5 @@
 		<child link="wall_ext19" />
 	</joint>
-        <link name="wall_ext20">
+	<link name="wall_ext20">
 		<inertial>
 			<origin xyz="0 0 0" />
@@ -469,4 +460,4 @@
 		<child link="wall_ext20" />
 	</joint>
-        </xacro:macro>
+	</xacro:macro>
 </robot>

Commit message: change to latest transmission format

File: cob_gazebo_worlds/urdf/ipa-apartment/elevator.urdf.xacro (robot description, xacro)
@@ -60,8 +60,12 @@
     <!--safety_controller k_velocity="10"/-->
   </joint>
-  <transmission name="elevator_left_trans" type="pr2_mechanism_model/SimpleTransmission">
-    <actuator name="elevator_left_motor"/>
-    <joint name="elevator_left_joint"/>
-    <mechanicalReduction>1</mechanicalReduction>
+  <transmission name="elevator_left_trans">
+    <type>transmission_interface/SimpleTransmission</type>
+    <joint name="elevator_left_joint">
+      <hardwareInterface>EffortJointInterface</hardwareInterface>
+    </joint>
+    <actuator name="elevator_left_motor">
+      <mechanicalReduction>1</mechanicalReduction>
+    </actuator>
   </transmission>
   <!-- wall elv5 -->
@@ -186,8 +190,12 @@
     <safety_controller k_velocity="10"/>
   </joint>
-  <transmission name="elevator_right_trans" type="pr2_mechanism_model/SimpleTransmission">
-     <actuator name="elevator_right_motor"/>
-     <joint name="elevator_right_joint"/>
-     <mechanicalReduction>1</mechanicalReduction>
+  <transmission name="elevator_right_trans">
+    <type>transmission_interface/SimpleTransmission</type>
+    <joint name="elevator_right_joint">
+      <hardwareInterface>EffortJointInterface</hardwareInterface>
+    </joint>
+    <actuator name="elevator_right_motor">
+      <mechanicalReduction>1</mechanicalReduction>
+    </actuator>
   </transmission>
   <!-- wall elv7 -->

Commit message: fix bumper plugin

File: cob_gazebo_worlds/urdf/ipa-apartment/elevator.urdf.xacro (robot description, xacro)
@@ -316,22 +316,21 @@
     <safety_controller k_velocity="10"/>
   </joint>
-  <!--gazebo reference="elevator_button1">
-    <selfCollide>true</selfCollide>
-        <sensor name='elevator_button1_contact_sensor' type='contact'>
-      <always_on>true</always_on>
+  <gazebo reference="elevator_button1">
+    <gravity>true</gravity>
+    <self_collide>false</self_collide>
+    <material>Gazebo/Red</material>
+    <sensor name='elevator_button1_contact_sensor' type='contact'>
+      <always_on>1</always_on>
       <update_rate>10</update_rate>
       <contact>
-        <collision>elevator_button1_geom</collision>
+        <collision>elevator_button1_collision</collision>
+        <topic>elevator_button1_bumper</topic>
       </contact>
       <plugin name="elevator_button1_gazebo_ros_bumper_controller" filename="libgazebo_ros_bumper.so">
-        <alwaysOn>true</alwaysOn>
-        <updateRate>10</updateRate>
         <frameName>elevator_button1</frameName>
         <bumperTopicName>elevator_button1_bumper</bumperTopicName>
       </plugin>
     </sensor>
-    <material>Gazebo/Red</material>
-    <turnGravityOff>false</turnGravityOff>
-  </gazebo-->
+  </gazebo>
   <link name="elevator_button2">
     <inertial>
@@ -363,22 +362,21 @@
     <safety_controller k_velocity="10"/>
   </joint>
-  <!--gazebo reference="elevator_button2">
-    <selfCollide>true</selfCollide>
-        <sensor name='elevator_button2_contact_sensor' type='contact'>
-      <always_on>true</always_on>
+  <gazebo reference="elevator_button2">
+    <gravity>true</gravity>
+    <self_collide>false</self_collide>
+    <material>Gazebo/Red</material>
+    <sensor name='elevator_button2_contact_sensor' type='contact'>
+      <always_on>1</always_on>
       <update_rate>10</update_rate>
       <contact>
-        <collision>elevator_button2_geom</collision>
+        <collision>elevator_button2_collision</collision>
+        <topic>elevator_button2_bumper</topic>
       </contact>
       <plugin name="elevator_button2_gazebo_ros_bumper_controller" filename="libgazebo_ros_bumper.so">
-        <alwaysOn>true</alwaysOn>
-        <updateRate>10</updateRate>
         <frameName>elevator_button2</frameName>
         <bumperTopicName>elevator_button2_bumper</bumperTopicName>
       </plugin>
     </sensor>
-    <material>Gazebo/Red</material>
-    <turnGravityOff>false</turnGravityOff>
-  </gazebo-->
+  </gazebo>
   <link name="wall_ext18">
     <inertial>

Commit message: fix ipa-apartment elevetor controllers

File: cob_gazebo_worlds/urdf/ipa-apartment/elevator.urdf.xacro (robot description, xacro)
@@ -37,13 +37,10 @@
     <child link="elevator_left" />
     <axis xyz = "0 1 0"/>
-    <calibration rising="0.0"/>
-    <dynamics damping="0.0" friction="0.0"/>
     <limit effort="100" velocity="1.0" lower="0" upper="0.87" />
-    <!--safety_controller k_velocity="10"/-->
   </joint>
   <transmission name="elevator_left_trans">
     <type>transmission_interface/SimpleTransmission</type>
     <joint name="elevator_left_joint">
-      <hardwareInterface>EffortJointInterface</hardwareInterface>
+      <hardwareInterface>PositionJointInterface</hardwareInterface>
     </joint>
     <actuator name="elevator_left_motor">
@@ -155,17 +152,14 @@
   </gazebo>
   <joint name="elevator_right_joint" type="prismatic">
+    <origin xyz="0 -1.085 0" rpy="0 0 0" />
+    <parent link="origin_elevator" />
+    <child link="elevator_right" />
     <axis xyz = "0 -1 0"/>
-    <origin xyz="0 -1.085 0" rpy="0 0 0" />
-    <parent link="origin_elevator" />
-    <child link="elevator_right" />
-    <calibration rising="0.0"/>
-    <dynamics damping="0.0" friction="0.0"/>
     <limit effort="100" velocity="1.0" lower="0" upper="0.87" />
-    <safety_controller k_velocity="10"/>
   </joint>
   <transmission name="elevator_right_trans">
     <type>transmission_interface/SimpleTransmission</type>
     <joint name="elevator_right_joint">
-      <hardwareInterface>EffortJointInterface</hardwareInterface>
+      <hardwareInterface>PositionJointInterface</hardwareInterface>
     </joint>
     <actuator name="elevator_right_motor">
@@ -277,9 +271,16 @@
     <parent link="origin_elevator" />
     <child link="elevator_button1" />
-    <calibration rising="0.0"/>
-    <dynamics damping="0.0" friction="0.0"/>
-    <limit effort="100" velocity="1.0" lower="0" upper="0" />
-    <safety_controller k_velocity="10"/>
-  </joint>
+    <axis xyz = "0 0 1"/>
+    <limit effort="100" velocity="1.0" lower="0" upper="0.1" />
+  </joint>
+  <transmission name="joint_elevator_button1_trans">
+    <type>transmission_interface/SimpleTransmission</type>
+    <joint name="joint_elevator_button1">
+      <hardwareInterface>PositionJointInterface</hardwareInterface>
+    </joint>
+    <actuator name="joint_elevator_button1_motor">
+      <mechanicalReduction>1</mechanicalReduction>
+    </actuator>
+  </transmission>
   <gazebo reference="elevator_button1">
     <gravity>true</gravity>
@@ -321,9 +322,16 @@
     <parent link="origin_elevator" />
     <child link="elevator_button2" />
-    <calibration rising="0.0"/>
-    <dynamics damping="0.0" friction="0.0"/>
-    <limit effort="100" velocity="1.0" lower="0" upper="0" />
-    <safety_controller k_velocity="10"/>
-  </joint>
+    <axis xyz = "0 0 1"/>
+    <limit effort="100" velocity="1.0" lower="0" upper="0.1" />
+  </joint>
+  <transmission name="joint_elevator_button2_trans">
+    <type>transmission_interface/SimpleTransmission</type>
+    <joint name="joint_elevator_button2">
+      <hardwareInterface>PositionJointInterface</hardwareInterface>
+    </joint>
+    <actuator name="joint_elevator_button2_motor">
+      <mechanicalReduction>1</mechanicalReduction>
+    </actuator>
+  </transmission>
   <gazebo reference="elevator_button2">
     <gravity>true</gravity>

Commit message: fix ipa-apartment elevator

File: cob_gazebo_worlds/urdf/ipa-apartment/elevator.urdf.xacro (robot description, xacro)
@@ -250,5 +250,5 @@
   <!--elevator buttons-->
   <link name="elevator_button1">
-    <xacro:box_inertial x="0.01" y="0.05" z="0.05" mass="1.0">
+    <xacro:box_inertial x="0.0" y="0.0" z="0.0" mass="0.001">
       <origin xyz="0 0 0" rpy="0 0 0" />
     </xacro:box_inertial>
@@ -267,17 +267,17 @@
     </collision>
   </link>
-  <joint name="joint_elevator_button1" type="prismatic">
+  <joint name="elevator_button1_joint" type="prismatic">
     <origin xyz="-0.04 0 ${-size_z_wall1/2+1.035}" rpy="0 0 0" />
     <parent link="origin_elevator" />
     <child link="elevator_button1" />
-    <axis xyz = "0 0 1"/>
-    <limit effort="100" velocity="1.0" lower="0" upper="0.1" />
-  </joint>
-  <transmission name="joint_elevator_button1_trans">
+    <axis xyz = "-1 0 0"/>
+    <limit effort="100" velocity="1.0" lower="0" upper="0.005" />
+  </joint>
+  <transmission name="elevator_button1_joint_trans">
     <type>transmission_interface/SimpleTransmission</type>
-    <joint name="joint_elevator_button1">
+    <joint name="elevator_button1_joint">
       <hardwareInterface>PositionJointInterface</hardwareInterface>
     </joint>
-    <actuator name="joint_elevator_button1_motor">
+    <actuator name="elevator_button1_joint_motor">
       <mechanicalReduction>1</mechanicalReduction>
     </actuator>
@@ -301,5 +301,5 @@
   </gazebo>
   <link name="elevator_button2">
-    <xacro:box_inertial x="0.01" y="0.05" z="0.05" mass="1.0">
+    <xacro:box_inertial x="0.0" y="0.0" z="0.0" mass="0.001">
       <origin xyz="0 0 0" rpy="0 0 0" />
     </xacro:box_inertial>
@@ -318,17 +318,17 @@
     </collision>
   </link>
-  <joint name="joint_elevator_button2" type="prismatic">
+  <joint name="elevator_button2_joint" type="prismatic">
     <origin xyz="-0.04 0 ${-size_z_wall1/2+1.095}" rpy="0 0 0" />
     <parent link="origin_elevator" />
     <child link="elevator_button2" />
-    <axis xyz = "0 0 1"/>
-    <limit effort="100" velocity="1.0" lower="0" upper="0.1" />
-  </joint>
-  <transmission name="joint_elevator_button2_trans">
+    <axis xyz = "-1 0 0"/>
+    <limit effort="100" velocity="1.0" lower="0" upper="0.005" />
+  </joint>
+  <transmission name="elevator_button2_joint_trans">
     <type>transmission_interface/SimpleTransmission</type>
-    <joint name="joint_elevator_button2">
+    <joint name="elevator_button2_joint">
       <hardwareInterface>PositionJointInterface</hardwareInterface>
     </joint>
-    <actuator name="joint_elevator_button2_motor">
+    <actuator name="elevator_button2_joint_motor">
       <mechanicalReduction>1</mechanicalReduction>
     </actuator>

Commit message: use default inertias

File: cob_gazebo_worlds/urdf/ipa-apartment/elevator.urdf.xacro (robot description, xacro)
@@ -33,5 +33,5 @@
   </gazebo>
   <joint name="elevator_left_joint" type="prismatic">
-    <origin xyz="0 1.085 0" rpy="0 0 0" />
+    <origin xyz="-0.04 1.085 0" rpy="0 0 0" />
     <parent link="origin_elevator" />
     <child link="elevator_left" />
@@ -152,5 +152,5 @@
   </gazebo>
   <joint name="elevator_right_joint" type="prismatic">
-    <origin xyz="0 -1.085 0" rpy="0 0 0" />
+    <origin xyz="-0.04 -1.085 0" rpy="0 0 0" />
     <parent link="origin_elevator" />
     <child link="elevator_right" />
@@ -250,7 +250,5 @@
   <!--elevator buttons-->
   <link name="elevator_button1">
-    <xacro:box_inertial x="0.0" y="0.0" z="0.0" mass="0.001">
-      <origin xyz="0 0 0" rpy="0 0 0" />
-    </xacro:box_inertial>
+    <xacro:default_inertial/>
     <visual>
       <origin xyz="0 0 0" />
@@ -272,5 +270,5 @@
     <child link="elevator_button1" />
     <axis xyz = "-1 0 0"/>
-    <limit effort="100" velocity="1.0" lower="0" upper="0.005" />
+    <limit effort="1" velocity="1.0" lower="0" upper="0.005" />
   </joint>
   <transmission name="elevator_button1_joint_trans">
@@ -301,7 +299,5 @@
   </gazebo>
   <link name="elevator_button2">
-    <xacro:box_inertial x="0.0" y="0.0" z="0.0" mass="0.001">
-      <origin xyz="0 0 0" rpy="0 0 0" />
-    </xacro:box_inertial>
+    <xacro:default_inertial/>
     <visual>
       <origin xyz="0 0 0" />
@@ -323,5 +319,5 @@
     <child link="elevator_button2" />
     <axis xyz = "-1 0 0"/>
-    <limit effort="100" velocity="1.0" lower="0" upper="0.005" />
+    <limit effort="1" velocity="1.0" lower="0" upper="0.005" />
   </joint>
   <transmission name="elevator_button2_joint_trans">
