Commit message: Renamed the materials

File: cob_gazebo_worlds/urdf/materials.urdf.xacro (robot description, xacro)
@@ -19,24 +19,12 @@
 		<color rgba="1.0 1.0 1.0 1.0"/>
 	</material>
-	<material name="Black">
+	<material name="IPA/Black">
 		<color rgba="0.0 0.0 0.0 1.0"/>
 	</material>
-        <material name="Transparent">
-                <color rgba="0.81 0.81 0.81 0.0"/>
-        </material>
-        <material name="LightBlue">
-                <color rgba="0.624 0.698 0.858 1"/>
-        </material>
-	<material name="Caster">
-		<texture filename="package://pr2_ogre/Media/materials/textures/pr2_caster_texture.png" />
-	</material>
-	<material name="Wheel_l">
-		<texture filename="package://pr2_ogre/Media/materials/textures/pr2_wheel_left.png" />
-	</material>
-	<material name="Wheel_r">
-		<texture filename="package://pr2_ogre/Media/materials/textures/pr2_wheel_right.png" />
-	</material>
-	<material name="RollLinks">
-		<texture filename="package://pr2_ogre/Media/materials/textures/pr2_wheel_left.png" />
-	</material>
+    <material name="Transparent">
+        <color rgba="0.81 0.81 0.81 0.0"/>
+    </material>
+    <material name="LightBlue">
+           <color rgba="0.624 0.698 0.858 1"/>
+    </material>
 </robot>

Commit message: Renamed colors

File: cob_gazebo_worlds/urdf/materials.urdf.xacro (robot description, xacro)
@@ -1,20 +1,20 @@
 <?xml version="1.0"?>
 <robot>
-	<material name="Blue">
+	<material name="IPA/Blue">
 		<color rgba="0.0 0.0 0.8 1.0"/>
 	</material>
-	<material name="Green">
+	<material name="IPA/Green">
 		<color rgba="0.0 0.8 0.0 1.0"/>
 	</material>
-	<material name="Grey">
+	<material name="IPA/Grey">
 		<color rgba="0.7 0.7 0.7 1.0"/>
 	</material>
-	<material name="Grey2">
+	<material name="IPA/Grey2">
 		<color rgba="0.81 0.81 0.81 1.0"/>
 	</material>
-	<material name="Red">
+	<material name="IPA/Red">
 		<color rgba="0.8 0.0 0.0 1.0"/>
 	</material>
-	<material name="White">
+	<material name="IPA/White">
 		<color rgba="1.0 1.0 1.0 1.0"/>
 	</material>
@@ -22,8 +22,8 @@
 		<color rgba="0.0 0.0 0.0 1.0"/>
 	</material>
-    <material name="Transparent">
+    <material name="IPA/Transparent">
         <color rgba="0.81 0.81 0.81 0.0"/>
     </material>
-    <material name="LightBlue">
+    <material name="IPA/LightBlue">
            <color rgba="0.624 0.698 0.858 1"/>
     </material>
