Commit message: fix environment to gazebo world frame + proper interia

File: cob_gazebo_worlds/urdf/ipa-kitchen/ipa-kitchen.urdf.xacro (robot description, xacro)
@@ -2,33 +2,15 @@
 <robot xmlns:xacro="http://www.ros.org/wiki/xacro"
        name="ipa-kitchen">
-<xacro:macro name="ipa-kitchen" params="name">
-<!-- dummy_link -->
-  <link name="dummy_link">
-    <inertial>
-      <origin xyz="0 0 0" />
-      <mass value="5.0" />
-      <inertia ixx="0.0" ixy="0.0" ixz="0.0" iyy="0.0" iyz="0.0" izz="0.0" />
-    </inertial>
-    <visual>
-      <origin xyz="0 0 0" />
-      <geometry>
-        <box size="0.00 0.00 0.00" />
-      </geometry>
-    </visual>
-    <collision>
-      <origin xyz="0 0 0" />
-      <geometry>
-        <box size="0.00 0.00 0.00" />
-      </geometry>
-    </collision>
-  </link>
-<!-- walls -->
+  <xacro:include filename="$(find cob_gazebo_worlds)/urdf/common.xacro" />
+  <xacro:include filename="$(find cob_gazebo_worlds)/urdf/materials.urdf.xacro" />
+  <xacro:macro name="ipa-kitchen" params="name">
+  <!-- world -->
+  <link name="world"/>
+  <!-- walls -->
   <!-- wall_00 -->
   <link name="wall_00">
-    <inertial>
-      <origin xyz="0 0 0" />
-      <mass value="5.0" />
-      <inertia ixx="0.0" ixy="0.0" ixz="0.0" iyy="0.0" iyz="0.0" izz="0.0" />
-    </inertial>
+    <xacro:box_inertial x="2.75" y="0.06" z="0.50" mass="5.0">
+      <origin xyz="0 0 0" rpy="0 0 0" />
+    </xacro:box_inertial>
     <visual>
       <origin xyz="0 0 0" />
@@ -49,14 +31,12 @@
   <joint name="joint_wall_00" type="fixed">
     <origin xyz="-2.156 4.791 0.250" rpy="0 0 0" />
-    <parent link="dummy_link" />
+    <parent link="world" />
     <child link="wall_00" />
   </joint>
   <!-- wall_01 -->
   <link name="wall_01">
-    <inertial>
-      <origin xyz="0 0 0" />
-      <mass value="5.0" />
-      <inertia ixx="0.0" ixy="0.0" ixz="0.0" iyy="0.0" iyz="0.0" izz="0.0" />
-    </inertial>
+    <xacro:box_inertial x="0.10" y="0.80" z="2.40" mass="5.0">
+      <origin xyz="0 0 0" rpy="0 0 0" />
+    </xacro:box_inertial>
     <visual>
       <origin xyz="0 0 0" />
@@ -77,14 +57,12 @@
   <joint name="joint_wall_01" type="fixed">
     <origin xyz="-0.731 4.421 1.200" rpy="0 0 0" />
-    <parent link="dummy_link" />
+    <parent link="world" />
     <child link="wall_01" />
   </joint>
   <!-- wall_02 -->
   <link name="wall_02">
-    <inertial>
-      <origin xyz="0 0 0" />
-      <mass value="5.0" />
-      <inertia ixx="0.0" ixy="0.0" ixz="0.0" iyy="0.0" iyz="0.0" izz="0.0" />
-    </inertial>
+    <xacro:box_inertial x="3.29" y="0.06" z="0.50" mass="5.0">
+      <origin xyz="0 0 0" rpy="0 0 0" />
+    </xacro:box_inertial>
     <visual>
       <origin xyz="0 0 0" />
@@ -105,14 +83,12 @@
   <joint name="joint_wall_02" type="fixed">
     <origin xyz="0.964 4.791 0.250" rpy="0 0 0" />
-    <parent link="dummy_link" />
+    <parent link="world" />
     <child link="wall_02" />
   </joint>
   <!-- wall_03 -->
   <link name="wall_03">
-    <inertial>
-      <origin xyz="0 0 0" />
-      <mass value="5.0" />
-      <inertia ixx="0.0" ixy="0.0" ixz="0.0" iyy="0.0" iyz="0.0" izz="0.0" />
-    </inertial>
+    <xacro:box_inertial x="0.80" y="0.10" z="3.20" mass="5.0">
+      <origin xyz="0 0 0" rpy="0 0 0" />
+    </xacro:box_inertial>
     <visual>
       <origin xyz="0 0 0" />
@@ -133,14 +109,12 @@
   <joint name="joint_wall_03" type="fixed">
     <origin xyz="3.009 4.771 1.600" rpy="0 0 0" />
-    <parent link="dummy_link" />
+    <parent link="world" />
     <child link="wall_03" />
   </joint>
   <!-- wall_04 -->
   <link name="wall_04">
-    <inertial>
-      <origin xyz="0 0 0" />
-      <mass value="5.0" />
-      <inertia ixx="0.0" ixy="0.0" ixz="0.0" iyy="0.0" iyz="0.0" izz="0.0" />
-    </inertial>
+    <xacro:box_inertial x="0.06" y="6.90" z="0.50" mass="5.0">
+      <origin xyz="0 0 0" rpy="0 0 0" />
+    </xacro:box_inertial>
     <visual>
       <origin xyz="0 0 0" />
@@ -161,14 +135,12 @@
   <joint name="joint_wall_04" type="fixed">
     <origin xyz="3.379 1.271 0.250" rpy="0 0 0" />
-    <parent link="dummy_link" />
+    <parent link="world" />
     <child link="wall_04" />
   </joint>
   <!-- wall_06 -->
   <link name="wall_06">
-    <inertial>
-      <origin xyz="0 0 0" />
-      <mass value="5.0" />
-      <inertia ixx="0.0" ixy="0.0" ixz="0.0" iyy="0.0" iyz="0.0" izz="0.0" />
-    </inertial>
+    <xacro:box_inertial x="6.88" y="0.06" z="0.50" mass="5.0">
+      <origin xyz="0 0 0" rpy="0 0 0" />
+    </xacro:box_inertial>
     <visual>
       <origin xyz="0 0 0" />
@@ -189,14 +161,12 @@
   <joint name="joint_wall_06" type="fixed">
     <origin xyz="-0.091 -2.149 0.250" rpy="0 0 0" />
-    <parent link="dummy_link" />
+    <parent link="world" />
     <child link="wall_06" />
   </joint>
   <!-- wall_07 -->
   <link name="wall_07">
-    <inertial>
-      <origin xyz="0 0 0" />
-      <mass value="5.0" />
-      <inertia ixx="0.0" ixy="0.0" ixz="0.0" iyy="0.0" iyz="0.0" izz="0.0" />
-    </inertial>
+    <xacro:box_inertial x="0.06" y="7.00" z="2.60" mass="5.0">
+      <origin xyz="0 0 0" rpy="0 0 0" />
+    </xacro:box_inertial>
     <visual>
       <origin xyz="0 0 0" />
@@ -217,14 +187,12 @@
   <joint name="joint_wall_07" type="fixed">
     <origin xyz="-3.561 1.321 1.300" rpy="0 0 0" />
-    <parent link="dummy_link" />
+    <parent link="world" />
     <child link="wall_07" />
   </joint>
   <!-- wall_08 -->
   <link name="wall_08">
-    <inertial>
-      <origin xyz="0 0 0" />
-      <mass value="5.0" />
-      <inertia ixx="0.0" ixy="0.0" ixz="0.0" iyy="0.0" iyz="0.0" izz="0.0" />
-    </inertial>
+    <xacro:box_inertial x="1.69" y="0.06" z="2.06" mass="5.0">
+      <origin xyz="0 0 0" rpy="0 0 0" />
+    </xacro:box_inertial>
     <visual>
       <origin xyz="0 0 0" />
@@ -245,14 +213,12 @@
   <joint name="joint_wall_08" type="fixed">
     <origin xyz="-2.686 3.641 1.030" rpy="0 0 0" />
-    <parent link="dummy_link" />
+    <parent link="world" />
     <child link="wall_08" />
   </joint>
   <!-- wall_09 -->
   <link name="wall_09">
-    <inertial>
-      <origin xyz="0 0 0" />
-      <mass value="5.0" />
-      <inertia ixx="0.0" ixy="0.0" ixz="0.0" iyy="0.0" iyz="0.0" izz="0.0" />
-    </inertial>
+    <xacro:box_inertial x="0.06" y="1.30" z="2.06" mass="5.0">
+      <origin xyz="0 0 0" rpy="0 0 0" />
+    </xacro:box_inertial>
     <visual>
       <origin xyz="0 0 0" />
@@ -273,14 +239,12 @@
   <joint name="joint_wall_09" type="fixed">
     <origin xyz="-1.811 3.021 1.030" rpy="0 0 0" />
-    <parent link="dummy_link" />
+    <parent link="world" />
     <child link="wall_09" />
   </joint>
   <!-- wall_10 -->
   <link name="wall_10">
-    <inertial>
-      <origin xyz="0 0 0" />
-      <mass value="5.0" />
-      <inertia ixx="0.0" ixy="0.0" ixz="0.0" iyy="0.0" iyz="0.0" izz="0.0" />
-    </inertial>
+    <xacro:box_inertial x="1.75" y="0.10" z="3.20" mass="5.0">
+      <origin xyz="0 0 0" rpy="0 0 0" />
+    </xacro:box_inertial>
     <visual>
       <origin xyz="0 0 0" />
@@ -301,14 +265,12 @@
   <joint name="joint_wall_10" type="fixed">
     <origin xyz="-2.656 2.321 1.600" rpy="0 0 0" />
-    <parent link="dummy_link" />
+    <parent link="world" />
     <child link="wall_10" />
   </joint>
   <!-- wall_11 -->
   <link name="wall_11">
-    <inertial>
-      <origin xyz="0 0 0" />
-      <mass value="5.0" />
-      <inertia ixx="0.0" ixy="0.0" ixz="0.0" iyy="0.0" iyz="0.0" izz="0.0" />
-    </inertial>
+    <xacro:box_inertial x="0.75" y="0.06" z="2.60" mass="5.0">
+      <origin xyz="0 0 0" rpy="0 0 0" />
+    </xacro:box_inertial>
     <visual>
       <origin xyz="0 0 0" />
@@ -329,14 +291,12 @@
   <joint name="joint_wall_11" type="fixed">
     <origin xyz="-1.406 2.301 1.300" rpy="0 0 0" />
-    <parent link="dummy_link" />
+    <parent link="world" />
     <child link="wall_11" />
   </joint>
 <!--
   <link name="door">
-    <inertial>
-      <origin xyz="0 0 0" />
-      <mass value="10.0" />
-      <inertia ixx="0.0" ixy="0.0" ixz="0.0" iyy="0.0" iyz="0.0" izz="10.0" />
-    </inertial>
+    <xacro:box_inertial x="0.85" y="0.06" z="2.05" mass="5.0">
+      <origin xyz="0.425 0 0" rpy="0 0 0" />
+    </xacro:box_inertial>
     <visual>
       <origin xyz="0.425 0 0" />
@@ -367,9 +327,7 @@
   <!-- wall_12 -->
   <link name="wall_12">
-    <inertial>
-      <origin xyz="0 0 0" />
-      <mass value="5.0" />
-      <inertia ixx="0.0" ixy="0.0" ixz="0.0" iyy="0.0" iyz="0.0" izz="0.0" />
-    </inertial>
+    <xacro:box_inertial x="0.85" y="0.06" z="0.55" mass="5.0">
+      <origin xyz="0 0 0" rpy="0 0 0" />
+    </xacro:box_inertial>
     <visual>
       <origin xyz="0 0 0" />
@@ -390,14 +348,12 @@
   <joint name="joint_wall_12" type="fixed">
     <origin xyz="-0.606 2.301 2.325" rpy="0 0 0" />
-    <parent link="dummy_link" />
+    <parent link="world" />
     <child link="wall_12" />
   </joint>
   <!-- wall_13 -->
   <link name="wall_13">
-    <inertial>
-      <origin xyz="0 0 0" />
-      <mass value="5.0" />
-      <inertia ixx="0.0" ixy="0.0" ixz="0.0" iyy="0.0" iyz="0.0" izz="0.0" />
-    </inertial>
+    <xacro:box_inertial x="0.15" y="0.06" z="2.60" mass="5.0">
+      <origin xyz="0 0 0" rpy="0 0 0" />
+    </xacro:box_inertial>
     <visual>
       <origin xyz="0 0 0" />
@@ -418,14 +374,12 @@
   <joint name="joint_wall_13" type="fixed">
     <origin xyz="-0.106 2.301 1.300" rpy="0 0 0" />
-    <parent link="dummy_link" />
+    <parent link="world" />
     <child link="wall_13" />
   </joint>
   <!-- wall_14 -->
   <link name="wall_14">
-    <inertial>
-      <origin xyz="0 0 0" />
-      <mass value="5.0" />
-      <inertia ixx="0.0" ixy="0.0" ixz="0.0" iyy="0.0" iyz="0.0" izz="0.0" />
-    </inertial>
+    <xacro:box_inertial x="0.06" y="0.54" z="0.75" mass="5.0">
+      <origin xyz="0 0 0" rpy="0 0 0" />
+    </xacro:box_inertial>
     <visual>
       <origin xyz="0 0 0" />
@@ -446,14 +400,12 @@
   <joint name="joint_wall_14" type="fixed">
     <origin xyz="-0.061 2.001 0.375" rpy="0 0 0" />
-    <parent link="dummy_link" />
+    <parent link="world" />
     <child link="wall_14" />
   </joint>
   <!-- wall_15 -->
   <link name="wall_15">
-    <inertial>
-      <origin xyz="0 0 0" />
-      <mass value="5.0" />
-      <inertia ixx="0.0" ixy="0.0" ixz="0.0" iyy="0.0" iyz="0.0" izz="0.0" />
-    </inertial>
+    <xacro:box_inertial x="0.06" y="0.54" z="0.55" mass="5.0">
+      <origin xyz="0 0 0" rpy="0 0 0" />
+    </xacro:box_inertial>
     <visual>
       <origin xyz="0 0 0" />
@@ -474,14 +426,12 @@
   <joint name="joint_wall_15" type="fixed">
     <origin xyz="-0.061 2.001 2.325" rpy="0 0 0" />
-    <parent link="dummy_link" />
+    <parent link="world" />
     <child link="wall_15" />
   </joint>
   <!-- wall_16 -->
   <link name="wall_16">
-    <inertial>
-      <origin xyz="0 0 0" />
-      <mass value="5.0" />
-      <inertia ixx="0.0" ixy="0.0" ixz="0.0" iyy="0.0" iyz="0.0" izz="0.0" />
-    </inertial>
+    <xacro:box_inertial x="0.06" y="0.06" z="2.60" mass="5.0">
+      <origin xyz="0 0 0" rpy="0 0 0" />
+    </xacro:box_inertial>
     <visual>
       <origin xyz="0 0 0" />
@@ -502,14 +452,12 @@
   <joint name="joint_wall_16" type="fixed">
     <origin xyz="-0.061 1.701 1.300" rpy="0 0 0" />
-    <parent link="dummy_link" />
+    <parent link="world" />
     <child link="wall_16" />
   </joint>
   <!-- wall_17 -->
   <link name="wall_17">
-    <inertial>
-      <origin xyz="0 0 0" />
-      <mass value="5.0" />
-      <inertia ixx="0.0" ixy="0.0" ixz="0.0" iyy="0.0" iyz="0.0" izz="0.0" />
-    </inertial>
+    <xacro:box_inertial x="1.63" y="0.06" z="0.75" mass="5.0">
+      <origin xyz="0 0 0" rpy="0 0 0" />
+    </xacro:box_inertial>
     <visual>
       <origin xyz="0 0 0" />
@@ -530,14 +478,12 @@
   <joint name="joint_wall_17" type="fixed">
     <origin xyz="0.784 1.701 0.375" rpy="0 0 0" />
-    <parent link="dummy_link" />
+    <parent link="world" />
     <child link="wall_17" />
   </joint>
   <!-- wall_18 -->
   <link name="wall_18">
-    <inertial>
-      <origin xyz="0 0 0" />
-      <mass value="5.0" />
-      <inertia ixx="0.0" ixy="0.0" ixz="0.0" iyy="0.0" iyz="0.0" izz="0.0" />
-    </inertial>
+    <xacro:box_inertial x="1.63" y="0.06" z="0.55" mass="5.0">
+      <origin xyz="0 0 0" rpy="0 0 0" />
+    </xacro:box_inertial>
     <visual>
       <origin xyz="0 0 0" />
@@ -558,14 +504,12 @@
   <joint name="joint_wall_18" type="fixed">
     <origin xyz="0.784 1.701 2.325" rpy="0 0 0" />
-    <parent link="dummy_link" />
+    <parent link="world" />
     <child link="wall_18" />
   </joint>
   <!-- wall_19 -->
   <link name="wall_19">
-    <inertial>
-      <origin xyz="0 0 0" />
-      <mass value="5.0" />
-      <inertia ixx="0.0" ixy="0.0" ixz="0.0" iyy="0.0" iyz="0.0" izz="0.0" />
-    </inertial>
+    <xacro:box_inertial x="0.06" y="0.06" z="2.60" mass="5.0">
+      <origin xyz="0 0 0" rpy="0 0 0" />
+    </xacro:box_inertial>
     <visual>
       <origin xyz="0 0 0" />
@@ -586,14 +530,12 @@
   <joint name="joint_wall_19" type="fixed">
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
Commit message: ipa-kitchen includes a door that can passively be pushed open

File: cob_gazebo_worlds/urdf/ipa-kitchen/ipa-kitchen.urdf.xacro (robot description, xacro)
@@ -5,4 +5,10 @@
   <xacro:include filename="$(find cob_gazebo_worlds)/urdf/materials.urdf.xacro" />
   <xacro:macro name="ipa-kitchen" params="name">
+  <gazebo>
+    <plugin name="environment_gazebo_ros_control" filename="libgazebo_ros_control.so">
+      <robotNamespace>world</robotNamespace>
+      <robotParam>/world_description</robotParam>
+    </plugin>
+  </gazebo>
   <!-- world -->
   <link name="world"/>
@@ -294,5 +300,5 @@
     <child link="wall_11" />
   </joint>
-<!--
+  <!-- door -->
   <link name="door">
     <xacro:box_inertial x="0.85" y="0.06" z="2.05" mass="5.0">
@@ -317,12 +323,18 @@
   <joint name="door_joint" type="revolute" >
     <origin xyz="0.375 0.0 -0.275" rpy="0 0 0" />
-    <axis xyz="0 0 1" />
-    <limit lower="-1.8" upper="1.8" effort="1000" velocity="10" />
-    <safety_controller soft_lower_limit="-1.7" soft_upper_limit="1.7" k_position="100.0" k_velocity="10.0" />
-    <dynamics damping="60" friction="2000.0" />
     <parent link="wall_11" />
     <child link="door" />
-  </joint>
--->
+    <axis xyz="0 0 1" />
+    <limit effort="0.1" velocity="1" lower="-1.8" upper="1.8" />
+  </joint>
+  <transmission name="door_trans">
+    <type>transmission_interface/SimpleTransmission</type>
+    <joint name="door_joint">
+      <hardwareInterface>EffortJointInterface</hardwareInterface>
+    </joint>
+    <actuator name="door_motor">
+      <mechanicalReduction>1</mechanicalReduction>
+    </actuator>
+  </transmission>
   <!-- wall_12 -->
   <link name="wall_12">

Commit message: velocity controller for door

File: cob_gazebo_worlds/urdf/ipa-kitchen/ipa-kitchen.urdf.xacro (robot description, xacro)
@@ -302,7 +302,5 @@
   <!-- door -->
   <link name="door">
-    <xacro:box_inertial x="0.85" y="0.06" z="2.05" mass="5.0">
-      <origin xyz="0.425 0 0" rpy="0 0 0" />
-    </xacro:box_inertial>
+    <xacro:default_inertial/>
     <visual>
       <origin xyz="0.425 0 0" />
@@ -331,5 +329,5 @@
     <type>transmission_interface/SimpleTransmission</type>
     <joint name="door_joint">
-      <hardwareInterface>EffortJointInterface</hardwareInterface>
+      <hardwareInterface>VelocityJointInterface</hardwareInterface>
     </joint>
     <actuator name="door_motor">
