Commit message: successful integration of bmw-assembly into cob_simulation

File: cob_gazebo_worlds/urdf/bmw-assembly/bmw-assembly.urdf.xacro (robot description, xacro)
@@ -1,20 +1,20 @@
 <?xml version="1.0" ?>
 <robot xmlns:xacro="http://www.ros.org/wiki/xacro"
-	name="bmw_assembly">
+	name="bmw-assembly">
   <!-- properties -->
   <xacro:property name="base_width" value="0.1" />
   <xacro:property name="base_length" value="250" />
   <xacro:property name="base_height" value="0.1" />
+  <xacro:property name="base_mass" value="5.0" />
   <xacro:property name="belt_width" value="4" />
   <xacro:property name="belt_length" value="250" />
   <xacro:property name="belt_height" value="0.1" />
-  <xacro:property name="base_mass" value="5.0" />
   <xacro:property name="belt_mass" value="5.0" />
-  <xacro:property name="box_width" value="1.5" />
-  <xacro:property name="box_length" value="3" />
-  <xacro:property name="box_height" value="1" />
+  <xacro:property name="box_width" value="2.0" />
+  <xacro:property name="box_length" value="3.8" />
+  <xacro:property name="box_height" value="0.4" />
   <xacro:property name="box_mass" value="0.1" />
-  <xacro:property name="world_to_base_joint_offset_x" value="5" />
   <xacro:property name="boxes_distance" value="10"/>
+  <xacro:property name="world_to_base_offset_x" value="5" />
   <!-- macros -->
   <xacro:macro name="box_inertial" params="x y z mass *origin">
@@ -42,7 +42,4 @@
       </collision>
       <xacro:default_inertial/>
-      <!--xacro:box_inertial x="${box_width}" y="${box_length}" z="${box_height}" mass="${box_mass}">
-        <origin xyz="0 0 0" rpy="0 0 0"/>
-      </xacro:box_inertial-->
     </link>
     <gazebo reference="box_${new_box_num}">
@@ -65,5 +62,6 @@
   <gazebo>
     <plugin name="gazebo_ros_control" filename="libgazebo_ros_control.so">
-      <robotNamespace>bmw_assembly</robotNamespace>
+      <robotNamespace>world</robotNamespace>
+      <robotParam>/world_description</robotParam>
     </plugin>
   </gazebo>
@@ -84,5 +82,4 @@
       </geometry>
     </collision>
-    <!--xacro:default_inertial/-->
     <xacro:box_inertial x="${base_width}" y="${base_length}" z="${base_height}" mass="${base_mass}">
 	<origin xyz="0 0 0" rpy="0 0 0"/>
@@ -92,5 +89,5 @@
 	<material>Gazebo/Black</material>
   </gazebo>
-  <!-- assembly belt -->
+  <!-- moving belt -->
   <link name="my_belt">
     <visual>
@@ -106,5 +103,4 @@
       </geometry>
     </collision>
-    <!--xacro:default_inertial/-->
     <xacro:box_inertial x="${belt_width}" y="${belt_length}" z="${belt_height}" mass="${belt_mass}">
 	<origin xyz="0 0 0" rpy="0 0 0"/>
@@ -132,8 +128,25 @@
   <xacro:new_box new_box_num="16"/>
   <xacro:new_box new_box_num="17"/>
+  <!--world objects-->
+  <model name="net_bin_1" static="true">
+    <link name="net_bin_1_link">
+      <origin pose="0 0 0 0 0 0"/>
+      <collision name="net_bin_1_collision">
+        <geometry>
+          <mesh filename="package://cob_gazebo_worlds/Media/models/dump-bin-retail/model.dae" scale="1 1 1"/>
+        </geometry>
+      </collision>
+      <visual name="net_bin_1_visual" cast_shadows="false">
+        <geometry>
+          <mesh filename="package://cob_gazebo_worlds/Media/models/dump-bin-retail/model.dae" scale="1 1 1"/>
+        </geometry>
+      </visual>
+    </link>
+  </model>
+  <!--joints-->
   <joint name="world_joint" type="fixed">
      <parent link="world"/>
      <child link="belt_base_link"/>
-     <origin xyz = "${world_to_base_joint_offset_x} 0 ${base_height/2}"/>
+     <origin xyz = "${world_to_base_offset_x} 0 ${base_height/2}"/>
   </joint>
   <joint name="base_to_belt" type="prismatic">
@@ -142,12 +155,13 @@
     <axis xyz="0 1 0"/>
     <dynamics damping="0.7"/>
-    <origin xyz="${belt_width+0.5} 0 ${base_height/2}"/>
+    <origin xyz="${belt_width/2+0.5} 0 ${base_height/2}"/>
     <limit lower="-100000" upper="100000" velocity="0.5" effort="10"/>
   </joint>
   <transmission name="belt_trans">
     <type>transmission_interface/SimpleTransmission</type>
-    <joint name="base_to_belt"/>
+    <joint name="base_to_belt" />
     <actuator name="belt_motor">
       <hardwareInterface>VelocityJointInterface</hardwareInterface>
+    <!--  <hardwareInterface>EffortJointInterface</hardwareInterface> -->
       <mechanicalReduction>1</mechanicalReduction>
     </actuator>

Commit message: added objects to the environment

File: cob_gazebo_worlds/urdf/bmw-assembly/bmw-assembly.urdf.xacro (robot description, xacro)
@@ -52,4 +52,29 @@
     </joint>
   </xacro:macro>
+  <xacro:macro name="new_object" params="new_object_num *mesh *origin">
+    <link name="world_object_${new_object_num}">
+      <visual>
+        <origin xyz="0 0 0" rpy="0 0 0"/>
+        <geometry>
+          <insert_block name = "mesh"/>
+        </geometry>
+      </visual>
+      <collision>
+        <origin xyz="0 0 0" rpy="0 0 0"/>
+        <geometry>
+          <insert_block name = "mesh"/>
+        </geometry>
+      </collision>
+      <xacro:default_inertial/>
+    </link>
+    <gazebo reference="world_object_${new_object_num}">
+      <static>true</static>
+    </gazebo>
+    <joint name="bin_joint_${new_object_num}" type="fixed">
+       <insert_block name="origin"/>
+       <parent link="belt_base_link"/>
+       <child link="world_object_${new_object_num}"/>
+    </joint>
+  </xacro:macro>
   <xacro:macro name="default_inertial">
     <inertial>
@@ -89,4 +114,9 @@
 	<material>Gazebo/Black</material>
   </gazebo>
+  <joint name="world_joint" type="fixed">
+     <parent link="world"/>
+     <child link="belt_base_link"/>
+     <origin xyz = "${world_to_base_offset_x} 0 ${base_height/2}"/>
+  </joint>
   <!-- moving belt -->
   <link name="my_belt">
@@ -110,4 +140,12 @@
     <material>Gazebo/WoodFloor</material>
   </gazebo>
+  <joint name="base_to_belt" type="prismatic">
+    <parent link="belt_base_link"/>
+    <child link="my_belt"/>
+    <axis xyz="0 1 0"/>
+    <dynamics damping="0.7"/>
+    <origin xyz="${belt_width/2+0.5} 0 ${base_height/2}"/>
+    <limit lower="-100000" upper="100000" velocity="0.5" effort="10"/>
+  </joint>
   <!--boxes-->
   <xacro:new_box new_box_num="1"/>
@@ -129,33 +167,48 @@
   <xacro:new_box new_box_num="17"/>
   <!--world objects-->
-  <model name="net_bin_1" static="true">
-    <link name="net_bin_1_link">
-      <origin pose="0 0 0 0 0 0"/>
-      <collision name="net_bin_1_collision">
-        <geometry>
-          <mesh filename="package://cob_gazebo_worlds/Media/models/dump-bin-retail/model.dae" scale="1 1 1"/>
-        </geometry>
-      </collision>
-      <visual name="net_bin_1_visual" cast_shadows="false">
-        <geometry>
-          <mesh filename="package://cob_gazebo_worlds/Media/models/dump-bin-retail/model.dae" scale="1 1 1"/>
-        </geometry>
-      </visual>
-    </link>
-  </model>
-  <!--joints-->
-  <joint name="world_joint" type="fixed">
-     <parent link="world"/>
-     <child link="belt_base_link"/>
-     <origin xyz = "${world_to_base_offset_x} 0 ${base_height/2}"/>
-  </joint>
-  <joint name="base_to_belt" type="prismatic">
-    <parent link="belt_base_link"/>
-    <child link="my_belt"/>
-    <axis xyz="0 1 0"/>
-    <dynamics damping="0.7"/>
-    <origin xyz="${belt_width/2+0.5} 0 ${base_height/2}"/>
-    <limit lower="-100000" upper="100000" velocity="0.5" effort="10"/>
-  </joint>
+  <xacro:new_object new_object_num="1" >
+    <mesh filename="package://cob_gazebo_worlds/Media/models/dump-bin-retail/model.dae"/>
+    <origin xyz="-7 -15 0" />
+  </xacro:new_object>
+  <xacro:new_object new_object_num="2" >
+    <mesh filename="package://cob_gazebo_worlds/Media/models/dump-bin-retail/model.dae"/>
+    <origin xyz="-7 -10 0" />
+  </xacro:new_object>
+  <xacro:new_object new_object_num="3" >
+    <mesh filename="package://cob_gazebo_worlds/Media/models/dump-bin-retail/model.dae"/>
+    <origin xyz="-7 -5 0" />
+  </xacro:new_object>
+  <xacro:new_object new_object_num="4" >
+    <mesh filename="package://cob_gazebo_worlds/Media/models/dump-bin-retail/model.dae"/>
+    <origin xyz="-7 0 0" />
+  </xacro:new_object>
+  <xacro:new_object new_object_num="5" >
+    <mesh filename="package://cob_gazebo_worlds/Media/models/dump-bin-retail/model.dae"/>
+    <origin xyz="-7 5 0" />
+  </xacro:new_object>
+  <xacro:new_object new_object_num="6" >
+    <mesh filename="package://cob_gazebo_worlds/Media/models/dump-bin-retail/model.dae"/>
+    <origin xyz="5 -15 0" />
+  </xacro:new_object>
+  <xacro:new_object new_object_num="7" >
+    <mesh filename="package://cob_gazebo_worlds/Media/models/dump-bin-retail/model.dae"/>
+    <origin xyz="5 -10 0" />
+  </xacro:new_object>
+  <xacro:new_object new_object_num="8" >
+    <mesh filename="package://cob_gazebo_worlds/Media/models/dump-bin-retail/model.dae"/>
+    <origin xyz="5 -5 0" />
+  </xacro:new_object>
+  <xacro:new_object new_object_num="9" >
+    <mesh filename="package://cob_gazebo_worlds/Media/models/dump-bin-retail/model.dae"/>
+    <origin xyz="5 0 0" />
+  </xacro:new_object>
+  <xacro:new_object new_object_num="10" >
+    <mesh filename="package://cob_gazebo_worlds/Media/models/dump-bin-retail/model.dae"/>
+    <origin xyz="5 5 0" />
+  </xacro:new_object>
+  <xacro:new_object new_object_num="11" >
+    <mesh filename="package://cob_gazebo_objects/Media/models/cabinet_ikea_galant.dae"/>
+    <origin xyz="-9 0 0" />
+  </xacro:new_object>
   <transmission name="belt_trans">
     <type>transmission_interface/SimpleTransmission</type>

Commit message: added hardwareInterface tag in Joint section of belt_trans transmission description

File: cob_gazebo_worlds/urdf/bmw-assembly/bmw-assembly.urdf.xacro (robot description, xacro)
@@ -213,5 +213,7 @@
   <transmission name="belt_trans">
     <type>transmission_interface/SimpleTransmission</type>
-    <joint name="base_to_belt" />
+    <joint name="base_to_belt">
+      <hardwareInterface>VelocityJointInterface</hardwareInterface>
+    </joint>
     <actuator name="belt_motor">
       <hardwareInterface>VelocityJointInterface</hardwareInterface>
