Commit message: changed color of boxes on the belt to grey

File: cob_gazebo_worlds/urdf/automotive-assembly-line/automotive-assembly-line.urdf.xacro (robot description, xacro)
@@ -44,5 +44,5 @@
     </link>
     <gazebo reference="box_${new_box_num}">
-      <material>Gazebo/Green</material>
+      <material>Gazebo/Grey</material>
     </gazebo>
     <joint name="belt_to_box_${new_box_num}" type="fixed">
