Commit message: removed the test object ramp

File: cob_gazebo_worlds/urdf/ipa-production-plant/machine-room.urdf.xacro (robot description, xacro)
@@ -2,8 +2,4 @@
 <robot xmlns:xacro="http://www.ros.org/wiki/xacro">
   <xacro:macro name="machine-room" params="name">
-  <xacro:object object_num="10" >
-    <mesh filename="package://cob_gazebo_objects/Media/models/ramp.dae"/>
-    <origin xyz="4 -12 0" />
-  </xacro:object>
   <xacro:object object_num="2a" >
     <mesh filename="package://cob_gazebo_worlds/Media/models/dump-bin-retail/model.dae"/>
