Commit message: Added some passages for the different rooms

File: cob_gazebo_worlds/urdf/ipa-production-plant/ipa-production-plant.property.xacro (robot description, xacro)
@@ -14,9 +14,9 @@
   <property name="room4_w1" value="36" />
   <property name="room4_w2" value="24" />
-  <property name="room4_w3" value="7.5" />
+  <property name="room4_w3" value="11.25" />
   <property name="room4_w4" value="7.5" />
-  <property name="room1_room2_w1" value="24" />
-  <property name="room1_room3_w1" value="22" />
-  <property name="room2_room4_w1" value="18" />
+  <property name="room1_room2_w1" value="10.5" />
+  <property name="room1_room3_w1" value="9.5" />
+  <property name="room2_room4_w1" value="11.25" />
   <property name="room3_room4_w1" value="17" />
   <property name="room3_room4_w2" value="4" />

File: cob_gazebo_worlds/urdf/ipa-production-plant/walls.urdf.xacro (robot description, xacro)
@@ -115,6 +115,6 @@
   </joint>
   <!-- room1_room2_w1 -->
-  <!-- wall_04 -->
-  <link name="wall_04">
+  <!-- wall_04a -->
+  <link name="wall_04a">
     <xacro:box_inertial x="${wall_depth}" y="${room1_room2_w1}" z="${wall_height}" mass="5.0">
       <origin xyz="0 0 0" rpy="0 0 0" />
@@ -134,15 +134,43 @@
     </collision>
   </link>
-  <gazebo reference="wall_04">
-    <material>wall_floor_05</material>
-  </gazebo>
-  <joint name="joint_wall_04" type="fixed">
-    <origin xyz="${22+position_offset_x} ${12+position_offset_y} ${wall_height/2+position_offset_z}" rpy="0 0 0" />
-    <parent link="world" />
-    <child link="wall_04" />
+  <gazebo reference="wall_04a">
+    <material>wall_floor_05</material>
+  </gazebo>
+  <joint name="joint_wall_04a" type="fixed">
+    <origin xyz="${22+position_offset_x} ${18.75+position_offset_y} ${wall_height/2+position_offset_z}" rpy="0 0 0" />
+    <parent link="world" />
+    <child link="wall_04a" />
+  </joint>
+    <!-- room1_room2_w1 -->
+  <!-- wall_04b -->
+  <link name="wall_04b">
+    <xacro:box_inertial x="${wall_depth}" y="${room1_room2_w1}" z="${wall_height}" mass="5.0">
+      <origin xyz="0 0 0" rpy="0 0 0" />
+    </xacro:box_inertial>
+    <visual>
+      <origin xyz="0 0 0" />
+      <geometry>
+        <box size="${wall_depth} ${room1_room2_w1} ${wall_height}" />
+      </geometry>
+      <material name="IPA/Grey"/>
+    </visual>
+    <collision>
+      <origin xyz="0 0 0" />
+      <geometry>
+        <box size="${wall_depth} ${room1_room2_w1} ${wall_height}" />
+      </geometry>
+    </collision>
+  </link>
+  <gazebo reference="wall_04b">
+    <material>wall_floor_05</material>
+  </gazebo>
+  <joint name="joint_wall_04b" type="fixed">
+    <origin xyz="${22+position_offset_x} ${5.25+position_offset_y} ${wall_height/2+position_offset_z}" rpy="0 0 0" />
+    <parent link="world" />
+    <child link="wall_04b" />
   </joint>
   <!-- room1_room3_w1 -->
-  <!-- wall_06 -->
-  <link name="wall_06">
+  <!-- wall_06a -->
+  <link name="wall_06a">
     <xacro:box_inertial x="${wall_depth}" y="${room1_room3_w1}" z="${wall_height}" mass="5.0">
       <origin xyz="0 0 0" rpy="0 0 0" />
@@ -162,11 +190,39 @@
     </collision>
   </link>
-  <gazebo reference="wall_06">
-    <material>wall_floor_05</material>
-  </gazebo>
-  <joint name="joint_wall_06" type="fixed">
-    <origin xyz="${11+position_offset_x} ${24+position_offset_y} ${wall_height/2+position_offset_z}" rpy="0 0 ${90*M_PI/180}" />
-    <parent link="world" />
-    <child link="wall_06" />
+  <gazebo reference="wall_06a">
+    <material>wall_floor_05</material>
+  </gazebo>
+  <joint name="joint_wall_06a" type="fixed">
+    <origin xyz="${4.75+position_offset_x} ${24+position_offset_y} ${wall_height/2+position_offset_z}" rpy="0 0 ${90*M_PI/180}" />
+    <parent link="world" />
+    <child link="wall_06a" />
+  </joint>
+  <!-- room1_room3_w1 -->
+  <!-- wall_06b -->
+  <link name="wall_06b">
+    <xacro:box_inertial x="${wall_depth}" y="${room1_room3_w1}" z="${wall_height}" mass="5.0">
+      <origin xyz="0 0 0" rpy="0 0 0" />
+    </xacro:box_inertial>
+    <visual>
+      <origin xyz="0 0 0" />
+      <geometry>
+        <box size="${wall_depth} ${room1_room3_w1} ${wall_height}" />
+      </geometry>
+      <material name="IPA/Grey"/>
+    </visual>
+    <collision>
+      <origin xyz="0 0 0" />
+      <geometry>
+        <box size="${wall_depth} ${room1_room3_w1} ${wall_height}" />
+      </geometry>
+    </collision>
+  </link>
+  <gazebo reference="wall_06b">
+    <material>wall_floor_05</material>
+  </gazebo>
+  <joint name="joint_wall_06b" type="fixed">
+    <origin xyz="${17.25+position_offset_x} ${24+position_offset_y} ${wall_height/2+position_offset_z}" rpy="0 0 ${90*M_PI/180}" />
+    <parent link="world" />
+    <child link="wall_06b" />
   </joint>
   <!-- room2_room4_w1 -->
@@ -194,5 +250,5 @@
   </gazebo>
   <joint name="joint_wall_07" type="fixed">
-    <origin xyz="${31+position_offset_x} ${24+position_offset_y} ${wall_height/2+position_offset_z}" rpy="0 0 ${90*M_PI/180}" />
+    <origin xyz="${27.625+position_offset_x} ${24+position_offset_y} ${wall_height/2+position_offset_z}" rpy="0 0 ${90*M_PI/180}" />
     <parent link="world" />
     <child link="wall_07" />
@@ -222,5 +278,5 @@
   </gazebo>
   <joint name="joint_wall_08" type="fixed">
-    <origin xyz="${43.75+position_offset_x} ${24+position_offset_y} ${wall_height/2+position_offset_z}" rpy="0 0 ${90*M_PI/180}" />
+    <origin xyz="${41.875+position_offset_x} ${24+position_offset_y} ${wall_height/2+position_offset_z}" rpy="0 0 ${90*M_PI/180}" />
     <parent link="world" />
     <child link="wall_08" />
@@ -418,5 +474,5 @@
   </gazebo>
   <joint name="joint_wall_15" type="fixed">
-    <origin xyz="${43.75+room4_w3/2+position_offset_x} ${12+position_offset_y} ${wall_height/2+position_offset_z}" rpy="0 0 0" />
+    <origin xyz="${47.5+position_offset_x} ${12+position_offset_y} ${wall_height/2+position_offset_z}" rpy="0 0 0" />
     <parent link="world" />
     <child link="wall_15" />

Commit message: Added new hallway to ipa_production_plant

File: cob_gazebo_worlds/urdf/ipa-production-plant/ipa-production-plant.property.xacro (robot description, xacro)
@@ -13,5 +13,5 @@
   <property name="room3_w2" value="22" />
   <property name="room4_w1" value="36" />
-  <property name="room4_w2" value="24" />
+  <property name="room4_w2" value="21" /> 24
   <property name="room4_w3" value="11.25" />
   <property name="room4_w4" value="7.5" />
@@ -24,4 +24,6 @@
   <property name="hallway_w2" value="58" />
   <property name="hallway_w3" value="5" />
+  <property name="hallway2_w1" value="3" />
+  <property name="hallway2_w2" value="53" />
   <property name="position_offset_x" value="-20" />
   <property name="position_offset_y" value="-35" />

File: cob_gazebo_worlds/urdf/ipa-production-plant/walls.urdf.xacro (robot description, xacro)
@@ -390,5 +390,5 @@
   </gazebo>
   <joint name="joint_wall_12" type="fixed">
-    <origin xyz="${58+position_offset_x} ${36+position_offset_y} ${wall_height/2+position_offset_z}" rpy="0 0 0" />
+    <origin xyz="${58+position_offset_x} ${34.5+position_offset_y} ${wall_height/2+position_offset_z}" rpy="0 0 0" />
     <parent link="world" />
     <child link="wall_12" />
@@ -590,4 +590,88 @@
     <child link="wall_19" />
   </joint>
+  <!-- hallway2 -->
+  <!-- wall_20 -->
+  <link name="wall_20">
+    <xacro:box_inertial x="${wall_depth}" y="${hallway2_w1}" z="${wall_height}" mass="5.0">
+      <origin xyz="0 0 0" rpy="0 0 0" />
+    </xacro:box_inertial>
+    <visual>
+      <origin xyz="0 0 0" />
+      <geometry>
+        <box size="${wall_depth} ${hallway2_w1} ${wall_height}" />
+      </geometry>
+      <material name="IPA/Grey"/>
+    </visual>
+    <collision>
+      <origin xyz="0 0 0" />
+      <geometry>
+        <box size="${wall_depth} ${hallway2_w1} ${wall_height}" />
+      </geometry>
+    </collision>
+  </link>
+  <gazebo reference="wall_20">
+    <material>wall_floor_05</material>
+  </gazebo>
+  <joint name="joint_wall_20" type="fixed">
+    <origin xyz="${hallway_w2+hallway2_w1/2+position_offset_x} ${-5+position_offset_y} ${wall_height/2+position_offset_z}" rpy="0 0 ${90*M_PI/180}" />
+    <parent link="world" />
+    <child link="wall_20" />
+  </joint>
+  <!-- hallway2 -->
+  <!-- wall_21 -->
+  <link name="wall_21">
+    <xacro:box_inertial x="${wall_depth}" y="${hallway2_w2}" z="${wall_height}" mass="5.0">
+      <origin xyz="0 0 0" rpy="0 0 0" />
+    </xacro:box_inertial>
+    <visual>
+      <origin xyz="0 0 0" />
+      <geometry>
+        <box size="${wall_depth} ${hallway2_w2} ${wall_height}" />
+      </geometry>
+      <material name="IPA/Grey"/>
+    </visual>
+    <collision>
+      <origin xyz="0 0 0" />
+      <geometry>
+        <box size="${wall_depth} ${hallway2_w2} ${wall_height}" />
+      </geometry>
+    </collision>
+  </link>
+  <gazebo reference="wall_21">
+    <material>wall_floor_05</material>
+  </gazebo>
+  <joint name="joint_wall_21" type="fixed">
+    <origin xyz="${hallway_w2+hallway2_w1+position_offset_x} ${hallway2_w2/2-5+position_offset_y} ${wall_height/2+position_offset_z}" rpy="0 0 0" />
+    <parent link="world" />
+    <child link="wall_21" />
+  </joint>
+  <!-- hallway2 -->
+  <!-- wall_22 -->
+  <link name="wall_22">
+    <xacro:box_inertial x="${wall_depth}" y="${hallway2_w1}" z="${wall_height}" mass="5.0">
+      <origin xyz="0 0 0" rpy="0 0 0" />
+    </xacro:box_inertial>
+    <visual>
+      <origin xyz="0 0 0" />
+      <geometry>
+        <box size="${wall_depth} ${hallway2_w1} ${wall_height}" />
+      </geometry>
+      <material name="IPA/Grey"/>
+    </visual>
+    <collision>
+      <origin xyz="0 0 0" />
+      <geometry>
+        <box size="${wall_depth} ${hallway2_w1} ${wall_height}" />
+      </geometry>
+    </collision>
+  </link>
+  <gazebo reference="wall_22">
+    <material>wall_floor_05</material>
+  </gazebo>
+  <joint name="joint_wall_22" type="fixed">
+    <origin xyz="${hallway_w2+hallway2_w1/2+position_offset_x} ${-5+hallway2_w2+position_offset_y} ${wall_height/2+position_offset_z}" rpy="0 0 ${90*M_PI/180}" />
+    <parent link="world" />
+    <child link="wall_22" />
+  </joint>
   </xacro:macro>
 </robot>
