Commit message: Updated some untitled namings

File: cob_gazebo_worlds/urdf/ipa-production-plant/ipa-production-plant.urdf.xacro (robot description, xacro)
@@ -36,17 +36,17 @@
   <!--world objects-->
   <xacro:object object_num="1a" >
-    <mesh filename = "package://cob_gazebo_worlds/Media/models/ipa-production-plant/wooden_container/untitled.dae" scale = "2.5 2.5 2.5"/>
+    <mesh filename = "package://cob_gazebo_worlds/Media/models/ipa-production-plant/wooden_container/wooden_container.dae" scale = "2.5 2.5 2.5"/>
     <origin xyz="-15 -20 0" />
   </xacro:object>
   <xacro:object object_num="1b" >
-    <mesh filename = "package://cob_gazebo_worlds/Media/models/ipa-production-plant/wooden_container/untitled.dae" scale = "2.5 2.5 2.5"/>
+    <mesh filename = "package://cob_gazebo_worlds/Media/models/ipa-production-plant/wooden_container/wooden_container.dae" scale = "2.5 2.5 2.5"/>
     <origin xyz="-5 -20 0" />
   </xacro:object>
   <xacro:object object_num="1c" >
-    <mesh filename = "package://cob_gazebo_worlds/Media/models/ipa-production-plant/wooden_container/untitled.dae" scale = "2.5 2.5 2.5"/>
+    <mesh filename = "package://cob_gazebo_worlds/Media/models/ipa-production-plant/wooden_container/wooden_container.dae" scale = "2.5 2.5 2.5"/>
     <origin xyz="-15 -30 0" />
   </xacro:object>
   <xacro:object object_num="1d" >
-    <mesh filename = "package://cob_gazebo_worlds/Media/models/ipa-production-plant/wooden_container/untitled.dae" scale = "2.5 2.5 2.5"/>
+    <mesh filename = "package://cob_gazebo_worlds/Media/models/ipa-production-plant/wooden_container/wooden_container.dae" scale = "2.5 2.5 2.5"/>
     <origin xyz="-5 -30 0" />
   </xacro:object>
@@ -80,45 +80,45 @@
   </xacro:object>
   <xacro:object object_num="4a" >
-    <mesh filename="package://cob_gazebo_worlds/Media/models/ipa-production-plant/back_workbench/models/untitled.dae"/>
+    <mesh filename="package://cob_gazebo_worlds/Media/models/ipa-production-plant/back_workbench/models/back_workbench.dae"/>
     <origin xyz="6 11 0" />
   </xacro:object>
   <xacro:object object_num="4b" >
-    <mesh filename="package://cob_gazebo_worlds/Media/models/ipa-production-plant/back_workbench/models/untitled.dae"/>
+    <mesh filename="package://cob_gazebo_worlds/Media/models/ipa-production-plant/back_workbench/models/back_workbench.dae"/>
     <origin xyz="11 11 0"/>
   </xacro:object>
   <xacro:object object_num="4c" >
-    <mesh filename="package://cob_gazebo_worlds/Media/models/ipa-production-plant/back_workbench/models/untitled.dae"/>
+    <mesh filename="package://cob_gazebo_worlds/Media/models/ipa-production-plant/back_workbench/models/back_workbench.dae"/>
     <origin xyz="16 11 0"/>
   </xacro:object>
   <xacro:object object_num="5a" >
-    <mesh filename="package://cob_gazebo_worlds/Media/models/ipa-production-plant/granite_assembly_bench/models/untitled.dae"/>
+    <mesh filename="package://cob_gazebo_worlds/Media/models/ipa-production-plant/granite_assembly_bench/models/granite_assembly_bench.dae"/>
     <origin xyz="10 0 0"/>
   </xacro:object>
   <xacro:object object_num="5b" >
-    <mesh filename="package://cob_gazebo_worlds/Media/models/ipa-production-plant/granite_assembly_bench/models/untitled.dae"/>
+    <mesh filename="package://cob_gazebo_worlds/Media/models/ipa-production-plant/granite_assembly_bench/models/granite_assembly_bench.dae"/>
     <origin xyz="13 0 0" />
   </xacro:object>
   <xacro:object object_num="5c" >
-    <mesh filename="package://cob_gazebo_worlds/Media/models/ipa-production-plant/granite_assembly_bench/models/untitled.dae"/>
+    <mesh filename="package://cob_gazebo_worlds/Media/models/ipa-production-plant/granite_assembly_bench/models/granite_assembly_bench.dae"/>
     <origin xyz="16 0 0" />
   </xacro:object>
   <xacro:object object_num="5d" >
-    <mesh filename="package://cob_gazebo_worlds/Media/models/ipa-production-plant/granite_assembly_bench/models/untitled.dae"/>
+    <mesh filename="package://cob_gazebo_worlds/Media/models/ipa-production-plant/granite_assembly_bench/models/granite_assembly_bench.dae"/>
     <origin xyz="19 0 0" />
   </xacro:object>
   <xacro:object object_num="5e" >
-    <mesh filename="package://cob_gazebo_worlds/Media/models/ipa-production-plant/granite_assembly_bench/models/untitled.dae"/>
+    <mesh filename="package://cob_gazebo_worlds/Media/models/ipa-production-plant/granite_assembly_bench/models/granite_assembly_bench.dae"/>
     <origin xyz="22 0 0" />
   </xacro:object>
   <xacro:object object_num="6a" >
-    <mesh filename="package://cob_gazebo_worlds/Media/models/ipa-production-plant/focus_stacking_platform/models/untitled.dae" scale = "8 8 8"/>
+    <mesh filename="package://cob_gazebo_worlds/Media/models/ipa-production-plant/focus_stacking_platform/models/focus_stacking_platform.dae" scale = "8 8 8"/>
     <origin xyz="28 5 0" />
   </xacro:object>
   <xacro:object object_num="6b" >
-    <mesh filename="package://cob_gazebo_worlds/Media/models/ipa-production-plant/focus_stacking_platform/models/untitled.dae" scale = "8 8 8"/>
+    <mesh filename="package://cob_gazebo_worlds/Media/models/ipa-production-plant/focus_stacking_platform/models/focus_stacking_platform.dae" scale = "8 8 8"/>
     <origin xyz="28 0 0" />
   </xacro:object>
   <xacro:object object_num="6c" >
-    <mesh filename="package://cob_gazebo_worlds/Media/models/ipa-production-plant/focus_stacking_platform/models/untitled.dae" scale = "8 8 8"/>
+    <mesh filename="package://cob_gazebo_worlds/Media/models/ipa-production-plant/focus_stacking_platform/models/focus_stacking_platform.dae" scale = "8 8 8"/>
     <origin xyz="28 -5 0" />
   </xacro:object>

Commit message: fix ipa-production-plant environment

File: cob_gazebo_worlds/urdf/ipa-production-plant/ipa-production-plant.urdf.xacro (robot description, xacro)
@@ -5,5 +5,11 @@
   <!--macros-->
   <xacro:macro name="object" params="object_num *mesh *origin">
+    <joint name="joint_object_${object_num}" type="fixed">
+       <insert_block name="origin"/>
+       <parent link="world"/>
+       <child link="object_${object_num}"/>
+    </joint>
     <link name="object_${object_num}">
+      <xacro:default_inertial/>
       <visual>
         <origin xyz="0 0 0" rpy="0 0 0"/>
@@ -18,5 +24,4 @@
         </geometry>
       </collision>
-      <xacro:default_inertial/>
     </link>
     <gazebo reference="object_${object_num}">
@@ -24,11 +29,6 @@
     </gazebo>
     <gazebo reference="object_${object_num}">
-	<turnGravityOff>false</turnGravityOff>
+      <turnGravityOff>false</turnGravityOff>
     </gazebo>
-    <joint name="joint_object_${object_num}" type="fixed">
-       <insert_block name="origin"/>
-       <parent link="world"/>
-       <child link="object_${object_num}"/>
-    </joint>
   </xacro:macro>
   <!-- world link -->

Commit message: Added static sensors to ipa-production-plant

File: cob_gazebo_worlds/urdf/ipa-production-plant/ipa-production-plant.urdf.xacro (robot description, xacro)
@@ -14,4 +14,6 @@
   <!-- work-area -->
   <!-- <xacro:include filename="$(find cob_gazebo_worlds)/urdf/ipa-production-plant/work-area.urdf.xacro" /> -->
+  <!-- sensors -->
+  <xacro:include filename="$(find cob_description)/urdf/sensors/sick_s300_laser.urdf.xacro"/>
   <!--macros-->
   <xacro:macro name="object" params="object_num *mesh *origin">
@@ -46,4 +48,21 @@
   <link name="world" />
   <!--world objects-->
+  <link name="sensors_link" />
+  <joint name="static_sensors_joint" type="fixed">
+    <parent link="world"/>
+    <child link="sensors_link"/>
+  </joint>
+  <xacro:sick_s300_laser_v0 name="static_laser_01" parent="sensors">
+    <origin xyz="19.08 -1.50 0.1" rpy="0 0 3.14" />
+    <gazebo>
+      <static>true</static>
+    </gazebo>
+  </xacro:sick_s300_laser_v0>
+  <xacro:sick_s300_laser_v0 name="static_laser_02" parent="sensors">
+    <origin xyz="27.08 -1.50 0.1" rpy="0 0 3.14" />
+    <gazebo>
+      <static>true</static>
+    </gazebo>
+  </xacro:sick_s300_laser_v0>
   <xacro:work-area name="work-area">
     </xacro:work-area>
