Commit message: Merged branch 'feature/ipa_production_plant_improvement' and updated the structure.

File: cob_gazebo_worlds/urdf/ipa-production-plant/ipa-production-plant.urdf.xacro (robot description, xacro)
@@ -1,545 +1,16 @@
 <?xml version="1.0"?>
-<robot xmlns:xacro="http://www.ros.org/wiki/xacro">
+<robot xmlns:xacro="http://www.ros.org/wiki/xacro"
+        name="ipa-production-plant">
   <xacro:include filename="$(find cob_gazebo_worlds)/urdf/common.xacro" />
   <xacro:include filename="$(find cob_gazebo_worlds)/urdf/ipa-production-plant/ipa-production-plant.property.xacro" />
-  <!--macros-->
-  <xacro:macro name="object" params="object_num *mesh *origin">
-    <joint name="joint_object_${object_num}" type="fixed">
-       <insert_block name="origin"/>
-       <parent link="world"/>
-       <child link="object_${object_num}"/>
-    </joint>
-    <link name="object_${object_num}">
-      <xacro:default_inertial/>
-      <visual>
-        <origin xyz="0 0 0" rpy="0 0 0"/>
-        <geometry>
-          <insert_block name = "mesh"/>
-        </geometry>
-      </visual>
-      <collision>
-        <origin xyz="0 0 0" rpy="0 0 0"/>
-        <geometry>
-          <insert_block name = "mesh"/>
-        </geometry>
-      </collision>
-    </link>
-    <gazebo reference="object_${object_num}">
-      <static>true</static>
-    </gazebo>
-    <gazebo reference="object_${object_num}">
-      <turnGravityOff>false</turnGravityOff>
-    </gazebo>
-  </xacro:macro>
+  <!-- walls -->
+  <xacro:include filename="$(find cob_gazebo_worlds)/urdf/ipa-production-plant/walls.urdf.xacro" />
+  <!-- sensors -->
+  <xacro:include filename="$(find cob_gazebo_worlds)/urdf/ipa-production-plant/sensors.urdf.xacro" />
   <!-- world link -->
   <link name="world" />
-  <!--world objects-->
-  <xacro:object object_num="1a" >
-    <mesh filename = "package://cob_gazebo_worlds/Media/models/ipa-production-plant/wooden_container/wooden_container.dae" scale = "2.5 2.5 2.5"/>
-    <origin xyz="-15 -20 0" />
-  </xacro:object>
-  <xacro:object object_num="1b" >
-    <mesh filename = "package://cob_gazebo_worlds/Media/models/ipa-production-plant/wooden_container/wooden_container.dae" scale = "2.5 2.5 2.5"/>
-    <origin xyz="-5 -20 0" />
-  </xacro:object>
-  <xacro:object object_num="1c" >
-    <mesh filename = "package://cob_gazebo_worlds/Media/models/ipa-production-plant/wooden_container/wooden_container.dae" scale = "2.5 2.5 2.5"/>
-    <origin xyz="-15 -30 0" />
-  </xacro:object>
-  <xacro:object object_num="1d" >
-    <mesh filename = "package://cob_gazebo_worlds/Media/models/ipa-production-plant/wooden_container/wooden_container.dae" scale = "2.5 2.5 2.5"/>
-    <origin xyz="-5 -30 0" />
-  </xacro:object>
-  <xacro:object object_num="2a" >
-    <mesh filename="package://cob_gazebo_worlds/Media/models/dump-bin-retail/model.dae"/>
-    <origin xyz="6 -10 0" />
-  </xacro:object>
-  <xacro:object object_num="2b" >
-    <mesh filename="package://cob_gazebo_worlds/Media/models/dump-bin-retail/model.dae"/>
-    <origin xyz="11 -10 0" />
-  </xacro:object>
-  <xacro:object object_num="2c" >
-    <mesh filename="package://cob_gazebo_worlds/Media/models/dump-bin-retail/model.dae"/>
-    <origin xyz="16 -10 0" />
-  </xacro:object>
-  <xacro:object object_num="2d" >
-    <mesh filename="package://cob_gazebo_worlds/Media/models/dump-bin-retail/model.dae"/>
-    <origin xyz="21 -10 0" />
-  </xacro:object>
-  <xacro:object object_num="3a" >
-    <mesh filename="package://cob_gazebo_objects/Media/models/cabinet_ikea_galant.dae"/>
-    <origin xyz="2.2 3 0"/>
-  </xacro:object>
-  <xacro:object object_num="3b" >
-    <mesh filename="package://cob_gazebo_objects/Media/models/cabinet_ikea_galant.dae"/>
-    <origin xyz="2.2 0 0"/>
-  </xacro:object>
-  <xacro:object object_num="3c" >
-    <mesh filename="package://cob_gazebo_objects/Media/models/cabinet_ikea_galant.dae"/>
-    <origin xyz="2.2 -3 0"/>
-  </xacro:object>
-  <xacro:object object_num="4a" >
-    <mesh filename="package://cob_gazebo_worlds/Media/models/ipa-production-plant/back_workbench/models/back_workbench.dae"/>
-    <origin xyz="6 11 0" />
-  </xacro:object>
-  <xacro:object object_num="4b" >
-    <mesh filename="package://cob_gazebo_worlds/Media/models/ipa-production-plant/back_workbench/models/back_workbench.dae"/>
-    <origin xyz="11 11 0"/>
-  </xacro:object>
-  <xacro:object object_num="4c" >
-    <mesh filename="package://cob_gazebo_worlds/Media/models/ipa-production-plant/back_workbench/models/back_workbench.dae"/>
-    <origin xyz="16 11 0"/>
-  </xacro:object>
-  <xacro:object object_num="5a" >
-    <mesh filename="package://cob_gazebo_worlds/Media/models/ipa-production-plant/granite_assembly_bench/models/granite_assembly_bench.dae"/>
-    <origin xyz="10 0 0"/>
-  </xacro:object>
-  <xacro:object object_num="5b" >
-    <mesh filename="package://cob_gazebo_worlds/Media/models/ipa-production-plant/granite_assembly_bench/models/granite_assembly_bench.dae"/>
-    <origin xyz="13 0 0" />
-  </xacro:object>
-  <xacro:object object_num="5c" >
-    <mesh filename="package://cob_gazebo_worlds/Media/models/ipa-production-plant/granite_assembly_bench/models/granite_assembly_bench.dae"/>
-    <origin xyz="16 0 0" />
-  </xacro:object>
-  <xacro:object object_num="5d" >
-    <mesh filename="package://cob_gazebo_worlds/Media/models/ipa-production-plant/granite_assembly_bench/models/granite_assembly_bench.dae"/>
-    <origin xyz="19 0 0" />
-  </xacro:object>
-  <xacro:object object_num="5e" >
-    <mesh filename="package://cob_gazebo_worlds/Media/models/ipa-production-plant/granite_assembly_bench/models/granite_assembly_bench.dae"/>
-    <origin xyz="22 0 0" />
-  </xacro:object>
-  <xacro:object object_num="6a" >
-    <mesh filename="package://cob_gazebo_worlds/Media/models/ipa-production-plant/focus_stacking_platform/models/focus_stacking_platform.dae" scale = "8 8 8"/>
-    <origin xyz="28 5 0" />
-  </xacro:object>
-  <xacro:object object_num="6b" >
-    <mesh filename="package://cob_gazebo_worlds/Media/models/ipa-production-plant/focus_stacking_platform/models/focus_stacking_platform.dae" scale = "8 8 8"/>
-    <origin xyz="28 0 0" />
-  </xacro:object>
-  <xacro:object object_num="6c" >
-    <mesh filename="package://cob_gazebo_worlds/Media/models/ipa-production-plant/focus_stacking_platform/models/focus_stacking_platform.dae" scale = "8 8 8"/>
-    <origin xyz="28 -5 0" />
-  </xacro:object>
-  <!-- room1_w1 -->
-  <!-- wall_01 -->
-  <link name="wall_01">
-    <xacro:box_inertial x="${wall_depth}" y= "${room1_w1}" z="${wall_height}" mass="5.0">
-      <origin xyz="0 0 0" rpy="0 0 0" />
-    </xacro:box_inertial>
-    <visual>
-      <origin xyz="0 0 0" />
-      <geometry>
-        <box size="${wall_depth} ${room1_w1} ${wall_height}" />
-      </geometry>
-      <material name="IPA/Grey"/>
-    </visual>
-    <collision>
-      <origin xyz="0 0 0" />
-      <geometry>
-        <box size="${wall_depth} ${room1_w1} ${wall_height}" />
-      </geometry>
-    </collision>
-  </link>
-  <gazebo reference="wall_01">
-    <material>wall_floor_05</material>
-  </gazebo>
-  <joint name="joint_wall_01" type="fixed">
-    <origin xyz="${4.75+position_offset_x} ${position_offset_y} ${wall_height/2+position_offset_z}" rpy="0 0 ${90*M_PI/180}" />
-    <parent link="world" />
-    <child link="wall_01" />
-  </joint>
-  <!-- room1_w2 -->
-  <!-- wall_02 -->
-  <link name="wall_02">
-    <xacro:box_inertial x="${wall_depth}" y="${room1_w2}" z="${wall_height}" mass="5.0">
-      <origin xyz="0 0 0" rpy="0 0 0" />
-    </xacro:box_inertial>
-    <visual>
-      <origin xyz="0 0 0" />
-      <geometry>
-        <box size="${wall_depth} ${room1_w2} ${wall_height}" />
-      </geometry>
-      <material name="IPA/Grey"/>
-    </visual>
-    <collision>
-      <origin xyz="0 0 0" />
-      <geometry>
-        <box size="${wall_depth} ${room1_w2} ${wall_height}" />
-      </geometry>
-    </collision>
-  </link>
-  <gazebo reference="wall_02">
-    <material>wall_floor_05</material>
-  </gazebo>
-  <joint name="joint_wall_02" type="fixed">
-    <origin xyz="${17.25+position_offset_x} ${position_offset_y} ${wall_height/2+position_offset_z}" rpy="0 0 ${90*M_PI/180}" />
-    <parent link="world" />
-    <child link="wall_02" />
-  </joint>
-  <!-- room2_w1 -->
-  <!-- wall_02b -->
-  <link name="wall_02b">
-    <xacro:box_inertial x="${wall_depth}" y="${room2_w1}" z="${wall_height}" mass="5.0">
-      <origin xyz="0 0 0" rpy="0 0 0" />
-    </xacro:box_inertial>
-    <visual>
-      <origin xyz="0 0 0" />
-      <geometry>
-        <box size="${wall_depth} ${room2_w1} ${wall_height}" />
-      </geometry>
-      <material name="IPA/Grey"/>
-    </visual>
-    <collision>
-      <origin xyz="0 0 0" />
-      <geometry>
-        <box size="${wall_depth} ${room2_w1} ${wall_height}" />
-      </geometry>
-    </collision>
-  </link>
-  <gazebo reference="wall_02b">
-    <material>wall_floor_05</material>
-  </gazebo>
-  <joint name="joint_wall_02b" type="fixed">
-    <origin xyz="${31+position_offset_x} ${position_offset_y} ${wall_height/2+position_offset_z}" rpy="0 0 ${90*M_PI/180}" />
-    <parent link="world" />
-    <child link="wall_02b" />
-  </joint>
-  <!-- room1_w3 -->
-  <!-- wall_03 -->
-  <link name="wall_03">
-    <xacro:box_inertial x="${wall_depth}" y="${room1_w3}" z="${wall_height}" mass="5.0">
-      <origin xyz="0 0 0" rpy="0 0 0" />
-    </xacro:box_inertial>
-    <visual>
-      <origin xyz="0 0 0" />
-      <geometry>
-        <box size="${wall_depth} ${room1_w3} ${wall_height}" />
-      </geometry>
-      <material name="IPA/Grey"/>
-    </visual>
-    <collision>
-      <origin xyz="0 0 0" />
-      <geometry>
-        <box size="${wall_depth} ${room1_w3} ${wall_height}" />
-      </geometry>
-    </collision>
-  </link>
-  <gazebo reference="wall_03">
-    <material>wall_floor_05</material>
-  </gazebo>
-  <joint name="joint_wall_03" type="fixed">
-    <origin xyz="${position_offset_x} ${12+position_offset_y} ${wall_height/2+position_offset_z}" rpy="0 0 0" />
-    <parent link="world" />
-    <child link="wall_03" />
-  </joint>
-  <!-- room1_room2_w1 -->
-  <!-- wall_04 -->
-  <link name="wall_04">
-    <xacro:box_inertial x="${wall_depth}" y="${room1_room2_w1}" z="${wall_height}" mass="5.0">
-      <origin xyz="0 0 0" rpy="0 0 0" />
-    </xacro:box_inertial>
-    <visual>
-      <origin xyz="0 0 0" />
-      <geometry>
-        <box size="${wall_depth} ${room1_room2_w1} ${wall_height}" />
-      </geometry>
-      <material name="IPA/Grey"/>
-    </visual>
-    <collision>
-      <origin xyz="0 0 0" />
-      <geometry>
-        <box size="${wall_depth} ${room1_room2_w1} ${wall_height}" />
-      </geometry>
-    </collision>
-  </link>
-  <gazebo reference="wall_04">
-    <material>wall_floor_05</material>
-  </gazebo>
-  <joint name="joint_wall_04" type="fixed">
-    <origin xyz="${22+position_offset_x} ${12+position_offset_y} ${wall_height/2+position_offset_z}" rpy="0 0 0" />
-    <parent link="world" />
-    <child link="wall_04" />
-  </joint>
-  <!-- room2_w2 -->
-  <!-- wall_05 -->
-  <link name="wall_05">
-    <xacro:box_inertial x="${wall_depth}" y="${room2_w2}" z="${wall_height}" mass="5.0">
-      <origin xyz="0 0 0" rpy="0 0 0" />
-    </xacro:box_inertial>
-    <visual>
-      <origin xyz="0 0 0" />
-      <geometry>
-        <box size="${wall_depth} ${room2_w2} ${wall_height}" />
-      </geometry>
-      <material name="IPA/Grey"/>
-    </visual>
-    <collision>
-      <origin xyz="0 0 0" />
-      <geometry>
-        <box size="${wall_depth} ${room2_w2} ${wall_height}" />
-      </geometry>
-    </collision>
-  </link>
-  <gazebo reference="wall_05">
-    <material>wall_floor_05</material>
-  </gazebo>
-  <joint name="joint_wall_05" type="fixed">
-    <origin xyz="${40+position_offset_x} ${13.5+position_offset_y} ${wall_height/2+position_offset_z}" rpy="0 0 0" />
-    <parent link="world" />
-    <child link="wall_05" />
-  </joint>
-  <!-- room1_room3_w1 -->
-  <!-- wall_06 -->
-  <link name="wall_06">
-    <xacro:box_inertial x="${wall_depth}" y="${room1_room3_w1}" z="${wall_height}" mass="5.0">
-      <origin xyz="0 0 0" rpy="0 0 0" />
-    </xacro:box_inertial>
-    <visual>
-      <origin xyz="0 0 0" />
-      <geometry>
-        <box size="${wall_depth} ${room1_room3_w1} ${wall_height}" />
-      </geometry>
-      <material name="IPA/Grey"/>
-    </visual>
-    <collision>
-      <origin xyz="0 0 0" />
-      <geometry>
-        <box size="${wall_depth} ${room1_room3_w1} ${wall_height}" />
-      </geometry>
-    </collision>
-  </link>
-  <gazebo reference="wall_06">
-    <material>wall_floor_05</material>
-  </gazebo>
-  <joint name="joint_wall_06" type="fixed">
-    <origin xyz="${11+position_offset_x} ${24+position_offset_y} ${wall_height/2+position_offset_z}" rpy="0 0 ${90*M_PI/180}" />
-    <parent link="world" />
-    <child link="wall_06" />
-  </joint>
-  <!-- room2_room4_w1 -->
-  <!-- wall_07 -->
-  <link name="wall_07">
-    <xacro:box_inertial x="${wall_depth}" y="${room2_room4_w1}" z="${wall_height}" mass="5.0">
-      <origin xyz="0 0 0" rpy="0 0 0" />
-    </xacro:box_inertial>
-    <visual>
-      <origin xyz="0 0 0" />
-      <geometry>
-        <box size="${wall_depth} ${room2_room4_w1} ${wall_height}" />
-      </geometry>
-      <material name="IPA/Grey"/>
-    </visual>
-    <collision>
-      <origin xyz="0 0 0" />
-      <geometry>
-        <box size="${wall_depth} ${room2_room4_w1} ${wall_height}" />
-      </geometry>
-    </collision>
-  </link>
-  <gazebo reference="wall_07">
-    <material>wall_floor_05</material>
-  </gazebo>
-  <joint name="joint_wall_07" type="fixed">
-    <origin xyz="${31+position_offset_x} ${24+position_offset_y} ${wall_height/2+position_offset_z}" rpy="0 0 ${90*M_PI/180}" />
-    <parent link="world" />
-    <child link="wall_07" />
-  </joint>
-  <!-- room4_w3 -->
-  <!-- wall_08 -->
-  <link name="wall_08">
-    <xacro:box_inertial x="${wall_depth}" y="${room4_w3}" z="${wall_height}" mass="5.0">
-      <origin xyz="0 0 0" rpy="0 0 0" />
-    </xacro:box_inertial>
-    <visual>
-      <origin xyz="0 0 0" />
-      <geometry>
-        <box size="${wall_depth} ${room4_w3} ${wall_height}" />
-      </geometry>
-      <material name="IPA/Grey"/>
-    </visual>
-    <collision>
-      <origin xyz="0 0 0" />
-      <geometry>
-        <box size="${wall_depth} ${room4_w3} ${wall_height}" />
-      </geometry>
-    </collision>
-  </link>
-  <gazebo reference="wall_08">
-    <material>wall_floor_05</material>
-  </gazebo>
-  <joint name="joint_wall_08" type="fixed">
-    <origin xyz="${43.75+position_offset_x} ${24+position_offset_y} ${wall_height/2+position_offset_z}" rpy="0 0 ${90*M_PI/180}" />
-    <parent link="world" />
-    <child link="wall_08" />
-  </joint>
-  <!-- room4_w4 -->
-  <!-- wall_09 -->
-  <link name="wall_09">
-    <xacro:box_inertial x="${wall_depth}" y="${room4_w4}" z="${wall_height}" mass="5.0">
-      <origin xyz="0 0 0" rpy="0 0 0" />
-    </xacro:box_inertial>
-    <visual>
-      <origin xyz="0 0 0" />
-      <geometry>
-        <box size="${wall_depth} ${room4_w4} ${wall_height}" />
-      </geometry>
-      <material name="IPA/Grey"/>
-    </visual>
-    <collision>
-      <origin xyz="0 0 0" />
-      <geometry>
-        <box size="${wall_depth} ${room4_w4} ${wall_height}" />
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
Commit message: fix ipa-production-plant

File: cob_gazebo_worlds/urdf/ipa-production-plant/ipa-production-plant.urdf.xacro (robot description, xacro)
@@ -1,5 +1,5 @@
 <?xml version="1.0"?>
 <robot xmlns:xacro="http://www.ros.org/wiki/xacro"
-        name="ipa-production-plant">
+       name="ipa-production-plant">
   <xacro:include filename="$(find cob_gazebo_worlds)/urdf/common.xacro" />
   <xacro:include filename="$(find cob_gazebo_worlds)/urdf/ipa-production-plant/ipa-production-plant.property.xacro" />
@@ -11,8 +11,6 @@
   <link name="world" />
   <!-- Spawn Walls -->
-  <xacro:sensors name="sensors">
-    </xacro:sensors>
+  <xacro:sensors name="sensors"/>
   <!-- Spawn Walls -->
-  <xacro:walls name="walls">
-    </xacro:walls>
+  <xacro:walls name="walls"/>
 </robot>

File: cob_gazebo_worlds/urdf/ipa-production-plant/sensors.urdf.xacro (robot description, xacro)
@@ -3,24 +3,18 @@
   <xacro:include filename="$(find cob_description)/urdf/sensors/sick_s300_laser.urdf.xacro"/>
   <xacro:macro name="sensors" params="name">
-  <!-- sensor link -->
-  <link name="sensors_link" />
-  <!-- connect links -->
-  <joint name="static_sensors_joint" type="fixed">
-    <parent link="world"/>
-    <child link="sensors_link"/>
-  </joint>
-  <!-- Spawn Sensors -->
-  <xacro:sick_s300_laser_v0 name="static_laser_01" parent="sensors">
-    <origin xyz="19.08 -1.50 0.1" rpy="0 0 3.14" />
-    <gazebo>
-      <static>true</static>
-    </gazebo>
-  </xacro:sick_s300_laser_v0>
-  <xacro:sick_s300_laser_v0 name="static_laser_02" parent="sensors">
-    <origin xyz="27.08 -1.50 0.1" rpy="0 0 3.14" />
-    <gazebo>
-      <static>true</static>
-    </gazebo>
-  </xacro:sick_s300_laser_v0>
+    <!-- sensor link -->
+    <link name="sensors_link" />
+    <!-- connect links -->
+    <joint name="static_sensors_joint" type="fixed">
+      <parent link="world"/>
+      <child link="sensors_link"/>
+    </joint>
+    <!-- Spawn Sensors -->
+    <xacro:sick_s300_laser_v0 name="static_laser_01" parent="sensors_link">
+      <origin xyz="19.08 -1.50 0.1" rpy="0 0 3.14" />
+    </xacro:sick_s300_laser_v0>
+    <xacro:sick_s300_laser_v0 name="static_laser_02" parent="sensors_link">
+      <origin xyz="27.08 -1.50 0.1" rpy="0 0 3.14" />
+    </xacro:sick_s300_laser_v0>
   </xacro:macro>
 </robot>
