Commit message: Moved ipa-office walls to cob gazebo worlds

File: cob_gazebo_worlds/urdf/ipa-office/ipa-office.urdf.xacro (robot description, xacro)
@@ -2,4 +2,6 @@
 <robot xmlns:xacro="http://www.ros.org/wiki/xacro"
        name="ipa-office">
+  <xacro:include filename="$(find cob_gazebo_worlds)/urdf/common.xacro" />
+  <xacro:include filename="$(find cob_gazebo_worlds)/urdf/materials.urdf.xacro" />
   <xacro:macro name="ipa-office" params="name">
     <gazebo>
@@ -10,4 +12,31 @@
     </gazebo>
     <link name="world"/>
+    <link name="walls">
+      <inertial>
+        <mass value="1.37" />
+        <origin xyz="0 0 0.0" />
+        <inertia ixx="1.0" ixy="0.0" ixz="0.0" iyy="1.0" iyz="0.0" izz="1.0"/>
+      </inertial>
+      <visual>
+        <origin xyz="6.75 0.25 0" rpy="0 0 0" />
+        <geometry>
+          <mesh filename="package://cob_gazebo_worlds/Media/models/ipa-office_walls.dae" scale="0.97 0.97 0.97"/>
+        </geometry>
+      </visual>
+      <collision>
+        <origin xyz="6.75 0.25 0" rpy="0 0 0" />
+        <geometry>
+          <mesh filename="package://cob_gazebo_worlds/Media/models/ipa-office_walls.dae" scale="0.97 0.97 0.97"/>
+        </geometry>
+      </collision>
+    </link>
+    <gazebo>
+      <static>true</static>
+    </gazebo>
+    <joint name="joint_walls" type="fixed">
+      <origin xyz="0 0 0" rpy="0 0 0" />
+      <parent link="world" />
+      <child link="walls" />
+    </joint>
   </xacro:macro>
   <xacro:ipa-office name="ipa-office" />
