Commit message: conflict between empty launch files and other scenarios solved

File: cob_gazebo_worlds/urdf/empty/empty.urdf.xacro (robot description, xacro)
@@ -2,9 +2,4 @@
 <robot xmlns:xacro="http://www.ros.org/wiki/xacro"
        name="empty">
-  <xacro:include filename="$(find cob_gazebo_worlds)/urdf/common.xacro" />
-  <xacro:include filename="$(find cob_gazebo_worlds)/urdf/materials.urdf.xacro" />
-  <!--Parameters-->
-  <property name="dist_axis_x" value="1.969" />
-  <property name="dist_axis_y" value="4.070" />
   <xacro:macro name="empty" params="name">
     <gazebo>
@@ -15,7 +10,4 @@
     </gazebo>
     <link name="world"/>
-    <xacro:landing name="landing" parent="world">
-        <origin xyz="${-13.9+dist_axis_x} ${-dist_axis_y} 0" rpy="0 0 0" />
-    </xacro:landing>
   </xacro:macro>
   <xacro:empty name="empty" />

Commit message: simplify launch files

File: cob_gazebo_worlds/urdf/empty/empty.urdf.xacro (robot description, xacro)
@@ -2,13 +2,4 @@
 <robot xmlns:xacro="http://www.ros.org/wiki/xacro"
        name="empty">
-  <xacro:macro name="empty" params="name">
-    <gazebo>
-      <plugin name="environment_gazebo_ros_control" filename="libgazebo_ros_control.so">
-        <robotNamespace>world</robotNamespace>
-        <robotParam>/world_description</robotParam>
-      </plugin>
-    </gazebo>
-    <link name="world"/>
-  </xacro:macro>
-  <xacro:empty name="empty" />
+  <link name="world"/>
 </robot>
