Commit message: rename IZS-carpark-top to izs-carpark-top

File: cob_gazebo_worlds/urdf/izs-carpark-top/izs-carpark-top.urdf.xacro (robot description, xacro)
@@ -1,10 +1,10 @@
 <?xml version="1.0"?>
 <robot xmlns:xacro="http://www.ros.org/wiki/xacro"
-       name="IZS-carpark-top">
+       name="izs-carpark-top">
   <xacro:include filename="$(find cob_gazebo_worlds)/urdf/common.xacro" />
   <xacro:include filename="$(find cob_gazebo_worlds)/urdf/materials.urdf.xacro" />
-  <xacro:macro name="IZS-carpark-top" params="name">
+  <xacro:macro name="izs-carpark-top" params="name">
   </xacro:macro>
-  <xacro:macro name="IZS-carpark-top" params="name">
+  <xacro:macro name="izs-carpark-top" params="name">
   <gazebo>
     <plugin name="environment_gazebo_ros_control" filename="libgazebo_ros_control.so">
@@ -303,4 +303,4 @@
   </joint>
   </xacro:macro>
-  <xacro:IZS-carpark-top name="IZS-carpark-top" />
+  <xacro:izs-carpark-top name="izs-carpark-top" />
 </robot>
